File: hardware/ws2812matrix/ws2812matrix.sch (KiCad schematic (older format))
At the start: 129 parts, among them J1 STM32WORLD_BASE

Commit message: Hmmm
Other:
- moved on the sheet: C1, C10, C11, C12, C13, C14, C15, C16, C17, C18, C19, C2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
