File: hardware/ws2812matrix/ws2812matrix.kicad_pcb (KiCad board)
At the start: 2 copper layers, 76.2 x 50.8 mm, 129 parts, among them J1 STM32WORLD_BASE

Commit message: Hmmmm
Routing:
- net Net-(D8-Pad1): track 34.8 -> 36.5 mm, vias 0 -> 2
- net Net-(D16-Pad1): track 34.8 -> 36.3 mm, vias 0 -> 2
- net +5V: track 433.4 -> 434.1 mm
