File: hardware/usbser/usbser.kicad_pcb (KiCad board)
At the start: 2 copper layers, 76.2 x 50.8 mm, 18 parts, among them J2 STM32WORLD_BASE, U1 XC6206P332MR, U2 CP2102N

Commit message: Hmmmm
Parts:
- removed R3, R4: 22R, Resistor_SMD:R_0402_1005Metric
- added U3: SRV05-4, Package_TO_SOT_SMD:SOT-23-6, F.Cu at (179.7, 110.5)
- moved C1 22.9 mm to (181.1, 92.5)
- moved C2 22.9 mm to (177.0, 92.5)
- moved D1 22.9 mm to (184.8, 89.5)
- moved U1 22.9 mm to (179.1, 89.5)
- moved R2 3.28 mm to (179.7, 98.4)
- moved R1 2.01 mm to (179.7, 104.8)
Connections:
- J1 pad A6: Net-(J1-PadA6) -> DP
- J1 pad A7: Net-(J1-PadA7) -> DM
- J1 pad B6: Net-(J1-PadA6) -> DP
- J1 pad B7: Net-(J1-PadA7) -> DM
