File: hardware/mcuf405/mcuf405.kicad_pcb (KiCad board)
At the start: 2 copper layers, 76.2 x 50.8 mm, 35 parts, among them J4 STM32WORLD_BASE, U1 STM32F405RGTx, U2 XC6206P332MR, Y1 16 MHz

Commit message: Hmmmm
Parts:
- moved J4 52.8 mm to (234.3, 102.2)
Connections:
- J1 pad 10: PA5 -> Net-(J1-Pad10)
- J1 pad 11: PA6 -> Net-(J1-Pad11)
- J1 pad 12: PA7 -> Net-(J1-Pad12)
- J1 pad 13: PA8 -> Net-(J1-Pad13)
- J1 pad 14: PA9 -> Net-(J1-Pad14)
- J1 pad 15: PA10 -> Net-(J1-Pad15)
- J1 pad 16: PA11 -> Net-(J1-Pad16)
- J1 pad 17: PA12 -> Net-(J1-Pad17)
- J1 pad 18: PA13 -> Net-(J1-Pad18)
- J1 pad 19: PA14 -> Net-(J1-Pad19)
- J1 pad 20: PA15 -> Net-(J1-Pad20)
- J1 pad 21: PB0 -> Net-(J1-Pad21)
- J1 pad 22: PB1 -> Net-(J1-Pad22)
- J1 pad 23: PB2 -> Net-(J1-Pad23)
- J1 pad 24: PB3 -> Net-(J1-Pad24)
- J1 pad 25: PB4 -> Net-(J1-Pad25)
- J1 pad 26: PB5 -> Net-(J1-Pad26)
- J1 pad 27: PB6 -> Net-(J1-Pad27)
- J1 pad 28: PB7 -> Net-(J1-Pad28)
- J1 pad 29: PB8 -> Net-(J1-Pad29)
- J1 pad 30: PB9 -> Net-(J1-Pad30)
- J1 pad 31: PB10 -> Net-(J1-Pad31)
- J1 pad 32: PB11 -> Net-(J1-Pad32)
- J1 pad 33: PB12 -> Net-(J1-Pad33)
- J1 pad 34: PB13 -> Net-(J1-Pad34)
- J1 pad 35: PB14 -> Net-(J1-Pad35)
- J1 pad 36: PB15 -> Net-(J1-Pad36)
- J1 pad 5: PA0 -> Net-(J1-Pad5)
- J1 pad 6: PA1 -> Net-(J1-Pad6)
- J1 pad 7: PA2 -> Net-(J1-Pad7)
- J1 pad 8: PA3 -> Net-(J1-Pad8)
- J1 pad 9: PA4 -> Net-(J1-Pad9)
- J4 pad 10: (no net) -> PA5
- J4 pad 11: (no net) -> PA6
- J4 pad 12: (no net) -> PA7
- J4 pad 13: (no net) -> PA8
- J4 pad 14: (no net) -> PA9
- J4 pad 15: (no net) -> PA10
- J4 pad 16: (no net) -> PA11
- J4 pad 17: (no net) -> PA12
- J4 pad 18: (no net) -> PA13
- J4 pad 19: (no net) -> PA14
- J4 pad 2: (no net) -> Net-(J4-Pad2)
- J4 pad 20: (no net) -> PA15
- J4 pad 21: (no net) -> PB0
- J4 pad 22: (no net) -> PB1
- J4 pad 23: (no net) -> PB2
- J4 pad 24: (no net) -> PB3
- J4 pad 25: (no net) -> PB4
- J4 pad 26: (no net) -> PB5
- J4 pad 27: (no net) -> PB6
- J4 pad 28: (no net) -> PB7
- J4 pad 29: (no net) -> PB8
- J4 pad 3: (no net) -> Net-(J4-Pad3)
- J4 pad 30: (no net) -> PB9
- J4 pad 31: (no net) -> PB10
- J4 pad 32: (no net) -> PB11
- J4 pad 33: (no net) -> PB12
- J4 pad 34: (no net) -> PB13
- J4 pad 35: (no net) -> PB14
- J4 pad 36: (no net) -> PB15
- J4 pad 37: (no net) -> Net-(J4-Pad37)
- J4 pad 38: (no net) -> Net-(J4-Pad38)
- J4 pad 39: (no net) -> Net-(J4-Pad39)
- J4 pad 4: (no net) -> Net-(J4-Pad4)
- J4 pad 40: (no net) -> Net-(J4-Pad40)
- J4 pad 41: (no net) -> Net-(J4-Pad41)
- J4 pad 42: (no net) -> Net-(J4-Pad42)
- J4 pad 43: (no net) -> Net-(J4-Pad43)
- J4 pad 44: (no net) -> Net-(J4-Pad44)
- J4 pad 45: (no net) -> Net-(J4-Pad45)
- J4 pad 46: (no net) -> Net-(J4-Pad46)
- J4 pad 47: (no net) -> Net-(J4-Pad47)
- J4 pad 48: (no net) -> Net-(J4-Pad48)
- J4 pad 49: (no net) -> Net-(J4-Pad49)
- J4 pad 5: (no net) -> PA0
- J4 pad 50: (no net) -> Net-(J4-Pad50)
- J4 pad 51: (no net) -> Net-(J4-Pad51)
- J4 pad 52: (no net) -> Net-(J4-Pad52)
- J4 pad 53: (no net) -> Net-(J4-Pad53)
- J4 pad 54: (no net) -> Net-(J4-Pad54)
- J4 pad 55: (no net) -> Net-(J4-Pad55)
- J4 pad 56: (no net) -> Net-(J4-Pad56)
- J4 pad 57: (no net) -> Net-(J4-Pad57)
- J4 pad 58: (no net) -> Net-(J4-Pad58)
- J4 pad 59: (no net) -> Net-(J4-Pad59)
- J4 pad 6: (no net) -> PA1
- J4 pad 60: (no net) -> Net-(J4-Pad60)
- J4 pad 61: (no net) -> Net-(J4-Pad61)
- J4 pad 62: (no net) -> Net-(J4-Pad62)
- J4 pad 63: (no net) -> Net-(J4-Pad63)
- J4 pad 64: (no net) -> Net-(J4-Pad64)
- J4 pad 65: (no net) -> Net-(J4-Pad65)
- J4 pad 66: (no net) -> Net-(J4-Pad66)
- J4 pad 67: (no net) -> Net-(J4-Pad67)
- J4 pad 68: (no net) -> Net-(J4-Pad68)
- J4 pad 69: (no net) -> Net-(J4-Pad69)
- J4 pad 7: (no net) -> PA2
- J4 pad 70: (no net) -> Net-(J4-Pad70)
- J4 pad 71: (no net) -> Net-(J4-Pad71)
- J4 pad 72: (no net) -> Net-(J4-Pad72)
- J4 pad 73: (no net) -> Net-(J4-Pad73)
- J4 pad 74: (no net) -> Net-(J4-Pad74)
- J4 pad 75: (no net) -> Net-(J4-Pad75)
- J4 pad 76: (no net) -> Net-(J4-Pad76)
- J4 pad 77: (no net) -> Net-(J4-Pad77)
- J4 pad 78: (no net) -> Net-(J4-Pad78)
- J4 pad 79: (no net) -> Net-(J4-Pad79)
- J4 pad 8: (no net) -> PA3
- J4 pad 80: (no net) -> Net-(J4-Pad80)
- J4 pad 9: (no net) -> PA4

Commit message: Hmmmm
Parts:
- removed J1, J2: ~, stm32world:PinSocket_2x20_P2.54mm_Vertical_Stackable
- moved J4 81.9 mm to (152.4, 101.6)
- moved C8 6.54 mm to (146.7, 109.2)
- moved D2 6.35 mm to (116.8, 92.7)
- moved R7 6.35 mm to (119.4, 92.7)
Connections:
- J4 pad 1: Net-(J4-Pad1) -> +3V3
- J4 pad 10: PA5 -> PA1
- J4 pad 11: PA6 -> PA2
- J4 pad 12: PA7 -> PA3
- J4 pad 13: PA8 -> PA4
- J4 pad 14: PA9 -> PA5
- J4 pad 15: PA10 -> PA6
- J4 pad 16: PA11 -> PA7
- J4 pad 17: PA12 -> PC4
- J4 pad 18: PA13 -> PC5
- J4 pad 19: PA14 -> PB0
- J4 pad 2: Net-(J4-Pad2) -> GND
- J4 pad 20: PA15 -> PB1
- J4 pad 21: PB0 -> PB2
- J4 pad 22: PB1 -> Net-(J4-Pad22)
- J4 pad 23: PB2 -> PB10
- J4 pad 24: PB3 -> PB11
- J4 pad 25: PB4 -> PB12
- J4 pad 26: PB5 -> PB13
- J4 pad 27: PB6 -> PB14
- J4 pad 28: PB7 -> PB15
- J4 pad 29: PB8 -> PC6
- J4 pad 3: Net-(J4-Pad3) -> BO0
- J4 pad 30: PB9 -> PC7
- J4 pad 31: PB10 -> PC8
- J4 pad 32: PB11 -> PC9
- J4 pad 33: PB12 -> Net-(J4-Pad33)
- J4 pad 34: PB13 -> Net-(J4-Pad34)
- J4 pad 35: PB14 -> Net-(J4-Pad35)
- J4 pad 36: PB15 -> Net-(J4-Pad36)
- J4 pad 39: Net-(J4-Pad39) -> +3V3
- J4 pad 4: Net-(J4-Pad4) -> NRST
- J4 pad 40: Net-(J4-Pad40) -> GND
- J4 pad 41: Net-(J4-Pad41) -> +3V3
- J4 pad 42: Net-(J4-Pad42) -> GND
- J4 pad 49: Net-(J4-Pad49) -> PA8
- J4 pad 5: PA0 -> PC0
- J4 pad 50: Net-(J4-Pad50) -> PA9
- J4 pad 51: Net-(J4-Pad51) -> PA10
- J4 pad 52: Net-(J4-Pad52) -> PA11
- J4 pad 53: Net-(J4-Pad53) -> PA12
- J4 pad 54: Net-(J4-Pad54) -> PA13
- J4 pad 55: Net-(J4-Pad55) -> PA14
- J4 pad 56: Net-(J4-Pad56) -> PA15
- J4 pad 59: Net-(J4-Pad59) -> PC10
- J4 pad 6: PA1 -> PC1
- J4 pad 60: Net-(J4-Pad60) -> PC11
- J4 pad 61: Net-(J4-Pad61) -> PC12
- J4 pad 63: Net-(J4-Pad63) -> PD2
- J4 pad 64: Net-(J4-Pad64) -> PB3
- J4 pad 65: Net-(J4-Pad65) -> PB4
- J4 pad 66: Net-(J4-Pad66) -> PB5
- J4 pad 67: Net-(J4-Pad67) -> PB6
- J4 pad 68: Net-(J4-Pad68) -> PB7
- J4 pad 69: Net-(J4-Pad69) -> PB8
- J4 pad 7: PA2 -> PC2
- J4 pad 70: Net-(J4-Pad70) -> PB9
- J4 pad 73: Net-(J4-Pad73) -> PC14
- J4 pad 74: Net-(J4-Pad74) -> PC13
- J4 pad 76: Net-(J4-Pad76) -> PC15
- J4 pad 79: Net-(J4-Pad79) -> +3V3
- J4 pad 8: PA3 -> PC3
- J4 pad 80: Net-(J4-Pad80) -> GND
- J4 pad 9: PA4 -> PA0
- R2 pad 1: BOOT0 -> BO0
- SW2 pad 1: BOOT0 -> BO0
- U1 pad 60: BOOT0 -> BO0
Routing:
- net +3V3: track 11.4 -> 225.0 mm, vias 0 -> 8
- net PC13: track 0.00 -> 45.8 mm
- net PA15: track 48.2 -> 13.7 mm
- net PC0: track 0.00 -> 30.5 mm
- net PC2: track 0.00 -> 28.4 mm
- net PC1: track 0.00 -> 26.5 mm
- net PA14: track 42.2 -> 16.8 mm
- net PC8: track 0.00 -> 24.2 mm
- net PC3: track 0.00 -> 24.0 mm
- net PC14: track 0.00 -> 23.6 mm
- net PC6: track 0.00 -> 22.3 mm
- net PC9: track 0.00 -> 22.3 mm
- net PC15: track 0.00 -> 21.7 mm
- net PB14: track 0.00 -> 21.4 mm
- net PB12: track 0.00 -> 20.8 mm
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- added copper zone on B.Cu, net +3V3
- added copper zone on F.Cu, net +3V3

Commit message: Hmmm
Parts:
- moved R2 1.91 mm to (123.2, 110.5)
Routing:
- net BO0: track 0.00 -> 63.9 mm, vias 0 -> 2
- net NRST: track 0.00 -> 40.0 mm
- net PC1: track 26.5 -> 23.7 mm
- net PC0: track 30.5 -> 27.7 mm
- net PC2: track 28.4 -> 25.6 mm
- net PB9: track 18.3 -> 15.7 mm
- net PB8: track 21.1 -> 18.4 mm
- net PC3: track 24.0 -> 21.6 mm

Commit message: Hmmmm
Parts:
- C5, C6, C7, C8: value 100nF -> C_100NF_0603; footprint Capacitor_SMD:C_0402_1005Metric -> Capacitor_SMD:C_0603_1608Metric
- U2: value XC6206P332MR -> AMS1117-3.3; footprint Package_TO_SOT_SMD:SOT-23 -> Package_TO_SOT_SMD:SOT-223-3_TabPin2
- moved C8 32.6 mm to (173.4, 90.6), turned to 0 degrees
- moved C7 23.8 mm to (173.4, 88.1)
- moved C6 11.3 mm to (169.4, 90.6)
- moved C1 5.75 mm to (182.9, 112.4), turned to 270 degrees
- moved C4 5.12 mm to (142.9, 90.2)
- moved D1 4.02 mm to (184.2, 109.2)
- moved U2 3.42 mm to (177.2, 111.8), turned to 180 degrees
- moved C3 0.90 mm to (171.4, 112.4), turned to 270 degrees
- moved C5 0.64 mm to (145.4, 95.2)
Routing:
- net +3V3: track 225.3 -> 199.0 mm
- net VBUS: track 17.2 -> 7.03 mm
- net +5V: track 7.03 -> 0.00 mm

Commit message: Hmmm
Parts:
- removed H1, H2, H3, H4: ~, MountingHole:MountingHole_3.2mm_M3
- removed J4: STM32WORLD_BASE, stm32world:STM32WORLD_BASE
- added C12: C_2.2UF_0603, Capacitor_SMD:C_0603_1608Metric, F.Cu at (160.9, 97.2)
- added J2: STM32WORLD_BASE, stm32world:STM32WORLD_BASE, F.Cu at (152.4, 101.6)
- C1, C3: value 10uF -> C_10UF_0805
- C10: value 10nF -> C_20PF_0603; footprint Capacitor_SMD:C_0402_1005Metric -> Capacitor_SMD:C_0603_1608Metric
- C11: value 20pF -> C_20PF_0603; footprint Capacitor_SMD:C_0402_1005Metric -> Capacitor_SMD:C_0603_1608Metric
- C2: value 100nF -> C_100NF_0603; footprint Capacitor_SMD:C_0402_1005Metric -> Capacitor_SMD:C_0603_1608Metric
- C4: value 1uF -> C_1UF_0603; footprint Capacitor_SMD:C_0402_1005Metric -> Capacitor_SMD:C_0603_1608Metric
- C9: value 20pF -> C_2.2UF_0603; footprint Capacitor_SMD:C_0402_1005Metric -> Capacitor_SMD:C_0603_1608Metric
- D2: value GR -> LED_GREEN_0603
- D3: value BLUE -> LED_BLUE_0603
- R1, R2: value 10k -> R_10K_0603; footprint Resistor_SMD:R_0402_1005Metric -> Resistor_SMD:R_0603_1608Metric
- R3, R4: value 5.1k -> R_5.1K_0603; footprint Resistor_SMD:R_0402_1005Metric -> Resistor_SMD:R_0603_1608Metric
- R5, R6: value 22R -> R_22_0603; footprint Resistor_SMD:R_0402_1005Metric -> Resistor_SMD:R_0603_1608Metric
- R7, R8: value 220 -> R_220_0603; footprint Resistor_SMD:R_0402_1005Metric -> Resistor_SMD:R_0603_1608Metric
- Y1: value 16 MHz -> X_16MHZ
- moved C7 37.4 mm to (141.0, 106.7), turned to 180 degrees
- moved C10 32.2 mm to (140.9, 97.1), turned to 0 degrees
- moved C8 31.4 mm to (148.6, 109.9), turned to 180 degrees
- moved C4 24.4 mm to (158.1, 109.2), turned to 0 degrees
- moved C9 22.1 mm to (158.1, 111.1)
- moved C6 9.68 mm to (160.9, 95.2)
- moved R7 3.24 mm to (120.0, 89.5)
- moved D2 3.17 mm to (116.8, 89.5)
- moved C2 2.54 mm to (123.2, 114.9)
- moved R1 2.54 mm to (123.2, 117.5)
- moved R8 2.01 mm to (120.0, 91.4)
- moved D3 1.91 mm to (116.8, 91.4)
- moved R4 1.42 mm to (178.4, 99.1), turned to 0 degrees
- moved R3 0.90 mm to (178.4, 104.8), turned to 0 degrees
- moved R6 0.90 mm to (178.4, 101.0), turned to 0 degrees
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- renumbered J3 to J1, U2 to U1, U1 to U2
Connections:
- C10 pad 1: +3V3 -> Net-(C10-Pad1)
- J1 pad A5: Net-(J3-PadA5) -> Net-(J1-PadA5)
- J1 pad A6: Net-(J3-PadA6) -> Net-(J1-PadA6)
- J1 pad A7: Net-(J3-PadA7) -> Net-(J1-PadA7)
- J1 pad B5: Net-(J3-PadB5) -> Net-(J1-PadB5)
- J1 pad B6: Net-(J3-PadA6) -> Net-(J1-PadA6)
- J1 pad B7: Net-(J3-PadA7) -> Net-(J1-PadA7)
- R3 pad 1: Net-(J3-PadA5) -> UCC
- R3 pad 2: UCC -> Net-(J1-PadA5)
- R4 pad 1: Net-(J3-PadB5) -> UCC
- R4 pad 2: UCC -> Net-(J1-PadB5)
- R5 pad 1: Net-(J3-PadA7) -> PA11
- R5 pad 2: PA11 -> Net-(J1-PadA7)
- R6 pad 1: Net-(J3-PadA6) -> PA12
- R6 pad 2: PA12 -> Net-(J1-PadA6)
- U2 pad 31: VCAP_1 -> Net-(C9-Pad1)
- U2 pad 47: VCAP_2 -> Net-(C12-Pad1)
- U2 pad 5: Net-(C9-Pad1) -> Net-(C10-Pad1)
- Y1 pad 1: Net-(C9-Pad1) -> Net-(C10-Pad1)
Routing:
- net +3V3: track 199.0 -> 275.6 mm, vias 8 -> 13
- net +5V: track 0.00 -> 62.0 mm
- net Net-(J3-PadA7): track 11.1 -> 0.00 mm
- net Net-(C10-Pad1): track 0.00 -> 9.38 mm
- net PC13: track 45.8 -> 37.8 mm, vias 0 -> 1
- net Net-(J3-PadA6): track 6.59 -> 0.00 mm
- net VBUS: track 7.03 -> 13.6 mm
- net Net-(J1-PadA7): track 0.00 -> 6.48 mm
- net UCC: track 0.00 -> 6.27 mm
- net Net-(J3-PadA5): track 5.40 -> 0.00 mm
- net Net-(J1-PadA6): track 0.00 -> 5.36 mm
- net Net-(J3-PadB5): track 5.19 -> 0.00 mm
- net Net-(C9-Pad1): track 9.38 -> 4.55 mm
- net Net-(J1-PadA5): track 0.00 -> 4.18 mm
- net Net-(J1-PadB5): track 0.00 -> 3.71 mm
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