File: ioaw9523/ioaw9523.sch (KiCad schematic (older format))
At the start: 6 parts, among them U1 AW9523B

Commit message: Hmmm
Parts:
- added JP1, JP3: ~, Jumper:SolderJumper-2_P1.3mm_Bridged2Bar_Pad1.0x1.5mm, symbol Jumper:Jumper_2_Bridged
- added JP2, JP4, JP7, JP8: ~, Jumper:SolderJumper-2_P1.3mm_Open_Pad1.0x1.5mm, symbol Jumper:Jumper_2_Open
- added JP5, JP6: ~, Jumper:SolderJumper-3_P1.3mm_Bridged12_Pad1.0x1.5mm, symbol Jumper:SolderJumper_3_Bridged12
- U1: symbol stm32world:AW9523B -> ioaw9523-rescue:AW9523B-stm32world
Connections:
- net labels added: AD0, AD1, I2C1_SCL, I2C1_SCL_ALT, I2C1_SDA, I2C1_SDA_ALT, I2C2_SCL, I2C2_SDA, INTN, RSTN, SCL, SDA
- wire segments 77 -> 113

Commit message: Hmmmm
Connections:
- wire segments 113 -> 114
Other:
- moved on the sheet: U1
