File: ioaw9523/ioaw9523.kicad_pcb (KiCad board)
At the start: 2 copper layers, 76.2 x 50.8 mm, 6 parts, among them U1 AW9523B

Commit message: Hmmm
Parts:
- added JP1: ~, Jumper:SolderJumper-2_P1.3mm_Bridged2Bar_Pad1.0x1.5mm, F.Cu at (124.5, 99.1)
- added JP2: ~, Jumper:SolderJumper-2_P1.3mm_Open_Pad1.0x1.5mm, F.Cu at (124.5, 101.6)
- added JP3: ~, Jumper:SolderJumper-2_P1.3mm_Bridged2Bar_Pad1.0x1.5mm, F.Cu at (133.3, 99.1)
- added JP4: ~, Jumper:SolderJumper-2_P1.3mm_Open_Pad1.0x1.5mm, F.Cu at (133.3, 101.6)
- added JP5: ~, Jumper:SolderJumper-3_P1.3mm_Bridged12_Pad1.0x1.5mm, F.Cu at (163.8, 91.4)
- added JP6: ~, Jumper:SolderJumper-3_P1.3mm_Bridged12_Pad1.0x1.5mm, F.Cu at (163.8, 94.0)
- added JP7: ~, Jumper:SolderJumper-2_P1.3mm_Open_Pad1.0x1.5mm, F.Cu at (124.5, 104.1)
- added JP8: ~, Jumper:SolderJumper-2_P1.3mm_Open_Pad1.0x1.5mm, F.Cu at (133.3, 104.1)
- moved R1 1.91 mm to (163.2, 99.7)
- moved R2 1.91 mm to (161.3, 99.7)
Connections:
- net Net-(U1-Pad22) renamed INTN
- net Net-(U1-Pad23) renamed RSTN
- J1 pad 23: Net-(J1-Pad23) -> I2C2_SCL
- J1 pad 24: Net-(J1-Pad24) -> I2C2_SDA
- J1 pad 67: Net-(J1-Pad67) -> I2C1_SCL
- J1 pad 68: Net-(J1-Pad68) -> I2C1_SDA
- J1 pad 69: Net-(J1-Pad69) -> I2C1_SCL_ALT
- J1 pad 70: Net-(J1-Pad70) -> I2C1_SDA_ALT
- R1 pad 2: Net-(R1-Pad2) -> SCL
- R2 pad 2: Net-(R2-Pad2) -> SDA
- U1 pad 18: Net-(U1-Pad18) -> AD0
- U1 pad 19: Net-(R2-Pad2) -> SCL
- U1 pad 20: Net-(R1-Pad2) -> SDA
- U1 pad 24: Net-(U1-Pad24) -> AD1
Routing:
- net SCL: track 0.00 -> 46.5 mm
- net SDA: track 0.00 -> 36.7 mm
- net I2C2_SCL: track 0.00 -> 28.7 mm
- net I2C1_SCL_ALT: track 0.00 -> 26.0 mm, vias 0 -> 1
- net I2C1_SCL: track 0.00 -> 23.4 mm, vias 0 -> 1
- net I2C2_SDA: track 0.00 -> 22.7 mm
- net I2C1_SDA_ALT: track 0.00 -> 20.4 mm, vias 0 -> 1
- net AD0: track 0.00 -> 19.1 mm
- net I2C1_SDA: track 0.00 -> 16.8 mm, vias 0 -> 1
- net AD1: track 0.00 -> 13.0 mm, vias 0 -> 2
- net +3V3: track 175.8 -> 182.0 mm
- net Net-(R1-Pad2): track 4.28 -> 0.00 mm
- net Net-(R2-Pad2): track 2.33 -> 0.00 mm
- net GND: vias 0 -> 5
Other:
- board text added: "I2C Port"
- board text added: "I2C1"
- board text added: "I2C1_ALT"
- board text added: "I2C2"
- board text added: "PB10"
- board text added: "PB11"
- board text added: "PB6"
- board text added: "PB7"
- board text added: "PB8"
- board text added: "PB9"
- board text added: "SCL"
- board text added: "SDA"

Commit message: Hmmm
Routing:
- net AD0: track 19.1 -> 16.7 mm
- net GND: vias 5 -> 6

Commit message: Hmmm
Parts:
- U1: footprint Package_DFN_QFN:TQFN-24-1EP_4x4mm_P0.5mm_EP2.8x2.8mm_PullBack_ThermalVias -> Package_DFN_QFN:TQFN-24-1EP_4x4mm_P0.5mm_EP2.8x2.8mm_PullBack
Connections:
- J1 pad 10: Net-(J1-Pad10) -> unconnected-(J1-Pad10)
- J1 pad 11: Net-(J1-Pad11) -> unconnected-(J1-Pad11)
- J1 pad 12: Net-(J1-Pad12) -> unconnected-(J1-Pad12)
- J1 pad 13: Net-(J1-Pad13) -> unconnected-(J1-Pad13)
- J1 pad 14: Net-(J1-Pad14) -> unconnected-(J1-Pad14)
- J1 pad 15: Net-(J1-Pad15) -> unconnected-(J1-Pad15)
- J1 pad 16: Net-(J1-Pad16) -> unconnected-(J1-Pad16)
- J1 pad 17: Net-(J1-Pad17) -> unconnected-(J1-Pad17)
- J1 pad 18: Net-(J1-Pad18) -> unconnected-(J1-Pad18)
- J1 pad 19: Net-(J1-Pad19) -> unconnected-(J1-Pad19)
- J1 pad 20: Net-(J1-Pad20) -> unconnected-(J1-Pad20)
- J1 pad 21: Net-(J1-Pad21) -> unconnected-(J1-Pad21)
- J1 pad 22: Net-(J1-Pad22) -> unconnected-(J1-Pad22)
- J1 pad 25: Net-(J1-Pad25) -> unconnected-(J1-Pad25)
- J1 pad 26: Net-(J1-Pad26) -> unconnected-(J1-Pad26)
- J1 pad 27: Net-(J1-Pad27) -> unconnected-(J1-Pad27)
- J1 pad 28: Net-(J1-Pad28) -> unconnected-(J1-Pad28)
- J1 pad 29: Net-(J1-Pad29) -> unconnected-(J1-Pad29)
- J1 pad 3: Net-(J1-Pad3) -> unconnected-(J1-Pad3)
- J1 pad 30: Net-(J1-Pad30) -> unconnected-(J1-Pad30)
- J1 pad 31: Net-(J1-Pad31) -> unconnected-(J1-Pad31)
- J1 pad 32: Net-(J1-Pad32) -> unconnected-(J1-Pad32)
- J1 pad 33: Net-(J1-Pad33) -> unconnected-(J1-Pad33)
- J1 pad 34: Net-(J1-Pad34) -> unconnected-(J1-Pad34)
- J1 pad 35: Net-(J1-Pad35) -> unconnected-(J1-Pad35)
- J1 pad 36: Net-(J1-Pad36) -> unconnected-(J1-Pad36)
- J1 pad 39: Net-(J1-Pad39) -> unconnected-(J1-Pad39)
- J1 pad 4: Net-(J1-Pad4) -> unconnected-(J1-Pad4)
- J1 pad 41: Net-(J1-Pad41) -> unconnected-(J1-Pad41)
- J1 pad 45: Net-(J1-Pad45) -> unconnected-(J1-Pad45)
- J1 pad 46: Net-(J1-Pad46) -> unconnected-(J1-Pad46)
- J1 pad 47: Net-(J1-Pad47) -> unconnected-(J1-Pad47)
- J1 pad 48: Net-(J1-Pad48) -> unconnected-(J1-Pad48)
- J1 pad 49: Net-(J1-Pad49) -> unconnected-(J1-Pad49)
- J1 pad 5: Net-(J1-Pad5) -> unconnected-(J1-Pad5)
- J1 pad 50: Net-(J1-Pad50) -> unconnected-(J1-Pad50)
- J1 pad 51: Net-(J1-Pad51) -> unconnected-(J1-Pad51)
- J1 pad 52: Net-(J1-Pad52) -> unconnected-(J1-Pad52)
- J1 pad 53: Net-(J1-Pad53) -> unconnected-(J1-Pad53)
- J1 pad 54: Net-(J1-Pad54) -> unconnected-(J1-Pad54)
- J1 pad 55: Net-(J1-Pad55) -> unconnected-(J1-Pad55)
- J1 pad 56: Net-(J1-Pad56) -> unconnected-(J1-Pad56)
- J1 pad 57: Net-(J1-Pad57) -> unconnected-(J1-Pad57)
- J1 pad 58: Net-(J1-Pad58) -> unconnected-(J1-Pad58)
- J1 pad 59: Net-(J1-Pad59) -> unconnected-(J1-Pad59)
- J1 pad 6: Net-(J1-Pad6) -> unconnected-(J1-Pad6)
- J1 pad 60: Net-(J1-Pad60) -> unconnected-(J1-Pad60)
- J1 pad 61: Net-(J1-Pad61) -> unconnected-(J1-Pad61)
- J1 pad 62: Net-(J1-Pad62) -> unconnected-(J1-Pad62)
- J1 pad 63: Net-(J1-Pad63) -> unconnected-(J1-Pad63)
- J1 pad 64: Net-(J1-Pad64) -> unconnected-(J1-Pad64)
- J1 pad 65: Net-(J1-Pad65) -> unconnected-(J1-Pad65)
- J1 pad 66: Net-(J1-Pad66) -> unconnected-(J1-Pad66)
- J1 pad 7: Net-(J1-Pad7) -> unconnected-(J1-Pad7)
- J1 pad 71: Net-(J1-Pad71) -> unconnected-(J1-Pad71)
- J1 pad 72: Net-(J1-Pad72) -> unconnected-(J1-Pad72)
- J1 pad 73: Net-(J1-Pad73) -> unconnected-(J1-Pad73)
- J1 pad 74: Net-(J1-Pad74) -> unconnected-(J1-Pad74)
- J1 pad 75: Net-(J1-Pad75) -> unconnected-(J1-Pad75)
- J1 pad 76: Net-(J1-Pad76) -> unconnected-(J1-Pad76)
- J1 pad 77: Net-(J1-Pad77) -> unconnected-(J1-Pad77)
- J1 pad 78: Net-(J1-Pad78) -> unconnected-(J1-Pad78)
- J1 pad 8: Net-(J1-Pad8) -> unconnected-(J1-Pad8)
- J1 pad 9: Net-(J1-Pad9) -> unconnected-(J1-Pad9)
Routing:
- net GND: vias 6 -> 7
Other:
- net class Default removed
