File: mcustm32g030/mcustm32g030.kicad_pcb (KiCad board)
At the start: 2 copper layers, 21 parts, among them J1 STM32WORLD_BASE, U2 STM32G030C6

Commit message: Hmmmm
Parts:
- added JP1: Jumper_2_Bridged, Jumper:SolderJumper-2_P1.3mm_Bridged2Bar_Pad1.0x1.5mm, F.Cu at (104.1, 104.8)
- C1, C7: value ~ -> 10uF
- C2: value ~ -> 1uF
- C3, C4, C5, C6: value ~ -> 100nF
- C8, C9: value ~ -> 20pF
- D1: value ~ -> GR
- D2: value ~ -> BL
- R1, R4: value ~ -> 10k
- R2, R3: value ~ -> 220R
- U1: value ~ -> AMS1117-3.3
- Y1: value ~ -> X_16MHZ
- moved R4 78.7 mm to (100.3, 109.2)
- moved D2 76.6 mm to (94.5, 85.1)
- moved R1 74.3 mm to (100.3, 103.5), turned to 180 degrees
- moved R2 72.3 mm to (100.3, 81.9)
- moved D1 70.7 mm to (95.2, 81.3)
- moved C3 69.3 mm to (100.3, 105.4)
- moved R3 67.1 mm to (101.2, 86.4)
- moved C6 59.8 mm to (118.7, 90.2), turned to 90 degrees
- moved C5 58.0 mm to (116.8, 90.2), turned to 90 degrees
- moved C9 55.2 mm to (116.8, 99.7), turned to 180 degrees
- moved C4 52.5 mm to (114.9, 90.2), turned to 90 degrees
- moved C8 51.8 mm to (116.8, 93.3)
- moved C2 19.7 mm to (150.5, 97.8), turned to 90 degrees
- moved C1 12.1 mm to (161.9, 101.6), turned to 90 degrees
- moved C7 2.62 mm to (150.5, 101.6), turned to -90 degrees
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Connections:
- J1 pad 1: unconnected-(J1-Pad1) -> +3V3
- J1 pad 2: unconnected-(J1-Pad2) -> GND
- J1 pad 29: unconnected-(J1-Pad29) -> PC6
- J1 pad 3: unconnected-(J1-Pad3) -> BO0
- J1 pad 30: unconnected-(J1-Pad30) -> PC7
- J1 pad 37: unconnected-(J1-Pad37) -> +3V3
- J1 pad 38: unconnected-(J1-Pad38) -> GND
- J1 pad 39: unconnected-(J1-Pad39) -> +5V
- J1 pad 4: unconnected-(J1-Pad4) -> NRST
- J1 pad 40: unconnected-(J1-Pad40) -> GND
- J1 pad 41: unconnected-(J1-Pad41) -> +5V
- J1 pad 42: unconnected-(J1-Pad42) -> GND
- J1 pad 43: unconnected-(J1-Pad43) -> +3V3
- J1 pad 44: unconnected-(J1-Pad44) -> GND
- J1 pad 63: unconnected-(J1-Pad63) -> PD2
- J1 pad 73: unconnected-(J1-Pad73) -> PC14
- J1 pad 74: unconnected-(J1-Pad74) -> PC13
- J1 pad 76: unconnected-(J1-Pad76) -> PC15
- J1 pad 79: unconnected-(J1-Pad79) -> +3V3
- J1 pad 80: unconnected-(J1-Pad80) -> GND
- U2 pad 38: PD0 -> unconnected-(U2-Pad38)
- U2 pad 39: PD1 -> unconnected-(U2-Pad39)
- U2 pad 41: PD3 -> unconnected-(U2-Pad41)
- U2 pad 5: unconnected-(U2-Pad5) -> +3V3
Routing:
- net +3V3: track 0.00 -> 95.3 mm, vias 0 -> 13
- net +5V: track 0.00 -> 56.7 mm
- net PA8: track 0.00 -> 26.9 mm, vias 0 -> 1
- net PA10: track 0.00 -> 26.3 mm
- net PC15: track 0.00 -> 25.6 mm
- net PA9: track 0.00 -> 25.4 mm, vias 0 -> 1
- net PC14: track 0.00 -> 25.4 mm
- net PC6: track 0.00 -> 25.0 mm
- net PA0: track 0.00 -> 23.5 mm
- net PC7: track 0.00 -> 23.0 mm
- net PA11: track 0.00 -> 21.9 mm
- net PA12: track 0.00 -> 21.9 mm
- net PA2: track 0.00 -> 20.7 mm
- net PB14: track 0.00 -> 20.4 mm
- net PC13: track 0.00 -> 20.4 mm
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- added copper zone on B.Cu, net +3V3
- added copper zone on F.Cu, net +3V3
- added copper zone on B.Cu, net GND
- added copper zone on F.Cu, net GND
Other:
- board outline added: 76.2 x 50.8 mm

Commit message: Almost there
Parts:
- moved R3 5.01 mm to (96.5, 84.5)
- moved R2 3.86 mm to (96.5, 82.5)
- moved D1 2.29 mm to (93.3, 82.5), turned to 180 degrees
- moved D2 1.29 mm to (93.3, 84.5), turned to 180 degrees
Routing:
- net +3V3: track 95.3 -> 224.8 mm
- net NRST: track 0.00 -> 41.8 mm
- net PA14: track 19.4 -> 55.9 mm, vias 0 -> 2
- net BO0: track 0.00 -> 11.7 mm
- net PB14: track 20.4 -> 23.0 mm
- net PC15: track 25.6 -> 23.3 mm
- net PB15: track 18.4 -> 20.3 mm
- net PC6: track 25.0 -> 26.7 mm
- net PC7: track 23.0 -> 24.3 mm
- net PA0: track 23.5 -> 24.2 mm
- net PC13: track 20.4 -> 21.1 mm
- net GND: vias 11 -> 12

Commit message: Hmmm
Parts:
- moved JP1 10.6 mm to (98.4, 113.7)
Routing:
- net PC13: track 21.1 -> 45.6 mm
- net +3V3: track 224.8 -> 242.8 mm
- net PA14: track 55.9 -> 67.9 mm
- net BO0: track 11.7 -> 17.0 mm
- net PA2: track 20.7 -> 24.4 mm
- net PA3: track 17.4 -> 20.2 mm
- net PA4: track 20.0 -> 22.6 mm
- net NRST: track 41.8 -> 44.2 mm
- net PA5: track 16.8 -> 18.8 mm
- net PA6: track 19.4 -> 21.1 mm
- net Net-(D2-Pad1): track 0.00 -> 1.56 mm
- net Net-(D1-Pad1): track 0.00 -> 1.56 mm
- net PA7: track 16.1 -> 17.3 mm
- net PA1: track 19.1 -> 19.6 mm
- net GND: vias 12 -> 37
