File: mcustm32g030/mcustm32g030.kicad_sch (KiCad schematic)
At the start: 1 part

Commit message: Hmmmm
Parts:
- added C? (x4): ~, symbol stm32world:C_100NF_0603
- added C? (x2): ~, symbol stm32world:C_10UF_0805
- added C? (x2): ~, symbol stm32world:C_20PF_0603
- added C?: ~, symbol stm32world:C_1UF_0603
- added D?: ~, symbol stm32world:LED_BLUE_0603
- added D?: ~, symbol stm32world:LED_GREEN_0603
- added R? (x2): ~, symbol stm32world:R_10K_0603
- added R? (x2): ~, symbol stm32world:R_220_0603
- added SW? (x2): ~, symbol stm32world:TS-1088R-02526
- added U?: ~, symbol stm32world:AMS1117-3.3
- added U?: (no value), symbol stm32world:STM32G030C6
- added Y?: ~, symbol stm32world:X_16MHZ
- J?: value (none) -> STM32WORLD_BASE; footprint (none) -> stm32world:STM32WORLD_BASE
Connections:
- new net: D?.1 (K), R?.1 (x2)
- new net: C?.1, U?.9 (OSC_OUT), Y?.3
- new net: C?.1, U?.8 (OSC_IN), Y?.1
- new net +3V3: C?.1, C?.1, C?.1, C?.1, C?.1, D?.2 (A), D?.2 (A), R?.1, SW?.2, U?.2 (VO), U?.4 (VBAT), U?.6 (VDD)
- new net +5V: C?.1, U?.3 (VI)
- new net BO0: R?.1, SW?.1
- new net GND: C?.2, C?.2, C?.2, C?.2, C?.2, C?.2, C?.2, C?.2, C?.2, R?.2, R?.2, SW?.1, U?.1 (GND), U?.7 (GND), Y?.2, Y?.4
- new net NRST: C?.1, R?.2, SW?.2
- new net PC13: R?.2
Other:
- note added: "Internal pull-up"

Commit message: Hmmmm
Parts:
- C1, C2, C3, C4, C5, C6, C7, C8, C9: renamed from C?; value ~ -> (none)
- D1, D2: renamed from D?; value ~ -> (none)
- J1: renamed from J?; value STM32WORLD_BASE -> (none); footprint stm32world:STM32WORLD_BASE -> (none)
- R1, R2, R3, R4: renamed from R?; value ~ -> (none)
- SW1, SW2: renamed from SW?; value ~ -> (none)
- U1: renamed from U?; value ~ -> (none)
- Y1: renamed from Y?; value ~ -> (none)
- gave numbers to parts that had none: 1
Connections:
- net NRST: now also U2.10 (NRST)
- net PA0: now also J1.9 (PA0), U2.11 (PA0)
- net PA1: now also J1.10 (PA1), U2.12 (PA1)
- net PA10: now also J1.51 (PA10), U2.32 (PA10)
- net PA11: now also J1.52 (PA11), U2.33 (PA11)
- net PA12: now also J1.53 (PA12), U2.34 (PA12)
- net PA13: now also J1.54 (PA13), U2.35 (PA13)
- net PA14: now also J1.55 (PA14), U2.36 (PA14_(BO0))
- net PA15: now also J1.56 (PA15), U2.37 (PA15)
- net PA2: now also J1.11 (PA2), U2.13 (PA2)
- net PA3: now also J1.12 (PA3), U2.14 (PA3)
- net PA4: now also J1.13 (PA4), U2.15 (PA4)
- net PA5: now also J1.14 (PA5), U2.16 (PA5)
- net PA6: now also J1.15 (PA6), U2.17 (PA6)
- net PA7: now also J1.16 (PA7), U2.18 (PA7)
- net PA8: now also J1.49 (PA8), U2.28 (PA8)
- net PA9: now also J1.50 (PA9), U2.29 (PA9)
- net PB0: now also J1.19 (PB0), U2.19 (PB0)
- net PB1: now also J1.20 (PB1), U2.20 (PB1)
- net PB10: now also J1.23 (PB10), U2.22 (PB10)
- net PB11: now also J1.24 (PB11), U2.23 (PB11)
- net PB12: now also J1.25 (PB12), U2.24 (PB12)
- net PB13: now also J1.26 (PB13), U2.25 (PB13)
- net PB14: now also J1.27 (PB14), U2.26 (PB14)
- net PB15: now also J1.28 (PB15), U2.27 (PB15)
- net PB2: now also J1.21 (PB2), U2.21 (PB2)
- net PB3: now also J1.64 (PB3), U2.42 (PB3)
- net PB4: now also J1.65 (PB4), U2.43 (PB4)
- net PB5: now also J1.66 (PB5), U2.44 (PB5)
- net PB6: now also J1.67 (PB6), U2.45 (PB6)
- net PB7: now also J1.68 (PB7), U2.46 (PB7)
- net PB8: now also J1.69 (PB8), U2.47 (PB8)
- net PB9: now also J1.70 (PB9), U2.48 (PB9)
- net PC13: now also U2.1 (PC13)
- net PC14: now also U2.2 (PC14)
- net PC15: now also U2.3 (PC15)
- net PC6: now also U2.30 (PC6)
- net PC7: now also U2.31 (PC7)
- net PD0: now also U2.38 (PD0)
- net PD1: now also U2.39 (PD1)
- net PD2: now also U2.40 (PD2)
- net PD3: now also U2.41 (PD3)
Other:
- note removed: "Internal pull-up"
- company: (none) -> ${COMPANY}
- title: (none) -> ${TITLE}

Commit message: Hmmmm
Parts:
- added JP1: (no value), symbol Jumper:Jumper_2_Bridged
- C1, C7: value (none) -> 10uF; footprint (none) -> Capacitor_SMD:C_0805_2012Metric
- C2: value (none) -> 1uF; footprint (none) -> Capacitor_SMD:C_0603_1608Metric
- C3, C4, C5, C6: value (none) -> 100nF; footprint (none) -> Capacitor_SMD:C_0603_1608Metric
- C8, C9: value (none) -> 20pF; footprint (none) -> Capacitor_SMD:C_0603_1608Metric
- D1: value (none) -> GR; footprint (none) -> LED_SMD:LED_0603_1608Metric
- D2: value (none) -> BL; footprint (none) -> LED_SMD:LED_0603_1608Metric
- J1: value (none) -> STM32WORLD_BASE; footprint (none) -> stm32world:STM32WORLD_BASE
- R1, R4: value (none) -> 10k; footprint (none) -> Resistor_SMD:R_0603_1608Metric
- R2, R3: value (none) -> 220R; footprint (none) -> Resistor_SMD:R_0603_1608Metric
- SW1, SW2: value (none) -> ~; footprint (none) -> stm32world:TS-1088R-02526
- U1: value (none) -> AMS1117-3.3; footprint (none) -> Package_TO_SOT_SMD:SOT-223-3_TabPin2
- U2: value (none) -> STM32G030C6; footprint (none) -> Package_QFP:LQFP-48_7x7mm_P0.5mm
- Y1: value (none) -> X_16MHZ; footprint (none) -> Crystal:Crystal_SMD_3225-4Pin_3.2x2.5mm
Connections:
- net +3V3: now also J1.1 (3.3V), J1.37 (3.3V), J1.43 (3.3V), J1.79 (3.3V), U2.5 (VREF+)
- net +5V: now also J1.39 (5V), J1.41 (5V)
- net BO0: now also J1.3 (BO0), JP1.1 (A)
- net GND: now also J1.2 (GND), J1.38 (GND), J1.40 (GND), J1.42 (GND), J1.44 (GND), J1.80 (GND)
- net NRST: now also J1.4 (NRST)
- net PA14: now also JP1.2 (B)
- net PC13: now also J1.74 (PC13)
- net PC14: now also J1.73 (PC14)
- net PC15: now also J1.76 (PC15)
- net PC6: now also J1.29 (PC6)
- net PC7: now also J1.30 (PC7)
- net PD2: now also J1.63 (PD2)
- net PD0: no longer names the net of U2.38 (PD0)
- net PD1: no longer names the net of U2.39 (PD1)
- net PD3: no longer names the net of U2.41 (PD3)
- no-connect marks 0 -> 31
Other:
- moved on the sheet: C8, C9, U2, Y1

Commit message: Hmmm
Parts:
- J1: value STM32WORLD_BASE -> (none)
- JP1: value (none) -> Jumper_2_Bridged; footprint (none) -> Jumper:SolderJumper-2_P1.3mm_Bridged2Bar_Pad1.0x1.5mm
Other:
- moved on the sheet: C3, D1, D2, J1, JP1, R1, R2, R3, R4, SW1, SW2
