File: mcucn32v307/mcucn32v307.kicad_pcb (KiCad board)
At the start: 2 copper layers, 76.2 x 50.8 mm, 29 parts, among them J1 USB_C_Receptacle_USB2.0, J2 STM32WORLD_BASE, SW1 TS-1088R-02526, SW2 TS-1088R-02526, U1 AMS1117-3.3, U2 SRV05-4, U3 CH32V307, Y1 X_16MHZ

Commit message: Hmmmm
Parts:
- moved U1 5.99 mm to (176.5, 111.1), turned to 90 degrees
- moved D2 3.70 mm to (183.5, 109.9)
- moved C4 3.42 mm to (171.4, 109.9), turned to 90 degrees
- moved C10 3.18 mm to (140.3, 104.1)
- moved C9 3.18 mm to (140.3, 96.5)
- moved Y1 3.18 mm to (140.3, 100.3)
- moved C3 2.62 mm to (171.4, 113.7), turned to -90 degrees
- moved C7 2.29 mm to (146.7, 108.0), turned to 180 degrees
- moved C5 2.06 mm to (145.4, 96.5), turned to 180 degrees
- moved C1 1.91 mm to (181.6, 113.7), turned to -90 degrees
- moved C8 1.90 mm to (158.1, 108.0)
- moved U2 1.80 mm to (186.1, 92.1)
- moved C6 1.42 mm to (159.4, 96.5)
Routing:
- net +3V3: track 0.00 -> 60.1 mm, vias 0 -> 10
- net PA11: track 0.00 -> 38.0 mm, vias 0 -> 1
- net PA12: track 4.15 -> 39.1 mm, vias 0 -> 1
- net PC14: track 0.00 -> 30.5 mm
- net PA8: track 0.00 -> 29.1 mm, vias 0 -> 1
- net PA10: track 0.00 -> 25.7 mm, vias 0 -> 1
- net PA9: track 0.00 -> 24.4 mm, vias 0 -> 1
- net PC13: track 0.00 -> 20.0 mm
- net VBUS: track 0.00 -> 19.0 mm
- net PB8: track 0.00 -> 18.4 mm
- net PB6: track 0.00 -> 18.0 mm
- net PB0: track 0.00 -> 16.7 mm
- net PB2: track 0.00 -> 15.8 mm
- net PB9: track 0.00 -> 15.7 mm
- net PB10: track 0.00 -> 15.3 mm
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- added copper zone on B.Cu, net +3V3
- added copper zone on F.Cu, net +3V3
