File: prgstl/prgstl.kicad_pcb (KiCad board)
At the start: 2 copper layers, 76.2 x 50.8 mm, 49 parts, among them J2 STM32WORLD_BASE, Q1 S9013, U1 AMS1117-3.3, U2 STM32F103CBTx, U3 SRV05-4, Y1 X_8MHZ

Commit message: Hmmm
Parts:
- turned D2 to 180 degrees
Routing:
- net LED: track 53.5 -> 58.4 mm
- net Net-(D2-Pad2): track 1.56 -> 3.75 mm
Changed lines of the file:
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@@
   )
   (footprint "LED_SMD:LED_0603_1608Metric" (layer "F.Cu")
-    (at 118.11 93.345)
+    (at 118.11 93.345 180)
     (descr "LED SMD 0603 (1608 Metric), square (rectangular) end terminal, IPC_7351 nominal, (Body size source: http://www.tortai-tech.com/upload/download/2011102023233369053.pdf), generated with kicad-footprint-generator")
     (tags "LED")
@@
     (property "Sheetname" "")
     (attr smd)
-    (fp_text reference "D2" (at -2.54 0 180) (layer "F.SilkS")
+    (fp_text reference "D2" (at 2.54 0) (layer "F.SilkS")
       (effects (font (size 1 1) (thickness 0.15)))
     )
@@
     (fp_line (start -0.8 -0.1) (end -0.8 0.4) (layer "F.Fab") (width 0.1))
     (fp_line (start -0.8 0.4) (end 0.8 0.4) (layer "F.Fab") (width 0.1))
-    (pad "1" smd roundrect (at -0.7875 0) (size 0.875 0.95) (layers "F.Cu" "F.Paste" "F.Mask") (roundrect_rratio 0.25)
+    (pad "1" smd roundrect (at -0.7875 0 180) (size 0.875 0.95) (layers "F.Cu" "F.Paste" "F.Mask") (roundrect_rratio 0.25)
       (net 27 "LED") (pinfunction "K") (pintype "passive"))
-    (pad "2" smd roundrect (at 0.7875 0) (size 0.875 0.95) (layers "F.Cu" "F.Paste" "F.Mask") (roundrect_rratio 0.25)
+    (pad "2" smd roundrect (at 0.7875 0 180) (size 0.875 0.95) (layers "F.Cu" "F.Paste" "F.Mask") (roundrect_rratio 0.25)
       (net 113 "Net-(D2-Pad2)") (pinfunction "A") (pintype "passive"))
     (model "${KICAD6_3DMODEL_DIR}/LED_SMD.3dshapes/LED_0603_1608Metric.wrl"
@@
   (segment (start 156.635 97.4375) (end 156.635 96.45) (width 0.2286) (layer "F.Cu") (net 1))
   (segment (start 154.462916 102.85) (end 155.2225 102.85) (width 0.2286) (layer "F.Cu") (net 1))
+  (segment (start 120.852624 90.69829) (end 121.44378 91.289446) (width 0.2286) (layer "F.Cu") (net 1))
   (segment (start 162.135 105.7625) (end 162.135 106.75) (width 0.2286) (layer "F.Cu") (net 1))
   (segment (start 163.5475 98.85) (end 163.5475 95.6725) (width 0.2286) (layer "F.Cu") (net 1))
+  (segment (start 117.3225 89.535) (end 118.48579 90.69829) (width 0.2286) (layer "F.Cu") (net 1))
   (segment (start 117.3225 87.79) (end 123.8325 81.28) (width 0.2286) (layer "F.Cu") (net 1))
   (segment (start 162.135 106.75) (end 163.195 107.81) (width 0.2286) (layer "F.Cu") (net 1))
-  (segment (start 121.44378 91.289446) (end 121.44378 92.67878) (width 0.2286) (layer "F.Cu") (net 1))
   (segment (start 162.135 98.85) (end 163.5475 98.85) (width 0.2286) (layer "F.Cu") (net 1))
   (segment (start 158.75 100.965) (end 156.635 98.85) (width 0.2286) (layer "F.Cu") (net 1))
-  (segment (start 118.48579 90.69829) (end 117.3225 89.535) (width 0.2286) (layer "F.Cu") (net 1))
   (segment (start 158.75 100.965) (end 160.02 100.965) (width 0.4572) (layer "F.Cu") (net 1))
   (segment (start 171.45 112.08) (end 173.695 112.08) (width 0.4572) (layer "F.Cu") (net 1))
-  (segment (start 118.48579 90.69829) (end 120.852624 90.69829) (width 0.2286) (layer "F.Cu") (net 1))
   (segment (start 183.8175 92.075) (end 182.245 92.075) (width 0.4572) (layer "F.Cu") (net 1))
   (segment (start 128.27 81.28) (end 123.8325 81.28) (width 0.2286) (layer "F.Cu") (net 1))
   (segment (start 160.02 102.235) (end 158.75 102.235) (width 0.4572) (layer "F.Cu") (net 1))
   (segment (start 162.135 104.35) (end 162.135 105.7625) (width 0.2286) (layer "F.Cu") (net 1))
+  (segment (start 121.44378 91.289446) (end 121.44378 92.330657) (width 0.2286) (layer "F.Cu") (net 1))
+  (segment (start 121.44378 92.330657) (end 122.11 92.996877) (width 0.2286) (layer "F.Cu") (net 1))
   (segment (start 156.635 98.85) (end 156.635 97.4375) (width 0.2286) (layer "F.Cu") (net 1))
   (segment (start 177.1705 102.108) (end 178.2064 102.108) (width 0.381) (layer "F.Cu") (net 1))
   (segment (start 150.165 109.41) (end 151.765 107.81) (width 0.2286) (layer "F.Cu") (net 1))
+  (segment (start 118.48579 90.69829) (end 120.852624 90.69829) (width 0.2286) (layer "F.Cu") (net 1))
   (segment (start 169.545 112.255) (end 171.275 112.255) (width 0.2286) (layer "F.Cu") (net 1))
-  (segment (start 120.852624 90.69829) (end 121.44378 91.289446) (width 0.2286) (layer "F.Cu") (net 1))
   (segment (start 160.02 102.235) (end 162.135 104.35) (width 0.2286) (layer "F.Cu") (net 1))
   (segment (start 178.435 111.76) (end 180.315 111.76) (width 0.4572) (layer "F.Cu") (net 1))
   (segment (start 155.2225 102.85) (end 158.135 102.85) (width 0.2286) (layer "F.Cu") (net 1))
   (segment (start 153.365 109.41) (end 151.765 107.81) (width 0.2286) (layer "F.Cu") (net 1))
-  (segment (start 121.44378 92.67878) (end 122.11 93.345) (width 0.2286) (layer "F.Cu") (net 1))
+  (segment (start 122.11 92.996877) (end 122.11 93.345) (width 0.2286) (layer "F.Cu") (net 1))
   (segment (start 156.635 96.45) (end 155.575 95.39) (width 0.2286) (layer "F.Cu") (net 1))
   (via locked (at 178.435 109.855) (size 0.7) (drill 0.35) (layers "F.Cu" "B.Cu") (net 1))
@@
   (segment (start 182.645 99.85) (end 176.24 99.85) (width 0.2286) (layer "F.Cu") (net 11))
   (segment (start 176.24 99.85) (end 175.45 99.06) (width 0.2286) (layer "F.Cu") (net 11))
+  (segment (start 118.06372 92.18122) (end 117.3225 91.44) (width 0.2286) (layer "F.Cu") (net 27))
+  (segment (start 118.8975 94.7675) (end 121.285 97.155) (width 0.2286) (layer "F.Cu") (net 27))
+  (segment (start 119.63872 94.08622) (end 120.853114 94.08622) (width 0.2286) (layer "F.Cu") (net 27))
+  (segment (start 118.8975 93.345) (end 118.8975 94.7675) (width 0.2286) (layer "F.Cu") (net 27))
   (segment (start 162.81 101.85) (end 161.925 100.965) (width 0.2286) (layer "F.Cu") (net 27))
-  (segment (start 117.3225 93.345) (end 117.3225 94.615) (width 0.2286) (layer "F.Cu") (net 27))
+  (segment (start 118.8975 93.345) (end 119.63872 94.08622) (width 0.2286) (layer "F.Cu") (net 27))
   (segment (start 161.925 100.965) (end 161.925 100.33) (width 0.2286) (layer "F.Cu") (net 27))
-  (segment (start 117.3225 91.44) (end 117.3225 93.345) (width 0.2286) (layer "F.Cu") (net 27))
+  (segment (start 120.853114 94.08622) (end 121.285 93.654334) (width 0.2286) (layer "F.Cu") (net 27))
   (segment (start 163.5475 101.85) (end 162.81 101.85) (width 0.2286) (layer "F.Cu") (net 27))
-  (segment (start 117.3225 94.615) (end 117.39875 94.69125) (width 0.2286) (layer "F.Cu") (net 27))
-  (segment (start 151.765 97.155) (end 119.8625 97.155) (width 0.2286) (layer "F.Cu") (net 27))
-  (segment (start 119.8625 97.155) (end 117.39875 94.69125) (width 0.2286) (layer "F.Cu") (net 27))
+  (segment (start 121.285 93.654334) (end 121.285 92.71) (width 0.2286) (layer "F.Cu") (net 27))
+  (segment (start 151.765 97.155) (end 121.285 97.155) (width 0.2286) (layer "F.Cu") (net 27))
+  (segment (start 120.75622 92.18122) (end 118.06372 92.18122) (width 0.2286) (layer "F.Cu") (net 27))
+  (segment (start 121.285 92.71) (end 120.75622 92.18122) (width 0.2286) (layer "F.Cu") (net 27))
   (via (at 151.765 97.155) (size 0.7) (drill 0.35) (layers "F.Cu" "B.Cu") (net 27))
   (via (at 161.925 100.33) (size 0.7) (drill 0.35) (layers "F.Cu" "B.Cu") (net 27))
@@
   (segment (start 148.505 100.47) (end 149.86 99.115) (width 0.2286) (layer "F.Cu") (net 111))
   (segment (start 118.8975 89.535) (end 120.46 89.535) (width 0.2286) (layer "F.Cu") (net 112))
-  (segment (start 118.8975 93.345) (end 120.46 93.345) (width 0.2286) (layer "F.Cu") (net 113))
+  (segment (start 120.46 93.345) (end 119.71878 92.60378) (width 0.2286) (layer "F.Cu") (net 113))
+  (segment (start 119.71878 92.60378) (end 118.06372 92.60378) (width 0.2286) (layer "F.Cu") (net 113))
+  (segment (start 118.06372 92.60378) (end 117.3225 93.345) (width 0.2286) (layer "F.Cu") (net 113))
   (segment (start 118.8975 91.44) (end 120.46 91.44) (width 0.2286) (layer "F.Cu") (net 114))
   (segment (start 155.2225 99.85) (end 154.462916 99.85) (width 0.2286) (layer "F.Cu") (net 115))

Commit message: Hmmm
Parts:
- renumbered J2 to Je

Commit message: Getting there
Parts:
- renumbered Je to J2
Other:
- board text added: "${TITLE}, rev. ${REVISION}"
- board text removed: "PRGSTL, rev. a"

Commit message: Hmmmm
Parts:
- U1: value AMS1117-3.3 -> AMS1117-3.3``
Other:
- board text added: "RX"
- board text added: "TX"

Commit message: Hmmm
Other:
- board text removed: "${TITLE}, rev. ${REVISION}"

Commit message: Playing with ordering files
Routing:
- net +5V: track 63.8 -> 66.2 mm
- net T_TX: track 41.7 -> 42.2 mm
- net T_CLK: track 30.1 -> 30.6 mm

Commit message: Hmmm
Routing:
- net USART1_TX: track 53.1 -> 40.5 mm, vias 1 -> 0
- net USART1_RX_ALT: track 32.6 -> 40.2 mm, vias 1 -> 0
- net USART1_RX: track 58.7 -> 52.3 mm, vias 1 -> 0
- net USART1_TX_ALT: track 31.4 -> 29.0 mm, vias 1 -> 2
- net GND: vias 31 -> 36
Other:
- board text added: "JLCJLCJLCJLC"

Commit message: Hmmmm
Routing:
- net USART1_TX_ALT: track 29.0 -> 27.5 mm
