File: prgstl/prgstl.kicad_sch (KiCad schematic)
At the start: 49 parts, among them J2 STM32WORLD_BASE, Q1 S9013, U1 AMS1117-3.3, U2 STM32F103CBTx, U3 SRV05-4, Y1 X_8MHZ

Commit message: Getting there
Parts:
- U1: value AMS1117-3.3 -> (none); footprint Package_TO_SOT_SMD:SOT-223-3_TabPin2 -> (none)
Other:
- company: STM32World -> ${COMPANY}
- title: PRGSTL -> ${TITLE}
Changed lines of the file:
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@@
   (paper "A4")
   (title_block
-    (title "PRGSTL")
+    (title "${TITLE}")
     (date "2021-06-14")
-    (rev "a")
-    (company "STM32World")
-    (comment 1 "lth@stm32world.com")
-    (comment 2 "Lars Boegild Thomsen")
+    (rev "${REVISION}")
+    (company "${COMPANY}")
+    (comment 1 "${AUTHOR_EMAIL}")
+    (comment 2 "${AUTHOR}")
   )
   (junction (at 29.21 57.15) (diameter 0) (color 0 0 0 0)
@@
     (in_bom yes) (on_board yes)
     (property "Reference" "U1" (id 0) (at 30.48 21.59 0))
-    (property "Value" "AMS1117-3.3" (id 1) (at 39.37 21.59 0))
-    (property "Footprint" "Package_TO_SOT_SMD:SOT-223-3_TabPin2" (id 2) (at 34.29 20.32 0)
+    (property "Value" "" (id 1) (at 39.37 21.59 0))
+    (property "Footprint" "" (id 2) (at 34.29 20.32 0)
       (effects (font (size 1.27 1.27)) hide)
     )
@@
     )
     (path "/00000000-0000-0000-0000-000060f141a5"
-      (reference "U1") (unit 1) (value "AMS1117-3.3") (footprint "Package_TO_SOT_SMD:SOT-223-3_TabPin2")
+      (reference "U1") (unit 1) (value "AMS1117-3.3``") (footprint "Package_TO_SOT_SMD:SOT-223-3_TabPin2")
     )
     (path "/00000000-0000-0000-0000-000061012542"

Commit message: Hmmmm
Parts:
- U1: value (none) -> AMS1117-3.3``; footprint (none) -> Package_TO_SOT_SMD:SOT-223-3_TabPin2
Connections:
- no-connect marks 2 -> 77
Changed lines of the file:
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@@
   (junction (at 43.18 146.05) (diameter 0) (color 0 0 0 0)
   )
+  (no_connect (at 163.83 99.06))
+  (no_connect (at 163.83 76.2))
+  (no_connect (at 163.83 83.82))
+  (no_connect (at 163.83 88.9))
+  (no_connect (at 163.83 86.36))
+  (no_connect (at 163.83 81.28))
+  (no_connect (at 163.83 78.74))
+  (no_connect (at 163.83 73.66))
+  (no_connect (at 163.83 71.12))
+  (no_connect (at 163.83 68.58))
+  (no_connect (at 163.83 66.04))
+  (no_connect (at 163.83 55.88))
+  (no_connect (at 163.83 63.5))
+  (no_connect (at 96.52 168.91))
+  (no_connect (at 96.52 173.99))
+  (no_connect (at 245.11 85.09))
+  (no_connect (at 245.11 100.33))
+  (no_connect (at 245.11 120.65))
+  (no_connect (at 245.11 123.19))
+  (no_connect (at 245.11 87.63))
+  (no_connect (at 245.11 90.17))
+  (no_connect (at 245.11 92.71))
+  (no_connect (at 245.11 95.25))
+  (no_connect (at 245.11 102.87))
+  (no_connect (at 245.11 105.41))
+  (no_connect (at 245.11 107.95))
+  (no_connect (at 245.11 110.49))
+  (no_connect (at 245.11 115.57))
+  (no_connect (at 245.11 59.69))
+  (no_connect (at 245.11 62.23))
+  (no_connect (at 245.11 64.77))
+  (no_connect (at 245.11 67.31))
+  (no_connect (at 245.11 54.61))
+  (no_connect (at 245.11 57.15))
+  (no_connect (at 262.89 54.61))
+  (no_connect (at 262.89 57.15))
+  (no_connect (at 262.89 67.31))
+  (no_connect (at 262.89 64.77))
+  (no_connect (at 262.89 62.23))
+  (no_connect (at 262.89 59.69))
+  (no_connect (at 196.85 63.5))
+  (no_connect (at 196.85 71.12))
+  (no_connect (at 196.85 81.28))
+  (no_connect (at 196.85 78.74))
+  (no_connect (at 196.85 76.2))
+  (no_connect (at 196.85 73.66))
+  (no_connect (at 245.11 29.21))
+  (no_connect (at 245.11 26.67))
+  (no_connect (at 245.11 31.75))
+  (no_connect (at 245.11 49.53))
+  (no_connect (at 245.11 46.99))
+  (no_connect (at 245.11 39.37))
+  (no_connect (at 245.11 41.91))
+  (no_connect (at 245.11 44.45))
+  (no_connect (at 245.11 34.29))
+  (no_connect (at 262.89 46.99))
+  (no_connect (at 262.89 49.53))
+  (no_connect (at 262.89 39.37))
+  (no_connect (at 262.89 41.91))
+  (no_connect (at 262.89 44.45))
+  (no_connect (at 262.89 34.29))
+  (no_connect (at 262.89 31.75))
+  (no_connect (at 262.89 29.21))
+  (no_connect (at 262.89 85.09))
+  (no_connect (at 262.89 87.63))
+  (no_connect (at 262.89 90.17))
+  (no_connect (at 262.89 92.71))
+  (no_connect (at 262.89 95.25))
+  (no_connect (at 262.89 100.33))
+  (no_connect (at 262.89 105.41))
+  (no_connect (at 262.89 107.95))
+  (no_connect (at 262.89 110.49))
+  (no_connect (at 262.89 113.03))
+  (no_connect (at 262.89 118.11))
+  (no_connect (at 262.89 123.19))
   (no_connect (at 40.64 158.75))
   (no_connect (at 40.64 156.21))
@@
     (in_bom yes) (on_board yes)
     (property "Reference" "U1" (id 0) (at 30.48 21.59 0))
-    (property "Value" "" (id 1) (at 39.37 21.59 0))
-    (property "Footprint" "" (id 2) (at 34.29 20.32 0)
-      (effects (font (size 1.27 1.27)) hide)
-    )
+    (property "Value" "AMS1117-3.3``" (id 1) (at 39.37 21.59 0))
+    (property "Footprint" "Package_TO_SOT_SMD:SOT-223-3_TabPin2" (id 2) (at 34.29 20.32 0)
+      (effects (font (size 1.27 1.27)) hide)
+    )

Commit message: Hmmm
Parts:
- U2: LCSC (none) -> C8304
Changed lines of the file:
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@@
     (rev "${REVISION}")
     (company "${COMPANY}")
-    (comment 1 "${AUTHOR_EMAIL}")
+    (comment 1 "${URL}")
     (comment 2 "${AUTHOR}")
+    (comment 3 "${AUTHOR_EMAIL}")
   )
   (junction (at 29.21 57.15) (diameter 0) (color 0 0 0 0)
@@
       (effects (font (size 1.27 1.27)) hide)
     )
+    (property "LCSC" "C8304" (id 4) (at 181.61 66.04 0)
+      (effects (font (size 1.27 1.27)) hide)
+    )

Commit message: Hmmmm
Connections:
- net +3V3: no longer J2.1 (3.3V), J2.79 (3.3V)
- no-connect marks 77 -> 79
Changed lines of the file:
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@@
   (junction (at 213.36 60.96) (diameter 0) (color 0 0 0 0)
   )
-  (junction (at 242.57 24.13) (diameter 0) (color 0 0 0 0)
-  )
   (junction (at 137.16 53.34) (diameter 0) (color 0 0 0 0)
   )
@@
   (junction (at 242.57 69.85) (diameter 0) (color 0 0 0 0)
   )
-  (junction (at 242.57 82.55) (diameter 0) (color 0 0 0 0)
-  )
   (junction (at 43.18 146.05) (diameter 0) (color 0 0 0 0)
   )
   (no_connect (at 163.83 99.06))
+  (no_connect (at 245.11 24.13))
+  (no_connect (at 245.11 82.55))
   (no_connect (at 163.83 76.2))
   (no_connect (at 163.83 83.82))
@@
     (stroke (width 0) (type default) (color 0 0 0 0))
   )
-  (wire (pts (xy 242.57 69.85) (xy 242.57 82.55))
+  (wire (pts (xy 242.57 69.85) (xy 242.57 128.27))
     (stroke (width 0) (type default) (color 0 0 0 0))
   )
@@
     (stroke (width 0) (type default) (color 0 0 0 0))
   )
-  (wire (pts (xy 242.57 82.55) (xy 245.11 82.55))
-    (stroke (width 0) (type default) (color 0 0 0 0))
-  )
   (wire (pts (xy 106.68 53.34) (xy 106.68 49.53))
     (stroke (width 0) (type default) (color 0 0 0 0))
@@
     (stroke (width 0) (type default) (color 0 0 0 0))
   )
-  (wire (pts (xy 242.57 128.27) (xy 242.57 82.55))
-    (stroke (width 0) (type default) (color 0 0 0 0))
-  )
   (wire (pts (xy 85.09 116.84) (xy 85.09 114.3))
     (stroke (width 0) (type default) (color 0 0 0 0))
@@
     (stroke (width 0) (type default) (color 0 0 0 0))
   )
-  (wire (pts (xy 242.57 24.13) (xy 245.11 24.13))
-    (stroke (width 0) (type default) (color 0 0 0 0))
-  )
   (wire (pts (xy 48.26 25.4) (xy 48.26 27.94))
     (stroke (width 0) (type default) (color 0 0 0 0))
@@
     (stroke (width 0) (type default) (color 0 0 0 0))
   )
-  (wire (pts (xy 242.57 24.13) (xy 242.57 69.85))
+  (wire (pts (xy 242.57 21.59) (xy 242.57 69.85))
     (stroke (width 0) (type default) (color 0 0 0 0))
   )
@@
     (stroke (width 0) (type default) (color 0 0 0 0))
   )
-  (wire (pts (xy 242.57 21.59) (xy 242.57 24.13))
-    (stroke (width 0) (type default) (color 0 0 0 0))
-  )

Commit message: Hmmm
Parts:
- removed J2: STM32WORLD_BASE, stm32world:STM32WORLD_BASE, symbol stm32world:STM32WORLD_BASE
- added J2: STM32WORLD_CONNECTOR_1, stm32world:PinSocket_2x20_P2.54mm_Vertical_Stackable, symbol stm32world:STM32WORLD_CONNECTOR_1
- added J3: STM32WORLD_CONNECTOR_2, stm32world:PinSocket_2x20_P2.54mm_Vertical_Stackable, symbol stm32world:STM32WORLD_CONNECTOR_2
- added J4: STM32WORLD_BOARD, stm32world:STM32WORLD_BOARD, symbol stm32world:STM32WORLD_BOARD
- renumbered D4 to D1, D1 to D2, D2 to D3, D3 to D4, R4 to R1, R12 to R11, R11 to R12, R5 to R2, R1 to R3, R6 to R4, R2 to R5, R3 to R6, U3 to U2, U2 to U3
Connections:
- net +3V3: now also J2.38 (3.3V), J3.4 (3.3V)
- net +5V: now also J2.40 (5V), J3.2 (5V)
- net GND: now also J2.1 (GND), J2.37 (GND), J2.39 (GND), J3.1 (GND), J3.3 (GND), J3.39 (GND)
- net P_CLK: now also J3.6 (U15)
- net P_DIO: now also J3.5 (U16)
- net T_CLK: now also J3.16 (PA14)
- net T_DIO: now also J3.13 (PA13)
- net T_RST: now also J2.3 (NRST)
- net T_SWO: now also J3.23
- net USART1_RX: now also J3.12 (PA10)
- net USART1_RX_ALT: now also J3.27 (PB7)
- net USART1_TX: now also J3.9 (PA9)
- net USART1_TX_ALT: now also J3.28 (PB6)
- net USART2_RX: now also J2.11 (PA3)
- net USART2_TX: now also J2.12 (PA2)
- net USART3_RX: now also J2.23 (PB11)
- net USART3_TX: now also J2.24 (PB10)

Commit message: Tweaking
Other:
- moved on the sheet: R1, R2
Changed lines of the file:
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@@
   (junction (at 179.07 25.4) (diameter 0) (color 0 0 0 0)
   )
-  (junction (at 59.69 135.89) (diameter 0) (color 0 0 0 0)
+  (junction (at 55.88 135.89) (diameter 0) (color 0 0 0 0)
   )
   (junction (at 179.07 106.68) (diameter 0) (color 0 0 0 0)
@@
     (stroke (width 0) (type default) (color 0 0 0 0))
   )
-  (wire (pts (xy 46.99 135.89) (xy 40.64 135.89))
+  (wire (pts (xy 44.45 135.89) (xy 40.64 135.89))
     (stroke (width 0) (type default) (color 0 0 0 0))
   )
@@
     (stroke (width 0) (type default) (color 0 0 0 0))
   )
-  (wire (pts (xy 40.64 133.35) (xy 46.99 133.35))
+  (wire (pts (xy 40.64 133.35) (xy 44.45 133.35))
     (stroke (width 0) (type default) (color 0 0 0 0))
   )
@@
     (stroke (width 0) (type default) (color 0 0 0 0))
   )
-  (wire (pts (xy 59.69 135.89) (xy 59.69 156.21))
+  (wire (pts (xy 55.88 135.89) (xy 55.88 186.69))
     (stroke (width 0) (type default) (color 0 0 0 0))
   )
@@
     (stroke (width 0) (type default) (color 0 0 0 0))
   )
-  (wire (pts (xy 54.61 133.35) (xy 59.69 133.35))
+  (wire (pts (xy 52.07 133.35) (xy 55.88 133.35))
     (stroke (width 0) (type default) (color 0 0 0 0))
   )
@@
     (stroke (width 0) (type default) (color 0 0 0 0))
   )
-  (wire (pts (xy 25.4 168.91) (xy 25.4 171.45))
+  (wire (pts (xy 25.4 168.91) (xy 25.4 186.69))
     (stroke (width 0) (type default) (color 0 0 0 0))
   )
@@
     (stroke (width 0) (type default) (color 0 0 0 0))
   )
-  (wire (pts (xy 54.61 135.89) (xy 59.69 135.89))
+  (wire (pts (xy 52.07 135.89) (xy 55.88 135.89))
     (stroke (width 0) (type default) (color 0 0 0 0))
   )
@@
     (stroke (width 0) (type default) (color 0 0 0 0))
   )
-  (wire (pts (xy 59.69 135.89) (xy 59.69 133.35))
+  (wire (pts (xy 55.88 135.89) (xy 55.88 133.35))
     (stroke (width 0) (type default) (color 0 0 0 0))
   )
@@
     (pin "2")
   )
-  (symbol (lib_id "power:GND") (at 25.4 171.45 0) (unit 1)
-    (in_bom yes) (on_board yes)
-    (property "Reference" "#PWR04" (id 0) (at 25.4 177.8 0)
-      (effects (font (size 1.27 1.27)) hide)
-    )
-    (property "Value" "GND" (id 1) (at 25.527 175.8442 0))
-    (property "Footprint" "" (id 2) (at 25.4 171.45 0)
-      (effects (font (size 1.27 1.27)) hide)
-    )
-    (property "Datasheet" "" (id 3) (at 25.4 171.45 0)
+  (symbol (lib_id "power:GND") (at 25.4 186.69 0) (unit 1)
+    (in_bom yes) (on_board yes)
+    (property "Reference" "#PWR04" (id 0) (at 25.4 193.04 0)
+      (effects (font (size 1.27 1.27)) hide)
+    )
+    (property "Value" "GND" (id 1) (at 25.527 191.0842 0))
+    (property "Footprint" "" (id 2) (at 25.4 186.69 0)
+      (effects (font (size 1.27 1.27)) hide)
+    )
+    (property "Datasheet" "" (id 3) (at 25.4 186.69 0)
       (effects (font (size 1.27 1.27)) hide)
     )
@@
     (pin "2")
   )
-  (symbol (lib_id "stm32world:R_5.1K_0603") (at 50.8 133.35 270) (unit 1)
-    (in_bom yes) (on_board yes)
-    (property "Reference" "R1" (id 0) (at 45.72 132.08 90))
-    (property "Value" "R_5.1K_0603" (id 1) (at 44.45 139.7 0)
-      (effects (font (size 1.27 1.27)) hide)
-    )
-    (property "Footprint" "Resistor_SMD:R_0603_1608Metric" (id 2) (at 50.8 131.572 90)
-      (effects (font (size 1.27 1.27)) hide)
-    )
-    (property "Datasheet" "~" (id 3) (at 50.8 133.35 0)
-      (effects (font (size 1.27 1.27)) hide)
-    )
-    (property "Display" "5k1" (id 4) (at 55.88 132.08 90))
-    (property "LCSC" "C23186" (id 5) (at 46.99 138.43 0)
-      (effects (font (size 1.27 1.27)) hide)
-    )
-    (pin "1")
-    (pin "2")
-  )
-  (symbol (lib_id "stm32world:R_5.1K_0603") (at 50.8 135.89 270) (unit 1)
-    (in_bom yes) (on_board yes)
-    (property "Reference" "R2" (id 0) (at 45.72 134.62 90))
-    (property "Value" "R_5.1K_0603" (id 1) (at 44.45 142.24 0)
-      (effects (font (size 1.27 1.27)) hide)
-    )
-    (property "Footprint" "Resistor_SMD:R_0603_1608Metric" (id 2) (at 50.8 134.112 90)
-      (effects (font (size 1.27 1.27)) hide)
-    )
-    (property "Datasheet" "~" (id 3) (at 50.8 135.89 0)
-      (effects (font (size 1.27 1.27)) hide)
-    )
-    (property "Display" "5k1" (id 4) (at 55.88 134.62 90))
-    (property "LCSC" "C23186" (id 5) (at 46.99 140.97 0)
+  (symbol (lib_id "stm32world:R_5.1K_0603") (at 48.26 133.35 270) (unit 1)
+    (in_bom yes) (on_board yes)
+    (property "Reference" "R1" (id 0) (at 43.18 132.08 90))
+    (property "Value" "R_5.1K_0603" (id 1) (at 41.91 139.7 0)
+      (effects (font (size 1.27 1.27)) hide)
+    )
+    (property "Footprint" "Resistor_SMD:R_0603_1608Metric" (id 2) (at 48.26 131.572 90)
+      (effects (font (size 1.27 1.27)) hide)
+    )
+    (property "Datasheet" "~" (id 3) (at 48.26 133.35 0)
+      (effects (font (size 1.27 1.27)) hide)
+    )
+    (property "Display" "5k1" (id 4) (at 53.34 132.08 90))
+    (property "LCSC" "C23186" (id 5) (at 44.45 138.43 0)
+      (effects (font (size 1.27 1.27)) hide)
+    )
+    (pin "1")
+    (pin "2")
+  )
+  (symbol (lib_id "stm32world:R_5.1K_0603") (at 48.26 135.89 270) (unit 1)
+    (in_bom yes) (on_board yes)
+    (property "Reference" "R2" (id 0) (at 43.18 134.62 90))
+    (property "Value" "R_5.1K_0603" (id 1) (at 41.91 142.24 0)
+      (effects (font (size 1.27 1.27)) hide)
+    )
+    (property "Footprint" "Resistor_SMD:R_0603_1608Metric" (id 2) (at 48.26 134.112 90)
+      (effects (font (size 1.27 1.27)) hide)
+    )
+    (property "Datasheet" "~" (id 3) (at 48.26 135.89 0)
+      (effects (font (size 1.27 1.27)) hide)
+    )
+    (property "Display" "5k1" (id 4) (at 53.34 134.62 90))
+    (property "LCSC" "C23186" (id 5) (at 44.45 140.97 0)
       (effects (font (size 1.27 1.27)) hide)
     )
@@
     (pin "1")
   )
-  (symbol (lib_id "power:GND") (at 59.69 156.21 0) (unit 1)
-    (in_bom yes) (on_board yes)
-    (property "Reference" "#PWR08" (id 0) (at 59.69 162.56 0)
-      (effects (font (size 1.27 1.27)) hide)
-    )
-    (property "Value" "GND" (id 1) (at 59.817 160.6042 0))
-    (property "Footprint" "" (id 2) (at 59.69 156.21 0)
-      (effects (font (size 1.27 1.27)) hide)
-    )
-    (property "Datasheet" "" (id 3) (at 59.69 156.21 0)
-      (effects (font (size 1.27 1.27)) hide)
-    )
+  (symbol (lib_id "power:GND") (at 55.88 186.69 0) (unit 1)
+    (in_bom yes) (on_board yes)
+    (property "Reference" "#PWR08" (id 0) (at 55.88 193.04 0)
+      (effects (font (size 1.27 1.27)) hide)
+    )
+    (property "Value" "GND" (id 1) (at 56.007 191.0842 0))
+    (property "Footprint" "" (id 2) (at 55.88 186.69 0)
+      (effects (font (size 1.27 1.27)) hide)
+    )
+    (property "Datasheet" "" (id 3) (at 55.88 186.69 0)
+      (effects (font (size 1.27 1.27)) hide)
+    )

Commit message: Ready to order prgctl
Connections:
- net T_CLK: now also U3.15 (PA5)
- no-connect marks 79 -> 78
