File: mcustm32f405/mcustm32f405.kicad_sch (KiCad schematic)
At the start: 31 parts, among them J2 STM32WORLD_BASE, U1 AMS1117-3.3, U2 STM32F405RGTx, U3 SRV05-4, Y1 X_16MHZ

Commit message: Hmmmm
Parts:
- added C2, C8: C_100NF_0603, Capacitor_SMD:C_0603_1608Metric, symbol stm32world:C_100NF_0603
- added FB1: FB_0603, Inductor_SMD:L_0603_1608Metric, symbol stm32world:FB_0603
- added JP1, JP2: SolderJumper_2_Bridged, Jumper:SolderJumper-2_P1.3mm_Bridged_RoundedPad1.0x1.5mm, symbol stm32world:SolderJumper_2_Bridged
- U3: renamed from U2; LCSC (none) -> C15742
- renumbered C2 to C10, C10 to C11, C9 to C12, C11 to C13, C12 to C14, C8 to C9, R3 to R1, R4 to R2, R5 to R3, R6 to R4, R1 to R5, R2 to R6, U3 to U2
Connections:
- net +3V3: now also JP1.1 (A), JP2.1 (A); no longer J2.1 (3.3V), J2.79 (3.3V), U3.1 (VBAT), U3.13 (VDDA)
- net GND: now also C2.2, C8.2
- new net VA: C8.1, FB1.2, U3.13 (VDDA)
- new net VBAT: C2.1, J2.79 (VB), JP1.2 (B), U3.1 (VBAT)
- new net VDDA: FB1.1, J2.1 (VA), JP2.2 (B)
Other:
- note added: "Shorted by default"
- note removed: "Internal pull-up"
- company: STM32World -> ${COMPANY}
- title: MCUSTM32F405 -> ${TITLE}
- moved on the sheet: C10, C11, C12, C13, C14, D1, D2, D3, J1, J2, R1, R2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

Commit message: Hmmmm
Parts:
- SW1, SW2: value ~ -> TS-1088R-02526
- renumbered C9 to C10, C10 to C9
Other:
- note added: "Analog power filtering"
- note added: "Battery power"
- note added: "Connector"
- note added: "Decoupling"
- note added: "LEDs"
- note added: "MCU and oscillator"
- note added: "Power regulation"
- note added: "Reset and boot0"
- note added: "USB-C Connector"
- moved on the sheet: C1, C3, C9, D1, D2, D3, J1, J2, R1, R2, R3, R4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

Commit message: Hmmm
Parts:
- removed R3, R4: R_22_0603, Resistor_SMD:R_0603_1608Metric, symbol stm32world:R_22_0603
- renumbered R5 to R3, R6 to R4, R7 to R5, R8 to R6
Connections:
- net GND: now also R1.1, R2.1
- net PA11: now also J1.A7 (D-), J1.B7 (D-), U2.3 (IO2)
- net PA12: now also J1.A6 (D+), J1.B6 (D+), U2.1 (IO1)
- net PC14: no longer R1.1, R2.1
Other:
- moved on the sheet: D1, J1, R1, R2, U2
