File: mcustm32f405/mcustm32f405.kicad_pcb (KiCad board)
At the start: 2 copper layers, 76.2 x 50.8 mm, 38 parts, among them J2 STM32WORLD_CONNECTOR_1, J3 STM32WORLD_CONNECTOR_2, J4 STM32WORLD_BOARD, SW1 TS-1088R-02526, SW2 TS-1088R-02526, U1 AMS1117-3.3, U2 STM32F405RGTx, Y1 X_16MHZ

Commit message: Wired B0 to PC15 so it can be read
Connections:
- J3 pad 35: PC15 -> BO0
- U2 pad 4: PC15 -> BO0
Routing:
- net PC15: track 22.8 -> 0.00 mm
- net BO0: track 51.3 -> 74.2 mm
- net +5V: track 61.7 -> 69.3 mm, vias 0 -> 1
- net GND: vias 23 -> 28

Commit message: Hmmmm
Parts:
- moved C14 0.25 mm to (160.7, 97.2)
- moved C7 0.25 mm to (160.7, 95.2)
Routing:
- net GND: vias 28 -> 29

Commit message: Hmmm
Routing:
- net BO0: track 74.2 -> 70.6 mm, vias 3 -> 4
- net GND: vias 29 -> 34
