File: mcustm32f446/mcustm32f446.kicad_sch (KiCad schematic)
At the start: 30 parts, among them J2 STM32WORLD_BASE, U1 AMS1117-3.3, U2 SRV05-4, U3 STM32F446RCTx, Y1 X_16MHZ

Commit message: Hmmmm
Parts:
- added C9: C_100NF_0603, Capacitor_SMD:C_0603_1608Metric, symbol stm32world:C_100NF_0603
- added JP1: ~, symbol Jumper:SolderJumper_2_Bridged
- renumbered C9 to C10, C10 to C11, C11 to C12
Connections:
- net +3V3: now also JP1.1 (A); no longer U3.1 (VBAT)
- net GND: now also C9.2
- new net VBAT: C9.1, JP1.2 (B), U3.1 (VBAT)
Other:
- moved on the sheet: C10, C11, C12, U3, Y1

Commit message: Hmmmm
Parts:
- removed JP1: ~, symbol Jumper:SolderJumper_2_Bridged
- added FB1: FB_0603, Inductor_SMD:L_0603_1608Metric, symbol stm32world:FB_0603
- added JP1, JP2: SolderJumper_2_Bridged, Jumper:SolderJumper-2_P1.3mm_Bridged_RoundedPad1.0x1.5mm, symbol stm32world:SolderJumper_2_Bridged
- renumbered C9 to C3, C3 to C4, C4 to C5, C5 to C6, C6 to C8, C8 to C9, R3 to R2, R4 to R3, R2 to R4
Connections:
- net +3V3: now also JP1.1 (A), JP2.1 (A); no longer C7.1, J2.1 (3.3V), J2.79 (3.3V), U3.13 (VDDA)
- net VBAT: now also J2.79 (VB), JP1.2 (B)
- new net VA: FB1.1, J2.1 (VA), JP2.2 (B)
- new net VDDA: C7.1, FB1.2, U3.13 (VDDA)
Other:
- note removed: "Internal pull-up"
- moved on the sheet: C10, C11, C12, C2, C3, C9, D1, D2, D3, J1, J2, R1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

Commit message: Hmmmm
Other:
- note added: "Shorted by default"
- moved on the sheet: C10, C11, C12, C2, C3, C7, D1, D3, FB1, JP1, JP2, R1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

Commit message: Hmmm
Parts:
- removed J2: STM32WORLD_BASE, stm32world:STM32WORLD_BASE, symbol stm32world:STM32WORLD_BASE
- removed R5, R6: R_22_0603, Resistor_SMD:R_0603_1608Metric, symbol stm32world:R_22_0603
- added C9: C_100NF_0603, Capacitor_SMD:C_0603_1608Metric, symbol stm32world:C_100NF_0603
- added J2: STM32WORLD_CONNECTOR_1, stm32world:PinSocket_2x20_P2.54mm_Vertical_Stackable, symbol stm32world:STM32WORLD_CONNECTOR_1
- added J3: STM32WORLD_CONNECTOR_2, stm32world:PinSocket_2x20_P2.54mm_Vertical_Stackable, symbol stm32world:STM32WORLD_CONNECTOR_2
- added J4: STM32WORLD_BOARD, stm32world:STM32WORLD_BOARD, symbol stm32world:STM32WORLD_BOARD
- renumbered C2 to C10, C10 to C11, C11 to C12, C12 to C13, C3 to C2, C4 to C3, C5 to C4, C6 to C5, C8 to C6, C9 to C7, C7 to C8, D2 to D1, D1 to D2, R2 to R1, R3 to R2, R1 to R3, R7 to R5, R8 to R6
Connections:
- net +3V3: now also C9.1, J2.38 (3.3V), J3.4 (3.3V)
- net +5V: now also J2.40 (5V), J3.2 (5V)
- net BO0: now also J2.4 (BO0)
- net GND: now also R1.1, R2.1, C9.2, J2.1 (GND), J2.37 (GND), J2.39 (GND), J3.1 (GND), J3.3 (GND), J3.39 (GND)
- net NRST: now also J2.3 (NRST)
- net PA0: now also J2.10 (PA0)
- net PA1: now also J2.9 (PA1)
- net PA10: now also J3.12 (PA10)
- net PA11: now also J1.A7 (D-), J1.B7 (D-), U2.3 (IO2), J3.11 (PA11)
- net PA12: now also J1.A6 (D+), J1.B6 (D+), U2.1 (IO1), J3.14 (PA12)
- net PA13: now also J3.13 (PA13)
- net PA14: now also J3.16 (PA14)
- net PA15: now also J3.15 (PA15)
- net PA2: now also J2.12 (PA2)
- net PA3: now also J2.11 (PA3)
- net PA4: now also J2.14 (PA4)
- net PA5: now also J2.13 (PA5)
- net PA6: now also J2.16 (PA6)
- net PA7: now also J2.15 (PA7)
- net PA8: now also J3.10 (PA8)
- net PA9: now also J3.9 (PA9)
- net PB0: now also J2.20 (PB0)
- net PB1: now also J2.19 (PB1)
- net PB10: now also J2.24 (PB10)
- net PB12: now also J2.26 (PB12)
- net PB13: now also J2.25 (PB13)
- net PB14: now also J2.28 (PB14)
- net PB15: now also J2.27 (PB15)
- net PB2: now also J2.22 (PB2)
- net PB3: now also J3.23
- net PB4: now also J3.26 (PB4)
- net PB5: now also J3.25 (PB5)
- net PB6: now also J3.28 (PB6)
- net PB7: now also J3.27 (PB7)
- net PB8: now also J3.30 (PB8)
- net PB9: now also J3.29 (PB9)
- net PC0: now also J2.6 (PC0)
- net PC1: now also J2.5 (PC1)
- net PC10: now also J3.20 (PC10)
- net PC11: now also J3.19 (PC11)
- net PC12: now also J3.22 (PC12)
- net PC13: now also J3.33 (PC13)
- net PC14: now also J3.34 (PC14); no longer R1.1, R2.1
- net PC15: now also J3.35 (PC15)
- net PC2: now also J2.8 (PC2)
- net PC3: now also J2.7 (PC3)
- net PC4: now also J2.18 (PC4)
- net PC5: now also J2.17 (PC5)
- net PC6: now also J2.30 (PC6)
- net PC7: now also J2.29 (PC7)
- net PC8: now also J2.32 (PC8)
- net PC9: now also J2.31 (PC9)
- net PD2: now also J3.24 (PD2)
- net VA: now also J2.2 (VA)
- net VBAT: now also J3.40 (VB)
- no-connect marks 2 -> 22
Other:
- moved on the sheet: D1, R1, R2, U2

Commit message: Ready to order prgctl
Connections:
- net VA: now also C8.1, FB1.2, U3.13 (VDDA); no longer FB1.1, J2.2 (VA), JP2.2 (B)
- net VDDA: now also FB1.1, J2.2 (VA), JP2.2 (B); no longer C8.1, FB1.2, U3.13 (VDDA)
Changed lines of the file:
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@@
   (junction (at 271.78 74.93) (diameter 0) (color 0 0 0 0)
   )
-  (junction (at 83.82 71.12) (diameter 0) (color 0 0 0 0)
-  )
   (junction (at 97.79 39.37) (diameter 0) (color 0 0 0 0)
   )
@@
     (stroke (width 0) (type default) (color 0 0 0 0))
   )
+  (wire (pts (xy 199.39 27.94) (xy 199.39 30.48))
+    (stroke (width 0) (type default) (color 0 0 0 0))
+  )
   (wire (pts (xy 271.78 85.09) (xy 271.78 130.81))
     (stroke (width 0) (type default) (color 0 0 0 0))
   )
+  (wire (pts (xy 97.79 78.74) (xy 101.6 78.74))
+    (stroke (width 0) (type default) (color 0 0 0 0))
+  )
   (wire (pts (xy 48.26 129.54) (xy 48.26 132.08))
     (stroke (width 0) (type default) (color 0 0 0 0))
@@
     (stroke (width 0) (type default) (color 0 0 0 0))
   )
+  (wire (pts (xy 83.82 80.01) (xy 83.82 78.74))
+    (stroke (width 0) (type default) (color 0 0 0 0))
+  )
   (wire (pts (xy 71.12 78.74) (xy 73.66 78.74))
     (stroke (width 0) (type default) (color 0 0 0 0))
@@
     (stroke (width 0) (type default) (color 0 0 0 0))
   )
+  (wire (pts (xy 238.76 26.67) (xy 238.76 24.13))
+    (stroke (width 0) (type default) (color 0 0 0 0))
+  )
   (wire (pts (xy 194.31 27.94) (xy 196.85 27.94))
     (stroke (width 0) (type default) (color 0 0 0 0))
@@
     (stroke (width 0) (type default) (color 0 0 0 0))
   )
-  (wire (pts (xy 88.9 71.12) (xy 83.82 71.12))
-    (stroke (width 0) (type default) (color 0 0 0 0))
-  )
   (wire (pts (xy 212.09 66.04) (xy 209.55 66.04))
     (stroke (width 0) (type default) (color 0 0 0 0))
@@
     (stroke (width 0) (type default) (color 0 0 0 0))
   )
+  (wire (pts (xy 201.93 27.94) (xy 199.39 27.94))
+    (stroke (width 0) (type default) (color 0 0 0 0))
+  )
   (wire (pts (xy 196.85 119.38) (xy 196.85 121.92))
     (stroke (width 0) (type default) (color 0 0 0 0))
@@
     (stroke (width 0) (type default) (color 0 0 0 0))
   )
+  (wire (pts (xy 83.82 76.2) (xy 83.82 78.74))
+    (stroke (width 0) (type default) (color 0 0 0 0))
+  )
   (wire (pts (xy 48.26 132.08) (xy 54.61 132.08))
     (stroke (width 0) (type default) (color 0 0 0 0))
@@
     (stroke (width 0) (type default) (color 0 0 0 0))
   )
-  (wire (pts (xy 83.82 71.12) (xy 83.82 78.74))
-    (stroke (width 0) (type default) (color 0 0 0 0))
-  )
   (wire (pts (xy 191.77 27.94) (xy 193.04 27.94))
     (stroke (width 0) (type default) (color 0 0 0 0))
@@
     (stroke (width 0) (type default) (color 0 0 0 0))
   )
-  (wire (pts (xy 186.69 30.48) (xy 186.69 27.94))
+  (wire (pts (xy 38.1 73.66) (xy 38.1 76.2))
     (stroke (width 0) (type default) (color 0 0 0 0))
   )
-  (wire (pts (xy 199.39 25.4) (xy 199.39 30.48))
+  (wire (pts (xy 186.69 30.48) (xy 186.69 27.94))
     (stroke (width 0) (type default) (color 0 0 0 0))
   )
@@
     (stroke (width 0) (type default) (color 0 0 0 0))
   )
-  (wire (pts (xy 241.3 26.67) (xy 251.46 26.67))
+  (wire (pts (xy 238.76 26.67) (xy 251.46 26.67))
     (stroke (width 0) (type default) (color 0 0 0 0))
   )
@@
     (effects (font (size 1.27 1.27)) (justify left bottom))
   )
+  (global_label "VA" (shape input) (at 201.93 27.94 0) (fields_autoplaced)
+    (effects (font (size 1.27 1.27)) (justify left))
+    (property "Intersheet References" "${INTERSHEET_REFS}" (id 0) (at 206.4313 27.8606 0)
+      (effects (font (size 1.27 1.27)) (justify left) hide)
+    )
+  )
   (global_label "PC8" (shape input) (at 171.45 96.52 180) (fields_autoplaced)
     (effects (font (size 1.27 1.27)) (justify right))
@@
     )
   )
-  (global_label "VA" (shape input) (at 241.3 26.67 180) (fields_autoplaced)
-    (effects (font (size 1.27 1.27)) (justify right))
-    (property "Intersheet References" "${INTERSHEET_REFS}" (id 0) (at 236.7987 26.7494 0)
-      (effects (font (size 1.27 1.27)) (justify right) hide)
-    )
-  )
   (global_label "PC8" (shape input) (at 241.3 64.77 180) (fields_autoplaced)
     (effects (font (size 1.27 1.27)) (justify right))
@@
     )
   )
-  (global_label "VA" (shape input) (at 88.9 71.12 0) (fields_autoplaced)
+  (global_label "VA" (shape input) (at 101.6 78.74 0) (fields_autoplaced)
     (effects (font (size 1.27 1.27)) (justify left))
-    (property "Intersheet References" "${INTERSHEET_REFS}" (id 0) (at 93.4013 71.0406 0)
+    (property "Intersheet References" "${INTERSHEET_REFS}" (id 0) (at 106.1013 78.6606 0)
       (effects (font (size 1.27 1.27)) (justify left) hide)
     )
@@
     (pin "4")
   )
-  (symbol (lib_id "power:PWR_FLAG") (at 97.79 78.74 270) (unit 1)
+  (symbol (lib_id "power:PWR_FLAG") (at 97.79 76.2 0) (unit 1)
     (in_bom yes) (on_board yes)
-    (property "Reference" "#FLG06" (id 0) (at 99.695 78.74 0)
+    (property "Reference" "#FLG06" (id 0) (at 97.79 74.295 0)
       (effects (font (size 1.27 1.27)) hide)
     )
-    (property "Value" "PWR_FLAG" (id 1) (at 102.1842 78.74 0)
+    (property "Value" "PWR_FLAG" (id 1) (at 97.79 71.8058 0)
       (effects (font (size 1.27 1.27)) hide)
     )
-    (property "Footprint" "" (id 2) (at 97.79 78.74 0)
+    (property "Footprint" "" (id 2) (at 97.79 76.2 0)
       (effects (font (size 1.27 1.27)) hide)
     )
-    (property "Datasheet" "~" (id 3) (at 97.79 78.74 0)
+    (property "Datasheet" "~" (id 3) (at 97.79 76.2 0)
       (effects (font (size 1.27 1.27)) hide)
     )
@@
     (pin "2")
   )
-  (symbol (lib_id "power:VDDA") (at 97.79 76.2 0) (unit 1)
-    (in_bom yes) (on_board yes) (fields_autoplaced)
-    (property "Reference" "#PWR015" (id 0) (at 97.79 80.01 0)
+  (symbol (lib_id "power:VDDA") (at 83.82 76.2 0) (unit 1)
+    (in_bom yes) (on_board yes)
+    (property "Reference" "#PWR015" (id 0) (at 83.82 80.01 0)
       (effects (font (size 1.27 1.27)) hide)
     )
-    (property "Value" "VDDA" (id 1) (at 97.79 71.12 0))
-    (property "Footprint" "" (id 2) (at 97.79 76.2 0)
+    (property "Value" "VDDA" (id 1) (at 83.82 72.39 0))
+    (property "Footprint" "" (id 2) (at 83.82 76.2 0)
       (effects (font (size 1.27 1.27)) hide)
     )
-    (property "Datasheet" "" (id 3) (at 97.79 76.2 0)
+    (property "Datasheet" "" (id 3) (at 83.82 76.2 0)
       (effects (font (size 1.27 1.27)) hide)
     )
@@
     (pin "2")
   )
-  (symbol (lib_id "power:PWR_FLAG") (at 83.82 71.12 0) (unit 1)
+  (symbol (lib_id "power:VDDA") (at 238.76 24.13 0) (unit 1)
     (in_bom yes) (on_board yes)
-    (property "Reference" "#FLG05" (id 0) (at 83.82 69.215 0)
+    (property "Reference" "#PWR0101" (id 0) (at 238.76 27.94 0)
       (effects (font (size 1.27 1.27)) hide)
     )
-    (property "Value" "PWR_FLAG" (id 1) (at 83.82 66.7258 0)
+    (property "Value" "VDDA" (id 1) (at 238.76 20.32 0))
+    (property "Footprint" "" (id 2) (at 238.76 24.13 0)
       (effects (font (size 1.27 1.27)) hide)
     )
-    (property "Footprint" "" (id 2) (at 83.82 71.12 0)
+    (property "Datasheet" "" (id 3) (at 238.76 24.13 0)
       (effects (font (size 1.27 1.27)) hide)
     )
-    (property "Datasheet" "~" (id 3) (at 83.82 71.12 0)
+    (pin "1")
+  )
+  (symbol (lib_id "power:PWR_FLAG") (at 83.82 80.01 180) (unit 1)
+    (in_bom yes) (on_board yes)
+    (property "Reference" "#FLG05" (id 0) (at 83.82 81.915 0)
+      (effects (font (size 1.27 1.27)) hide)
+    )
+    (property "Value" "PWR_FLAG" (id 1) (at 83.82 84.4042 0)
+      (effects (font (size 1.27 1.27)) hide)
+    )
+    (property "Footprint" "" (id 2) (at 83.82 80.01 0)
+      (effects (font (size 1.27 1.27)) hide)
+    )
+    (property "Datasheet" "~" (id 3) (at 83.82 80.01 0)
       (effects (font (size 1.27 1.27)) hide)
     )
@@
     (pin "1")
   )
-  (symbol (lib_id "power:PWR_FLAG") (at 38.1 76.2 0) (unit 1)
+  (symbol (lib_id "power:PWR_FLAG") (at 38.1 73.66 0) (unit 1)
     (in_bom yes) (on_board yes)
-    (property "Reference" "#FLG02" (id 0) (at 38.1 74.295 0)
+    (property "Reference" "#FLG02" (id 0) (at 38.1 71.755 0)
       (effects (font (size 1.27 1.27)) hide)
     )
-    (property "Value" "PWR_FLAG" (id 1) (at 38.1 71.8058 0)
+    (property "Value" "PWR_FLAG" (id 1) (at 38.1 69.2658 0)
       (effects (font (size 1.27 1.27)) hide)
     )
-    (property "Footprint" "" (id 2) (at 38.1 76.2 0)
+    (property "Footprint" "" (id 2) (at 38.1 73.66 0)
       (effects (font (size 1.27 1.27)) hide)
     )
-    (property "Datasheet" "~" (id 3) (at 38.1 76.2 0)
+    (property "Datasheet" "~" (id 3) (at 38.1 73.66 0)
       (effects (font (size 1.27 1.27)) hide)
     )
@@
     (pin "1")
   )
-  (symbol (lib_id "power:VDDA") (at 199.39 25.4 0) (unit 1)
-    (in_bom yes) (on_board yes)
-    (property "Reference" "#PWR031" (id 0) (at 199.39 29.21 0)
-      (effects (font (size 1.27 1.27)) hide)
-    )
-    (property "Value" "VDDA" (id 1) (at 199.39 21.59 0))
-    (property "Footprint" "" (id 2) (at 199.39 25.4 0)
-      (effects (font (size 1.27 1.27)) hide)
-    )
-    (property "Datasheet" "" (id 3) (at 199.39 25.4 0)
-      (effects (font (size 1.27 1.27)) hide)
-    )
-    (pin "1")
-  )
   (sheet_instances
     (path "/" (page "1"))
@@
       (reference "#PWR030") (unit 1) (value "+3V3") (footprint "")
     )
-    (path "/fdf71bf7-b8ed-4c8d-8f6e-bf629ca091e7"
-      (reference "#PWR031") (unit 1) (value "VDDA") (footprint "")
-    )
     (path "/00000000-0000-0000-0000-0000611ee08c"
       (reference "#PWR032") (unit 1) (value "+5V") (footprint "")
@@
       (reference "#PWR034") (unit 1) (value "GND") (footprint "")
     )
+    (path "/75e20e62-7433-4ded-8089-4cf33a7d8928"
+      (reference "#PWR0101") (unit 1) (value "VDDA") (footprint "")
+    )
     (path "/00000000-0000-0000-0000-000060f3d5aa"
