File: mcump151/mcump151.kicad_pcb (KiCad board)
At the start: 8 copper layers, 76.2 x 50.8 mm, 4 parts, among them J1 STM32WORLD_BOARD, J2 STM32WORLD_CONNECTOR_1, J3 STM32WORLD_CONNECTOR_2, U1 STM32MP151AACx

Commit message: Playing with mcustm32mp151
Parts:
- added J4: USB_C_Receptacle_USB2.0, stm32world:USB_C_Receptacle_HRO_TYPE-C-31-M-12, F.Cu at (180.3, 88.9)
- added J5: USB_C_Receptacle_USB2.0, stm32world:USB_C_Receptacle_HRO_TYPE-C-31-M-12, F.Cu at (180.3, 101.5)
- added U2: AS4C256M16D3, Package_BGA:BGA-96_9.0x13.0mm_Layout2x3x16_P0.8mm, F.Cu at (162.2, 92.5)
- U1: footprint stm32world:TFBGA361_12X12_STM -> Package_BGA:ST_TFBGA-361_12x12mm_Layout23x23_P0.5mmP0.65mm
Routing:
- net GND: track 0.27 -> 0.63 mm, vias 1 -> 2
