File: mcump151/mcump151.kicad_sch (KiCad schematic)
At the start: 4 parts, among them J1 STM32WORLD_BOARD, J2 STM32WORLD_CONNECTOR_1, J3 STM32WORLD_CONNECTOR_2, U1 STM32MP151AACx

Commit message: Playing with mcustm32mp151
Parts:
- added J4, J5: USB_C_Receptacle_USB2.0, stm32world:USB_C_Receptacle_HRO_TYPE-C-31-M-12, symbol stm32world:USB_C_Receptacle_USB2.0
- added U2: AS4C256M16D3, Package_BGA:BGA-96_9.0x13.0mm_Layout2x3x16_P0.8mm, symbol Memory_RAM:AS4C256M16D3
- U1: footprint stm32world:TFBGA361_12X12_STM -> Package_BGA:ST_TFBGA-361_12x12mm_Layout23x23_P0.5mmP0.65mm
Connections:
- new net: J4.A1 (GND), J4.A12 (GND), J4.B1 (GND), J4.B12 (GND)
- new net: J4.A4 (VBUS), J4.A9 (VBUS), J4.B4 (VBUS), J4.B9 (VBUS)
- new net: J5.A1 (GND), J5.A12 (GND), J5.B1 (GND), J5.B12 (GND)
- new net: J5.A4 (VBUS), J5.A9 (VBUS), J5.B4 (VBUS), J5.B9 (VBUS)
- new net: U2.A1 (VDDQ), U2.A8 (VDDQ), U2.C1 (VDDQ), U2.C9 (VDDQ), U2.D2 (VDDQ), U2.E9 (VDDQ), U2.F1 (VDDQ), U2.H2 (VDDQ), U2.H9 (VDDQ)
- new net: U2.A9 (VSS), U2.B3 (VSS), U2.E1 (VSS), U2.G8 (VSS), U2.J2 (VSS), U2.J8 (VSS), U2.M1 (VSS), U2.M9 (VSS), U2.P1 (VSS), U2.P9 (VSS), U2.T1 (VSS), U2.T9 (VSS)
- new net: U2.B1 (VSSQ), U2.B9 (VSSQ), U2.D1 (VSSQ), U2.D8 (VSSQ), U2.E2 (VSSQ), U2.E8 (VSSQ), U2.F9 (VSSQ), U2.G1 (VSSQ), U2.G9 (VSSQ)
- new net: U2.B2 (VDD), U2.D9 (VDD), U2.G7 (VDD), U2.K2 (VDD), U2.K8 (VDD), U2.N1 (VDD), U2.N9 (VDD), U2.R1 (VDD), U2.R9 (VDD)
Changed lines of the file:
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@@
     (stroke (width 0) (type default))
+  )
+  (symbol (lib_id "stm32world:USB_C_Receptacle_USB2.0") (at 49.53 133.35 0) (unit 1)
+    (in_bom yes) (on_board yes) (dnp no) (fields_autoplaced)
+    (property "Reference" "J4" (at 49.53 107.95 0)
+      (effects (font (size 1.27 1.27)))
+    )
+    (property "Value" "USB_C_Receptacle_USB2.0" (at 49.53 110.49 0)
+      (effects (font (size 1.27 1.27)))
+    )
+    (property "Footprint" "stm32world:USB_C_Receptacle_HRO_TYPE-C-31-M-12" (at 53.34 133.35 0)
+      (effects (font (size 1.27 1.27)) hide)
+    )
+    (property "Datasheet" "" (at 53.34 133.35 0)
+      (effects (font (size 1.27 1.27)) hide)
+    )
+    (property "LCSC" "C165948" (at 49.53 113.03 0)
+      (effects (font (size 1.27 1.27)))
+    )
+    (pin "A1")
+    (pin "A12")
+    (pin "A4")
+    (pin "A5")
+    (pin "A6")
+    (pin "A7")
+    (pin "A8")
+    (pin "A9")
+    (pin "B1")
+    (pin "B12")
+    (pin "B4")
+    (pin "B5")
+    (pin "B6")
+    (pin "B7")
+    (pin "B8")
+    (pin "B9")
+    (pin "S1")
+    (instances
+      (project "mcump151"
+        (path "/45483761-40cc-431f-bcc2-65a9a869d9c1"
+          (reference "J4") (unit 1)
+        )
+      )
+    )
   )
   (symbol (lib_id "stm32world:STM32WORLD_CONNECTOR_2") (at 552.45 118.11 0) (unit 1)
@@
       (effects (font (size 1.27 1.27)) (justify left))
     )
-    (property "Footprint" "stm32world:TFBGA361_12X12_STM" (at 215.9 384.81 0)
+    (property "Footprint" "Package_BGA:ST_TFBGA-361_12x12mm_Layout23x23_P0.5mmP0.65mm" (at 215.9 384.81 0)
       (effects (font (size 1.27 1.27)) (justify right) hide)
     )
@@
         )
       )
+    )
+  )
+  (symbol (lib_id "stm32world:USB_C_Receptacle_USB2.0") (at 46.99 199.39 0) (unit 1)
+    (in_bom yes) (on_board yes) (dnp no) (fields_autoplaced)
+    (property "Reference" "J5" (at 46.99 173.99 0)
+      (effects (font (size 1.27 1.27)))
+    )
+    (property "Value" "USB_C_Receptacle_USB2.0" (at 46.99 176.53 0)
+      (effects (font (size 1.27 1.27)))
+    )
+    (property "Footprint" "stm32world:USB_C_Receptacle_HRO_TYPE-C-31-M-12" (at 50.8 199.39 0)
+      (effects (font (size 1.27 1.27)) hide)
+    )
+    (property "Datasheet" "" (at 50.8 199.39 0)
+      (effects (font (size 1.27 1.27)) hide)
+    )
+    (property "LCSC" "C165948" (at 46.99 179.07 0)
+      (effects (font (size 1.27 1.27)))
+    )
+    (pin "A1")
+    (pin "A12")
+    (pin "A4")
+    (pin "A5")
+    (pin "A6")
+    (pin "A7")
+    (pin "A8")
+    (pin "A9")
+    (pin "B1")
+    (pin "B12")
+    (pin "B4")
+    (pin "B5")
+    (pin "B6")
+    (pin "B7")
+    (pin "B8")
+    (pin "B9")
+    (pin "S1")
+    (instances
+      (project "mcump151"
+        (path "/45483761-40cc-431f-bcc2-65a9a869d9c1"
+          (reference "J5") (unit 1)
+        )
+      )
+    )
+  )
+  (symbol (lib_id "Memory_RAM:AS4C256M16D3") (at 435.61 175.26 0) (unit 1)
+    (in_bom yes) (on_board yes) (dnp no) (fields_autoplaced)
+    (property "Reference" "U2" (at 437.8041 218.44 0)
+      (effects (font (size 1.27 1.27)) (justify left))
+    )
+    (property "Value" "AS4C256M16D3" (at 437.8041 220.98 0)
+      (effects (font (size 1.27 1.27)) (justify left))
+    )
+    (property "Footprint" "Package_BGA:BGA-96_9.0x13.0mm_Layout2x3x16_P0.8mm" (at 434.34 129.54 0)
+      (effects (font (size 1.27 1.27)) hide)
+    )
+    (property "Datasheet" "https://www.alliancememory.com/wp-content/uploads/pdf/ddr3/4GB-AS4C256M16D3.pdf" (at 434.34 106.68 0)
+      (effects (font (size 1.27 1.27)) hide)
+    )
+    (pin "A1")
+    (pin "A8")
+    (pin "A9")
+    (pin "B1")
+    (pin "B2")
+    (pin "B3")
+    (pin "B9")
+    (pin "C1")
+    (pin "C9")
+    (pin "D1")
+    (pin "D2")
+    (pin "D8")
+    (pin "D9")
+    (pin "E1")
+    (pin "E2")
+    (pin "E3")
+    (pin "E8")
+    (pin "E9")
+    (pin "F1")
+    (pin "F2")
+    (pin "F7")
+    (pin "F8")
+    (pin "F9")
+    (pin "G1")
+    (pin "G2")
+    (pin "G7")
+    (pin "G8")
+    (pin "G9")
+    (pin "H1")
+    (pin "H2")
+    (pin "H3")
+    (pin "H7")
+    (pin "H8")
+    (pin "H9")
+    (pin "J2")
+    (pin "J8")
+    (pin "K2")
+    (pin "K8")
+    (pin "L2")
+    (pin "L7")
+    (pin "M1")
+    (pin "M9")
+    (pin "N1")
+    (pin "N2")
+    (pin "N3")
+    (pin "N7")
+    (pin "N9")
+    (pin "P1")
+    (pin "P2")
+    (pin "P3")
+    (pin "P7")
+    (pin "P8")
+    (pin "P9")
+    (pin "R1")
+    (pin "R2")
+    (pin "R3")
+    (pin "R7")
+    (pin "R8")
+    (pin "R9")
+    (pin "T1")
+    (pin "T2")
+    (pin "T3")
+    (pin "T7")
+    (pin "T8")
+    (pin "T9")
+    (pin "A2")
+    (pin "A3")
+    (pin "A7")
+    (pin "B7")
+    (pin "B8")
+    (pin "C2")
+    (pin "C3")
+    (pin "C7")
+    (pin "C8")
+    (pin "D3")
+    (pin "D7")
+    (pin "E7")
+    (pin "F3")
+    (pin "G3")
+    (pin "J1")
+    (pin "J3")
+    (pin "J7")
+    (pin "J9")
+    (pin "K1")
+    (pin "K3")
+    (pin "K7")
+    (pin "K9")
+    (pin "L1")
+    (pin "L3")
+    (pin "L8")
+    (pin "L9")
+    (pin "M2")
+    (pin "M3")
+    (pin "M7")
+    (pin "M8")
+    (pin "N8")
+    (instances
+      (project "mcump151"
+        (path "/45483761-40cc-431f-bcc2-65a9a869d9c1"
+          (reference "U2") (unit 1)
+        )
+      )
