File: mcustm32mp151/mcustm32mp151.kicad_sch (KiCad schematic)
At the start: 7 parts, among them J1 STM32WORLD_BOARD, J2 STM32WORLD_CONNECTOR_1, J3 STM32WORLD_CONNECTOR_2, J4 USB_C_Receptacle_USB2.0, J5 USB_C_Receptacle_USB2.0, U1 STM32MP151AACx, U2 AS4C256M16D3

Commit message: Hmmmm
Parts:
- U1: footprint Package_BGA:ST_TFBGA-361_12x12mm_Layout23x23_P0.5mmP0.65mm -> stm32world:ST_TFBGA-361_12x12mm_Layout23x23_P0.5mmP0.65mm
Changed lines of the file:
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@@
     (pin "S1")
     (instances
-      (project "mcump151"
+      (project "mcustm32mp151"
         (path "/45483761-40cc-431f-bcc2-65a9a869d9c1"
           (reference "J4") (unit 1)
@@
     (pin "9")
     (instances
-      (project "mcump151"
+      (project "mcustm32mp151"
         (path "/45483761-40cc-431f-bcc2-65a9a869d9c1"
           (reference "J3") (unit 1)
@@
     )
     (instances
-      (project "mcump151"
+      (project "mcustm32mp151"
         (path "/45483761-40cc-431f-bcc2-65a9a869d9c1"
           (reference "J1") (unit 1)
@@
       (effects (font (size 1.27 1.27)) (justify left))
     )
-    (property "Footprint" "Package_BGA:ST_TFBGA-361_12x12mm_Layout23x23_P0.5mmP0.65mm" (at 215.9 384.81 0)
+    (property "Footprint" "stm32world:ST_TFBGA-361_12x12mm_Layout23x23_P0.5mmP0.65mm" (at 215.9 384.81 0)
       (effects (font (size 1.27 1.27)) (justify right) hide)
     )
@@
     (pin "Y9")
     (instances
-      (project "mcump151"
+      (project "mcustm32mp151"
         (path "/45483761-40cc-431f-bcc2-65a9a869d9c1"
           (reference "U1") (unit 1)
@@
     (pin "S1")
     (instances
-      (project "mcump151"
+      (project "mcustm32mp151"
         (path "/45483761-40cc-431f-bcc2-65a9a869d9c1"
           (reference "J5") (unit 1)
@@
     (pin "N8")
     (instances
-      (project "mcump151"
+      (project "mcustm32mp151"
         (path "/45483761-40cc-431f-bcc2-65a9a869d9c1"
           (reference "U2") (unit 1)
@@
     (pin "1")
     (instances
-      (project "mcump151"
+      (project "mcustm32mp151"
         (path "/45483761-40cc-431f-bcc2-65a9a869d9c1"
           (reference "#PWR01") (unit 1)
@@
     (pin "9")
     (instances
-      (project "mcump151"
+      (project "mcustm32mp151"
         (path "/45483761-40cc-431f-bcc2-65a9a869d9c1"
           (reference "J2") (unit 1)
