File: proto/proto.kicad_sch (KiCad schematic)
At the start: 307 parts, among them J1 STM32WORLD_CONNECTOR_2, J2 STM32WORLD_CONNECTOR_1, J3 STM32WORLD_BOARD

Commit message: mem24cxx ready
Parts:
- renumbered J2 to J1, J1 to J2
Other:
- company: (none) -> ${COMPANY}
- title: (none) -> ${TITLE}
- moved on the sheet: J1, J2, TP1, TP10, TP100, TP101, TP102, TP103, TP104, TP105, TP106, TP107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
