File: mem24cxx/mem24cxx.kicad_pcb (KiCad board)
At the start: 2 copper layers, 76.2 x 50.8 mm, 22 parts, among them J1 STM32WORLD_CONNECTOR_1, J2 STM32WORLD_CONNECTOR_2, J3 STM32WORLD_BASE, U1 M24M01, U2 M24M01, U3 M24M01, U4 M24M01

Commit message: Wired B0 to PC15 so it can be read
Parts:
- J3: value STM32WORLD_BASE -> STM32WORLD_BOARD
Changed lines of the file:
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@@
         (effects (font (size 1 1) (thickness 0.15)))
     )
-    (fp_text value "STM32WORLD_BASE" (at 0 26.67) (layer "F.Fab")
+    (fp_text value "STM32WORLD_BOARD" (at 0 26.67) (layer "F.Fab")
         (effects (font (size 1 1) (thickness 0.15)))
     )
