File: can/can.kicad_sch (KiCad schematic)
At the start: 8 parts, among them J1 STM32WORLD_BOARD, J2 STM32WORLD_CONNECTOR_1, J3 STM32WORLD_CONNECTOR_2, U1 SN65HVD230DR, U2 SN65HVD230DR

Commit message: fixed label
Parts:
- added J5: ~, TerminalBlock_4Ucon:TerminalBlock_4Ucon_1x02_P3.50mm_Horizontal, symbol Connector_Generic:Conn_01x02
- added JP3, JP4, JP5, JP6, JP7, JP8: ~, Jumper:SolderJumper-2_P1.3mm_Open_TrianglePad1.0x1.5mm, symbol Jumper:Jumper_2_Open
Connections:
- net at JP1.1 (A), U1.1 (D): now also JP3.1 (A)
- net at JP2.1 (A), U1.4 (R): now also JP4.1 (A)
- net at U1.6 (CANL): now also J4.2 (Pin_2)
- net at U1.7 (CANH): now also J4.1 (Pin_1)
- net at U2.1 (D): now also JP5.1 (A), JP7.1 (A)
- net at U2.4 (R): now also JP6.1 (A), JP8.1 (A)
- net at U2.6 (CANL): now also J5.2 (Pin_2)
- net at U2.7 (CANH): now also J5.1 (Pin_1)
Other:
- moved on the sheet: J4

Commit message: Hmmmm
Parts:
- added C1, C2: 100nF, Capacitor_SMD:C_0603_1608Metric, symbol Device:C
- added JP10, JP9: ~, Jumper:SolderJumper-2_P1.3mm_Open_TrianglePad1.0x1.5mm, symbol Jumper:Jumper_2_Open
- added R1, R2: 120R, Resistor_SMD:R_0603_1608Metric, symbol Device:R
- J4, J5: footprint TerminalBlock_4Ucon:TerminalBlock_4Ucon_1x02_P3.50mm_Horizontal -> TerminalBlock_Phoenix:TerminalBlock_Phoenix_PT-1,5-2-5.0-H_1x02_P5.00mm_Horizontal
Connections:
- net +3V3: now also C1.1, C2.1
- net GND: now also U1.8 (Rs), U2.8 (Rs), C1.2, C2.2
- net CAN1D: now reaches JP1.1 (A), JP3.1 (A), U1.1 (D)
- net CAN1R: now reaches JP2.1 (A), JP4.1 (A), U1.4 (R)
- net CAN1H: now reaches J4.2 (Pin_2)
- net CAN1H: now also U1.7 (CANH), JP9.2 (B); no longer U1.6 (CANL)
- net CAN1L: now reaches J4.1 (Pin_1)
- net CAN1L: now also U1.6 (CANL), R1.2; no longer U1.7 (CANH)
- net CAN1_RX: now reaches J3.11 (PA11)
- net CAN1_RX: now also JP2.2 (B)
- net CAN1_TX: now reaches J3.14 (PA12)
- net CAN1_TX: now also JP1.2 (B)
- net CAN2_RX_A: now reaches J3.25 (PB5)
- net CAN2_RX_A: now also JP8.2 (B)
- net CAN2_TX_A: now reaches J3.28 (PB6)
- net CAN2_TX_A: now also JP7.2 (B)
- net CAN1_TX_A: now reaches J3.29 (PB9)
- net CAN1_TX_A: now also JP3.2 (B)
- net CAN1_RX_A: now reaches J3.30 (PB8)
- net CAN1_RX_A: now also JP4.2 (B)
- net CAN2R: now reaches JP6.1 (A), JP8.1 (A), U2.4 (R)
- net CAN2D: now reaches JP5.1 (A), JP7.1 (A), U2.1 (D)
- net CAN2H: now reaches J5.2 (Pin_2)
- net CAN2H: now also U2.7 (CANH), JP10.2 (B); no longer U2.6 (CANL)
- net CAN2L: now reaches J5.1 (Pin_1)
- net CAN2L: now also U2.6 (CANL), R2.2; no longer U2.7 (CANH)
- net CAN2_TX: now reaches J2.25 (PB13)
- net CAN2_TX: now also JP5.2 (B)
- net CAN2_RX: now reaches J2.26 (PB12)
- net CAN2_RX: now also JP6.2 (B)
- new net: JP9.1 (A), R1.1
- new net: JP10.1 (A), R2.1
Other:
- moved on the sheet: J4, J5, JP1, JP2, JP3, JP4, JP5, JP6, JP7, JP8, U1, U2
