File: can/can.kicad_pcb (KiCad board)
At the start: 2 copper layers, 76.2 x 50.8 mm, 6 parts, among them J1 STM32WORLD_BOARD, J2 STM32WORLD_CONNECTOR_1, J3 STM32WORLD_CONNECTOR_2, U1 SN65HVD230DR, U2 SN65HVD230DR

Commit message: fixed label
Parts:
- added JP1: ~, Jumper:SolderJumper-2_P1.3mm_Open_TrianglePad1.0x1.5mm, F.Cu at (136.1, 91.9)
- added JP2: ~, Jumper:SolderJumper-2_P1.3mm_Open_TrianglePad1.0x1.5mm, F.Cu at (136.1, 95.5)
- added JP3: ~, Jumper:SolderJumper-2_P1.3mm_Open_TrianglePad1.0x1.5mm, F.Cu at (136.1, 99.0)
- added JP4: ~, Jumper:SolderJumper-2_P1.3mm_Open_TrianglePad1.0x1.5mm, F.Cu at (136.1, 102.5)
- added JP5: ~, Jumper:SolderJumper-2_P1.3mm_Open_TrianglePad1.0x1.5mm, F.Cu at (136.1, 106.1)
- added JP6: ~, Jumper:SolderJumper-2_P1.3mm_Open_TrianglePad1.0x1.5mm, F.Cu at (140.4, 91.9)
- added JP7: ~, Jumper:SolderJumper-2_P1.3mm_Open_TrianglePad1.0x1.5mm, F.Cu at (140.4, 95.5)
- added JP8: ~, Jumper:SolderJumper-2_P1.3mm_Open_TrianglePad1.0x1.5mm, F.Cu at (140.4, 99.0)
Connections:
- U1 pad 1: unconnected-(U1-D-Pad1) -> Net-(JP1-A)
- U1 pad 4: unconnected-(U1-R-Pad4) -> Net-(JP2-A)

Commit message: Hmmmm
Parts:
- added C1: 100nF, Capacitor_SMD:C_0603_1608Metric, F.Cu at (160.7, 91.4)
- added C2: 100nF, Capacitor_SMD:C_0603_1608Metric, F.Cu at (160.7, 105.4)
- added J5: ~, TerminalBlock_Phoenix:TerminalBlock_Phoenix_PT-1,5-2-5.0-H_1x02_P5.00mm_Horizontal, F.Cu at (181.6, 109.8)
- added JP10: ~, Jumper:SolderJumper-2_P1.3mm_Open_TrianglePad1.0x1.5mm, F.Cu at (172.7, 104.1)
- added JP9: ~, Jumper:SolderJumper-2_P1.3mm_Open_TrianglePad1.0x1.5mm, F.Cu at (172.7, 90.2)
- added R1: 120R, Resistor_SMD:R_0603_1608Metric, F.Cu at (172.7, 92.7)
- added R2: 120R, Resistor_SMD:R_0603_1608Metric, F.Cu at (172.7, 106.7)
- J4: footprint TerminalBlock_4Ucon:TerminalBlock_4Ucon_1x02_P3.50mm_Horizontal -> TerminalBlock_Phoenix:TerminalBlock_Phoenix_PT-1,5-2-5.0-H_1x02_P5.00mm_Horizontal
- moved JP6 17.5 mm to (149.9, 106.7), turned to 180 degrees
- moved JP4 16.9 mm to (149.9, 92.7), turned to 180 degrees
- moved JP2 14.8 mm to (149.9, 90.2), turned to 180 degrees
- moved JP7 12.3 mm to (145.4, 106.7), turned to 180 degrees
- moved JP3 11.3 mm to (145.4, 92.7), turned to 180 degrees
- moved JP8 10.7 mm to (149.9, 104.1), turned to 180 degrees
- moved JP5 9.54 mm to (145.4, 104.1), turned to 180 degrees
- moved JP1 9.50 mm to (145.4, 90.2), turned to 180 degrees
- moved J4 7.28 mm to (181.7, 93.9), turned to 90 degrees
- moved U1 5.72 mm to (165.7, 91.4)
- moved U2 3.43 mm to (165.7, 105.4)
Connections:
- J2 pad 25: unconnected-(J2-PB13-Pad25) -> CAN2_TX
- J2 pad 26: unconnected-(J2-PB12-Pad26) -> CAN2_RX
- J3 pad 11: unconnected-(J3-PA11-Pad11) -> CAN1_RX
- J3 pad 14: unconnected-(J3-PA12-Pad14) -> CAN1_TX
- J3 pad 25: unconnected-(J3-PB5-Pad25) -> CAN2_RX_A
- J3 pad 28: unconnected-(J3-PB6-Pad28) -> CAN2_TX_A
- J3 pad 29: unconnected-(J3-PB9-Pad29) -> CAN1_TX_A
- J3 pad 30: unconnected-(J3-PB8-Pad30) -> CAN1_RX_A
- J4 pad 1: unconnected-(J4-Pin_1-Pad1) -> /CAN1L
- J4 pad 2: unconnected-(J4-Pin_2-Pad2) -> /CAN1H
- JP1 pad 1: Net-(JP1-A) -> /CAN1D
- JP1 pad 2: unconnected-(JP1-B-Pad2) -> CAN1_TX
- JP2 pad 1: Net-(JP2-A) -> /CAN1R
- JP2 pad 2: unconnected-(JP2-B-Pad2) -> CAN1_RX
- JP3 pad 1: unconnected-(JP3-A-Pad1) -> /CAN1D
- JP3 pad 2: unconnected-(JP3-B-Pad2) -> CAN1_TX_A
- JP4 pad 1: unconnected-(JP4-A-Pad1) -> /CAN1R
- JP4 pad 2: unconnected-(JP4-B-Pad2) -> CAN1_RX_A
- JP5 pad 1: unconnected-(JP5-A-Pad1) -> /CAN2D
- JP5 pad 2: unconnected-(JP5-B-Pad2) -> CAN2_TX
- JP6 pad 1: unconnected-(JP6-A-Pad1) -> /CAN2R
- JP6 pad 2: unconnected-(JP6-B-Pad2) -> CAN2_RX
- JP7 pad 1: unconnected-(JP7-A-Pad1) -> /CAN2D
- JP7 pad 2: unconnected-(JP7-B-Pad2) -> CAN2_TX_A
- JP8 pad 1: unconnected-(JP8-A-Pad1) -> /CAN2R
- JP8 pad 2: unconnected-(JP8-B-Pad2) -> CAN2_RX_A
- U1 pad 1: Net-(JP1-A) -> /CAN1D
- U1 pad 4: Net-(JP2-A) -> /CAN1R
- U1 pad 6: unconnected-(U1-CANL-Pad6) -> /CAN1L
- U1 pad 7: unconnected-(U1-CANH-Pad7) -> /CAN1H
- U1 pad 8: unconnected-(U1-Rs-Pad8) -> GND
- U2 pad 1: unconnected-(U2-D-Pad1) -> /CAN2D
- U2 pad 4: unconnected-(U2-R-Pad4) -> /CAN2R
- U2 pad 6: unconnected-(U2-CANL-Pad6) -> /CAN2L
- U2 pad 7: unconnected-(U2-CANH-Pad7) -> /CAN2H
- U2 pad 8: unconnected-(U2-Rs-Pad8) -> GND
Routing:
- net +3V3: track 0.00 -> 58.1 mm
- net CAN2_TX_A: track 0.00 -> 30.4 mm
- net CAN2_RX_A: track 0.00 -> 26.4 mm, vias 0 -> 1
- net /CAN2D: track 0.00 -> 23.0 mm
- net /CAN1D: track 0.00 -> 20.2 mm
- net CAN1_TX: track 0.00 -> 20.2 mm
- net CAN2_TX: track 0.00 -> 19.1 mm, vias 0 -> 1
- net CAN1_RX_A: track 0.00 -> 19.1 mm, vias 0 -> 1
- net CAN1_RX: track 0.00 -> 18.2 mm, vias 0 -> 1
- net /CAN1H: track 0.00 -> 15.8 mm
- net CAN2_RX: track 0.00 -> 15.6 mm
- net /CAN2L: track 0.00 -> 15.6 mm
- net /CAN2R: track 0.00 -> 15.5 mm
- net /CAN1R: track 0.00 -> 15.5 mm
- net /CAN2H: track 0.00 -> 15.4 mm
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- added copper zone on B.Cu, net GND
- added copper zone on F.Cu, net GND
Other:
- board text added: "ALT"
- board text added: "CAN1"
- board text added: "CAN2"

Commit message: Ordering can rev_a
Routing:
- net +3V3: track 58.1 -> 69.0 mm, vias 0 -> 2
- net CAN2_RX_A: track 26.4 -> 26.9 mm
Changed lines of the file:
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@@
       (layer "F.SilkS" (type "Top Silk Screen"))
       (layer "F.Paste" (type "Top Solder Paste"))
-      (layer "F.Mask" (type "Top Solder Mask") (thickness 0.01))
+      (layer "F.Mask" (type "Top Solder Mask") (color "Green") (thickness 0.01))
       (layer "F.Cu" (type "copper") (thickness 0.035))
       (layer "dielectric 1" (type "core") (thickness 1.11) (material "FR4") (epsilon_r 4.5) (loss_tangent 0.02))
       (layer "B.Cu" (type "copper") (thickness 0.035))
-      (layer "B.Mask" (type "Bottom Solder Mask") (thickness 0.01))
+      (layer "B.Mask" (type "Bottom Solder Mask") (color "Green") (thickness 0.01))
       (layer "B.Paste" (type "Bottom Solder Paste"))
       (layer "B.SilkS" (type "Bottom Silk Screen"))
@@
       (disableapertmacros false)
       (usegerberextensions false)
-      (usegerberattributes true)
+      (usegerberattributes false)
       (usegerberadvancedattributes true)
       (creategerberjobfile true)
@@
       (viasonmask false)
       (mode 1)
-      (useauxorigin false)
+      (useauxorigin true)
       (hpglpennumber 1)
       (hpglpenspeed 20)
@@
       (outputformat 1)
       (mirror false)
-      (drillshape 1)
+      (drillshape 0)
       (scaleselection 1)
-      (outputdirectory "")
+      (outputdirectory "rev_a/")
     )
   )
@@
   (segment (start 155.0933 116.377447) (end 155.0933 118.2633) (width 0.2286) (layer "F.Cu") (net 26))
   (segment (start 163.26 92.075) (end 164.234999 92.075) (width 0.2286) (layer "F.Cu") (net 37))
-  (segment (start 164.465 92.075) (end 165.916729 90.623271) (width 0.2286) (layer "F.Cu") (net 37))
-  (segment (start 170.3333 116.377447) (end 170.3333 118.2633) (width 0.2286) (layer "F.Cu") (net 37))
-  (segment (start 170.0267 80.1633) (end 170.0267 85.606758) (width 0.2286) (layer "F.Cu") (net 37))
-  (segment (start 164.234999 106.045) (end 163.26 106.045) (width 0.2286) (layer "F.Cu") (net 37))
-  (segment (start 163.26 92.075) (end 164.465 92.075) (width 0.2286) (layer "F.Cu") (net 37))
-  (segment (start 164.234999 92.075) (end 165.735 93.575001) (width 0.2286) (layer "F.Cu") (net 37))
-  (segment (start 171.45 78.74) (end 170.0267 80.1633) (width 0.2286) (layer "F.Cu") (net 37))
+  (segment (start 167.005 108.585) (end 172.6048 108.585) (width 0.3048) (layer "F.Cu") (net 37))
+  (segment (start 163.26 106.045) (end 164.465 106.045) (width 0.3048) (layer "F.Cu") (net 37))
+  (segment (start 164.465 106.045) (end 167.005 108.585) (width 0.3048) (layer "F.Cu") (net 37))
   (segment (start 160.795 106.045) (end 160.655 106.185) (width 0.2286) (layer "F.Cu") (net 37))
-  (segment (start 164.5017 111.7967) (end 165.735 113.03) (width 0.2286) (layer "F.Cu") (net 37))
+  (segment (start 167.64 95.25) (end 172.6048 95.25) (width 0.3048) (layer "F.Cu") (net 37))
   (segment (start 163.26 106.045) (end 160.795 106.045) (width 0.2286) (layer "F.Cu") (net 37))
   (segment (start 163.26 92.075) (end 160.795 92.075) (width 0.2286) (layer "F.Cu") (net 37))
-  (segment (start 165.735 93.575001) (end 165.735 104.544999) (width 0.2286) (layer "F.Cu") (net 37))
   (segment (start 160.795 92.075) (end 160.655 92.215) (width 0.2286) (layer "F.Cu") (net 37))
-  (segment (start 165.735 113.03) (end 166.985853 113.03) (width 0.2286) (layer "F.Cu") (net 37))
-  (segment (start 164.465 106.045) (end 164.5017 106.0817) (width 0.2286) (layer "F.Cu") (net 37))
-  (segment (start 165.916729 90.623271) (end 165.916729 89.716729) (width 0.2286) (layer "F.Cu") (net 37))
-  (segment (start 163.26 106.045) (end 164.465 106.045) (width 0.2286) (layer "F.Cu") (net 37))
-  (segment (start 170.3333 118.2633) (end 171.45 119.38) (width 0.2286) (layer "F.Cu") (net 37))
-  (segment (start 165.735 104.544999) (end 164.234999 106.045) (width 0.2286) (layer "F.Cu") (net 37))
-  (segment (start 170.0267 85.606758) (end 165.916729 89.716729) (width 0.2286) (layer "F.Cu") (net 37))
-  (segment (start 164.5017 106.0817) (end 164.5017 111.7967) (width 0.2286) (layer "F.Cu") (net 37))
-  (segment (start 166.985853 113.03) (end 170.3333 116.377447) (width 0.2286) (layer "F.Cu") (net 37))
+  (segment (start 163.26 92.075) (end 164.465 92.075) (width 0.3048) (layer "F.Cu") (net 37))
+  (segment (start 164.465 92.075) (end 167.64 95.25) (width 0.3048) (layer "F.Cu") (net 37))
+  (via (at 172.6048 108.585) (size 0.7) (drill 0.35) (layers "F.Cu" "B.Cu") (net 37))
+  (via (at 172.6048 95.25) (size 0.7) (drill 0.35) (layers "F.Cu" "B.Cu") (net 37))
+  (segment (start 172.6048 95.25) (end 172.6048 108.585) (width 0.3048) (layer "B.Cu") (net 37))
+  (segment (start 171.45 78.74) (end 172.6048 79.8948) (width 0.3048) (layer "B.Cu") (net 37))
+  (segment (start 172.6048 108.585) (end 172.6048 118.2252) (width 0.3048) (layer "B.Cu") (net 37))
+  (segment (start 172.6048 79.8948) (end 172.6048 95.25) (width 0.3048) (layer "B.Cu") (net 37))
+  (segment (start 172.6048 118.2252) (end 171.45 119.38) (width 0.3048) (layer "B.Cu") (net 37))
   (segment (start 149.135 90.17) (end 147.955 90.17) (width 0.2286) (layer "F.Cu") (net 38))
   (via locked (at 147.955 90.17) (size 0.7) (drill 0.35) (layers "F.Cu" "B.Cu") (net 38))
@@
   (segment (start 149.135 104.14) (end 147.955 104.14) (width 0.2286) (layer "F.Cu") (net 42))
   (via (at 147.955 104.14) (size 0.7) (drill 0.35) (layers "F.Cu" "B.Cu") (net 42))
-  (segment (start 148.5717 91.658846) (end 146.05 89.137146) (width 0.2286) (layer "B.Cu") (net 42))
-  (segment (start 148.5717 96.5383) (end 148.5717 91.658846) (width 0.2286) (layer "B.Cu") (net 42))
-  (segment (start 147.955 104.14) (end 147.955 97.155) (width 0.2286) (layer "B.Cu") (net 42))
-  (segment (start 146.05 89.137146) (end 146.05 83.82) (width 0.2286) (layer "B.Cu") (net 42))
-  (segment (start 146.05 83.82) (end 143.51 81.28) (width 0.2286) (layer "B.Cu") (net 42))
-  (segment (start 147.955 97.155) (end 148.5717 96.5383) (width 0.2286) (layer "B.Cu") (net 42))
+  (segment (start 149.225 92.312146) (end 149.225 95.885) (width 0.2286) (layer "B.Cu") (net 42))
+  (segment (start 146.05 89.137146) (end 149.225 92.312146) (width 0.2286) (layer "B.Cu") (net 42))
+  (segment (start 143.51 81.28) (end 146.05 83.82) (width 0.2286) (layer "B.Cu") (net 42))
+  (segment (start 149.225 95.885) (end 147.955 97.155) (width 0.2286) (layer "B.Cu") (net 42))
+  (segment (start 146.05 83.82) (end 146.05 89.137146) (width 0.2286) (layer "B.Cu") (net 42))
+  (segment (start 147.955 97.155) (end 147.955 104.14) (width 0.2286) (layer "B.Cu") (net 42))
   (segment (start 139.8533 79.8567) (end 140.97 78.74) (width 0.2286) (layer "F.Cu") (net 50))
   (segment (start 144.69 106.68) (end 139.8533 101.8433) (width 0.2286) (layer "F.Cu") (net 50))

Commit message: Hmmmm
Routing:
- net /CAN2D: track 23.0 -> 22.3 mm
- net GND: vias 0 -> 12
Changed lines of the file:
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@@
   (property "AUTHOR_EMAIL" "lbthomsen@gmail.com")
   (property "COMPANY" "stm32world")
-  (property "REVISION" "a")
+  (property "REVISION" "b")
   (property "TITLE" "can")
-  (property "URL" "https://stm32world.com/wiki/CAN")
+  (property "URL" "https://stm32world.com/wiki/CANTRANS")
   (net 0 "")
   (net 1 "GND")
@@
     (effects (font (size 1 1) (thickness 0.15)) (justify right bottom))
   )
+  (via (at 156.21 91.44) (size 0.7) (drill 0.35) (layers "F.Cu" "B.Cu") (free) (net 1))
+  (via (at 175.26 105.41) (size 0.7) (drill 0.35) (layers "F.Cu" "B.Cu") (free) (net 1))
+  (via (at 181.61 100.965) (size 0.7) (drill 0.35) (layers "F.Cu" "B.Cu") (free) (net 1))
+  (via (at 158.115 91.44) (size 0.7) (drill 0.35) (layers "F.Cu" "B.Cu") (free) (net 1))
+  (via (at 156.21 105.41) (size 0.7) (drill 0.35) (layers "F.Cu" "B.Cu") (free) (net 1))
+  (via (at 158.115 105.41) (size 0.7) (drill 0.35) (layers "F.Cu" "B.Cu") (free) (net 1))
+  (via (at 165.735 105.41) (size 0.7) (drill 0.35) (layers "F.Cu" "B.Cu") (free) (net 1))
+  (via (at 181.61 85.09) (size 0.7) (drill 0.35) (layers "F.Cu" "B.Cu") (free) (net 1))
+  (via (at 165.735 91.44) (size 0.7) (drill 0.35) (layers "F.Cu" "B.Cu") (free) (net 1))
+  (via (at 181.61 113.665) (size 0.7) (drill 0.35) (layers "F.Cu" "B.Cu") (free) (net 1))
+  (via (at 175.26 91.44) (size 0.7) (drill 0.35) (layers "F.Cu" "B.Cu") (free) (net 1))
+  (via (at 181.61 97.79) (size 0.7) (drill 0.35) (layers "F.Cu" "B.Cu") (free) (net 1))
   (segment (start 144.69 104.14) (end 143.51 104.14) (width 0.2286) (layer "F.Cu") (net 25))
   (via (at 143.51 104.14) (size 0.7) (drill 0.35) (layers "F.Cu" "B.Cu") (net 25))
@@
   (segment (start 173.445 104.14) (end 177.8 104.14) (width 0.2286) (layer "F.Cu") (net 81))
   (segment (start 173.445 103.39) (end 172.9933 102.9383) (width 0.2286) (layer "F.Cu") (net 81))
+  (segment (start 156.5917 89.535) (end 156.21 89.1533) (width 0.2286) (layer "F.Cu") (net 82))
   (segment (start 146.14 90.17) (end 146.14 92.71) (width 0.2286) (layer "F.Cu") (net 82))
+  (segment (start 163.26 89.535) (end 156.5917 89.535) (width 0.2286) (layer "F.Cu") (net 82))
+  (segment (start 156.21 89.1533) (end 147.1567 89.1533) (width 0.2286) (layer "F.Cu") (net 82))
   (segment (start 147.1567 89.1533) (end 146.14 90.17) (width 0.2286) (layer "F.Cu") (net 82))
-  (segment (start 162.8783 89.1533) (end 147.1567 89.1533) (width 0.2286) (layer "F.Cu") (net 82))
-  (segment (start 163.26 89.535) (end 162.8783 89.1533) (width 0.2286) (layer "F.Cu") (net 82))
   (segment (start 150.585 92.71) (end 150.585 90.17) (width 0.2286) (layer "F.Cu") (net 83))
   (segment (start 163.26 93.345) (end 151.22 93.345) (width 0.2286) (layer "F.Cu") (net 83))
   (segment (start 151.22 93.345) (end 150.585 92.71) (width 0.2286) (layer "F.Cu") (net 83))
   (segment (start 146.14 102.78) (end 147.32 101.6) (width 0.2286) (layer "F.Cu") (net 84))
-  (segment (start 147.32 101.6) (end 162.56 101.6) (width 0.2286) (layer "F.Cu") (net 84))
+  (segment (start 163.26 103.505) (end 158.115 103.505) (width 0.2286) (layer "F.Cu") (net 84))
+  (segment (start 158.115 103.505) (end 156.21 101.6) (width 0.2286) (layer "F.Cu") (net 84))
   (segment (start 146.14 104.14) (end 146.14 106.68) (width 0.2286) (layer "F.Cu") (net 84))
-  (segment (start 162.56 101.6) (end 163.26 102.3) (width 0.2286) (layer "F.Cu") (net 84))
   (segment (start 146.14 104.14) (end 146.14 102.78) (width 0.2286) (layer "F.Cu") (net 84))
-  (segment (start 163.26 102.3) (end 163.26 103.505) (width 0.2286) (layer "F.Cu") (net 84))
+  (segment (start 147.32 101.6) (end 156.21 101.6) (width 0.2286) (layer "F.Cu") (net 84))
   (segment (start 151.22 107.315) (end 150.585 106.68) (width 0.2286) (layer "F.Cu") (net 85))
   (segment (start 163.26 107.315) (end 151.22 107.315) (width 0.2286) (layer "F.Cu") (net 85))
