File: ws2812/ws2812.kicad_sch (KiCad schematic)
At the start: 8 parts, among them J1 STM32WORLD_BOARD, J2 STM32WORLD_CONNECTOR_1, J3 STM32WORLD_CONNECTOR_2, U1 WS2812E, U2 WS2812E, U3 WS2812E, U4 WS2812E, U5 WS2812E

Commit message: Hmmmm
Parts:
- added U10, U11, U12, U13, U14, U15, U16, U17, U18, U19, U20, U6, U7, U8, U9: WS2812E, stm32world:LED-SMD_4P-L3.7-W3.5-P1.75-BR-SK6812MINI, symbol stm32world:WS2812E-MINI-X1
Connections:
- net at U4.1 (DI): now also U3.3 (DO)
- net VCC: now reaches U4.2 (VDD)
- net VCC: now also U1.2 (VDD), U2.2 (VDD), U3.2 (VDD), U5.2 (VDD), U10.2 (VDD), U11.2 (VDD), U12.2 (VDD), U13.2 (VDD), U14.2 (VDD), U15.2 (VDD), U16.2 (VDD), U17.2 (VDD), U18.2 (VDD), U19.2 (VDD), U20.2 (VDD), U6.2 (VDD), U7.2 (VDD), U8.2 (VDD), U9.2 (VDD)
- net at U4.3 (DO): now also U5.1 (DI)
- net GND: now reaches U4.4 (GND)
- net GND: now also U1.4 (GND), U2.4 (GND), U3.4 (GND), U5.4 (GND), U10.4 (GND), U11.4 (GND), U12.4 (GND), U13.4 (GND), U14.4 (GND), U15.4 (GND), U16.4 (GND), U17.4 (GND), U18.4 (GND), U19.4 (GND), U20.4 (GND), U6.4 (GND), U7.4 (GND), U8.4 (GND), U9.4 (GND)
- net at U2.1 (DI): now also U1.3 (DO)
- net at U2.3 (DO): now also U3.1 (DI)
- net at U5.3 (DO): now also U6.1 (DI)
- new net: U6.3 (DO), U7.1 (DI)
- new net: U7.3 (DO), U8.1 (DI)
- new net: U12.3 (DO), U13.1 (DI)
- new net: U13.3 (DO), U14.1 (DI)
- new net: U15.3 (DO), U16.1 (DI)
- new net: U16.3 (DO), U17.1 (DI)
- new net: U8.3 (DO), U9.1 (DI)
- new net: U19.3 (DO), U20.1 (DI)
- new net: U14.3 (DO), U15.1 (DI)
- new net: U17.3 (DO), U18.1 (DI)
- new net: U18.3 (DO), U19.1 (DI)
- new net: U11.3 (DO), U12.1 (DI)
- new net: U10.1 (DI), U9.3 (DO)
Other:
- moved on the sheet: U1, U2, U3, U4, U5

Commit message: More
Parts:
- added JP1: ~, Jumper:SolderJumper-3_P1.3mm_Bridged2Bar12_RoundedPad1.0x1.5mm, symbol Jumper:SolderJumper_3_Bridged12
- added JP2, JP3, JP4, JP5: ~, Jumper:SolderJumper-2_P1.3mm_Open_RoundedPad1.0x1.5mm, symbol Jumper:SolderJumper_2_Open
- added U21, U22, U23, U24, U25, U26, U27, U28, U29, U30, U31, U32, U33, U34, U35, U36, U37, U38, U39, U40, U41, U42, U43, U44, U45, U46, U47, U48, U49, U50: WS2812E, stm32world:LED-SMD_4P-L3.7-W3.5-P1.75-BR-SK6812MINI, symbol stm32world:WS2812E-MINI-X1
Connections:
- net GND: now also J2.1 (GND), J2.37 (GND), J2.39 (GND), J3.1 (GND), J3.3 (GND), U21.4 (GND), U22.4 (GND), U23.4 (GND), U24.4 (GND), U25.4 (GND), U26.4 (GND), U27.4 (GND), U28.4 (GND), U29.4 (GND), U30.4 (GND), U31.4 (GND), U32.4 (GND), U33.4 (GND), U34.4 (GND), U35.4 (GND), U36.4 (GND), U37.4 (GND), U38.4 (GND), U39.4 (GND), U40.4 (GND), U41.4 (GND), U42.4 (GND), U43.4 (GND), U44.4 (GND), U45.4 (GND), U46.4 (GND), U47.4 (GND), U48.4 (GND), U49.4 (GND), U50.4 (GND)
- net VCC: now also JP1.2 (C), U21.2 (VDD), U22.2 (VDD), U23.2 (VDD), U24.2 (VDD), U25.2 (VDD), U26.2 (VDD), U27.2 (VDD), U28.2 (VDD), U29.2 (VDD), U30.2 (VDD), U31.2 (VDD), U32.2 (VDD), U33.2 (VDD), U34.2 (VDD), U35.2 (VDD), U36.2 (VDD), U37.2 (VDD), U38.2 (VDD), U39.2 (VDD), U40.2 (VDD), U41.2 (VDD), U42.2 (VDD), U43.2 (VDD), U44.2 (VDD), U45.2 (VDD), U46.2 (VDD), U47.2 (VDD), U48.2 (VDD), U49.2 (VDD), U50.2 (VDD)
- net TIM5_1: now reaches J2.10 (PA0)
- net TIM5_1: now also JP2.1 (A)
- net TIM5_4: now reaches J2.11 (PA3)
- net TIM5_4: now also JP5.1 (A)
- net TIM5_3: now reaches J2.12 (PA2)
- net TIM5_3: now also JP4.1 (A)
- net +3.3V: now reaches J2.38 (3.3V)
- net +3.3V: now also J3.4 (3.3V), JP1.3 (B)
- net +5V: now reaches J2.40 (5V)
- net +5V: now also J3.2 (5V), JP1.1 (A)
- net TIM5_2: now reaches J2.9 (PA1)
- net TIM5_2: now also JP3.1 (A)
- net at U20.3 (DO): now also U21.1 (DI)
- net LED: now reaches U1.1 (DI)
- net LED: now also JP2.2 (B), JP3.2 (B), JP4.2 (B), JP5.2 (B)
- net at U11.1 (DI): now also U10.3 (DO)
- new net: U28.3 (DO), U29.1 (DI)
- new net: U29.3 (DO), U30.1 (DI)
- new net: U34.3 (DO), U35.1 (DI)
- new net: U35.3 (DO), U36.1 (DI)
- new net: U25.3 (DO), U26.1 (DI)
- new net: U26.3 (DO), U27.1 (DI)
- new net: U42.3 (DO), U43.1 (DI)
- new net: U43.3 (DO), U44.1 (DI)
- new net: U47.3 (DO), U48.1 (DI)
- new net: U48.3 (DO), U49.1 (DI)
- new net: U30.3 (DO), U31.1 (DI)
- new net: U31.3 (DO), U32.1 (DI)
- new net: U40.3 (DO), U41.1 (DI)
- new net: U41.3 (DO), U42.1 (DI)
- new net: U32.3 (DO), U33.1 (DI)
- new net: U38.3 (DO), U39.1 (DI)
- new net: U39.3 (DO), U40.1 (DI)
- new net: U49.3 (DO), U50.1 (DI)
- new net: U21.3 (DO), U22.1 (DI)
- new net: U22.3 (DO), U23.1 (DI)
- new net: U37.3 (DO), U38.1 (DI)
- new net: U23.3 (DO), U24.1 (DI)
- new net: U24.3 (DO), U25.1 (DI)
- new net: U45.3 (DO), U46.1 (DI)
- new net: U46.3 (DO), U47.1 (DI)
- new net: U44.3 (DO), U45.1 (DI)
- new net: U33.3 (DO), U34.1 (DI)
- new net: U36.3 (DO), U37.1 (DI)
- new net: U27.3 (DO), U28.1 (DI)
Other:
- moved on the sheet: J2, J3, U1, U10, U11, U12, U13, U14, U15, U16, U17, U18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

Commit message: Hmmm
Parts:
- added JP10, JP11, JP12, JP13, JP14, JP15, JP16, JP17, JP18, JP19, JP20, JP21, JP6, JP7, JP8, JP9: ~, Jumper:SolderJumper-2_P1.3mm_Open_RoundedPad1.0x1.5mm, symbol Jumper:SolderJumper_2_Open
Connections:
- net LED: now also JP10.2 (B), JP11.2 (B), JP12.2 (B), JP13.2 (B), JP14.2 (B), JP15.2 (B), JP16.2 (B), JP17.2 (B), JP18.2 (B), JP19.2 (B), JP20.2 (B), JP21.2 (B), JP6.2 (B), JP7.2 (B), JP8.2 (B), JP9.2 (B)
- net TIM2_4: now reaches J2.23 (PB11)
- net TIM2_4: now also JP15.1 (A)
- net TIM2_3: now reaches J2.24 (PB10)
- net TIM2_3: now also JP14.1 (A)
- net TIM3_2: now reaches J2.29 (PC7)
- net TIM3_2: now also JP7.1 (A)
- net TIM3_1: now reaches J2.30 (PC6)
- net TIM3_1: now also JP6.1 (A)
- net TIM3_4: now reaches J2.31 (PC9)
- net TIM3_4: now also JP17.1 (A)
- net TIM3_3: now reaches J2.32 (PC8)
- net TIM3_3: now also JP16.1 (A)
- net TIM1_1: now reaches J3.10 (PA8)
- net TIM1_1: now also JP8.1 (A)
- net TIM1_4: now reaches J3.11 (PA11)
- net TIM1_4: now also JP11.1 (A)
- net TIM1_3: now reaches J3.12 (PA10)
- net TIM1_3: now also JP10.1 (A)
- net TIM2_1: now reaches J3.15 (PA15)
- net TIM2_1: now also JP12.1 (A)
- net TIM2_2: now reaches J3.23 (PB3)
- net TIM2_2: now also JP13.1 (A)
- net TIM4_2: now reaches J3.27 (PB7)
- net TIM4_2: now also JP19.1 (A)
- net TIM4_1: now reaches J3.28 (PB6)
- net TIM4_1: now also JP18.1 (A)
- net TIM4_4: now reaches J3.29 (PB9)
- net TIM4_4: now also JP21.1 (A)
- net TIM4_3: now reaches J3.30 (PB8)
- net TIM4_3: now also JP20.1 (A)
- net TIM1_2: now reaches J3.9 (PA9)
- net TIM1_2: now also JP9.1 (A)
Other:
- moved on the sheet: JP1, JP2, JP3, JP4, JP5
