File: mcustm32f402/mcustm32f402.kicad_sch (KiCad schematic)
At the start: 37 parts, among them J2 STM32WORLD_CONNECTOR_1, J3 STM32WORLD_CONNECTOR_2, J4 STM32WORLD_BOARD, SW1 TS-1088R-02526, SW2 TS-1088R-02526, U1 AMS1117-3.3, U2 STM32F401RCTx, Y1 X_16MHZ

Commit message: Hmmm
Connections:
- net VA: now also U2.13 (VREF+)
Changed lines of the file:
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@@
+	(wire
+		(pts
+			(xy 163.83 50.8) (xy 166.37 50.8)
+		)
+		(stroke
+			(width 0)
+			(type default)
+		)
+	)
 	(wire
 		(pts

Commit message: Hmmm
Parts:
- D2: value ~ -> B5819W
- D3: LCSC C72043 -> C19171301
- D4: LCSC C72041 -> C2288
- J1: value ~ -> TYPE-C-31-M-12
- U2: LCSC (none) -> C2915304
Changed lines of the file:
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@@
 			)
 		)
-		(property "Value" "~"
+		(property "Value" "B5819W"
 			(at 54.61 127.6096 0)
 			(effects
@@
 			)
 		)
-		(property "Datasheet" "~"
+		(property "Datasheet" "https://jlcpcb.com/api/file/downloadByFileSystemAccessId/8579707605708554240"
 			(at 54.61 130.81 0)
 			(effects
@@
 			)
 		)
-		(property "Value" "~"
+		(property "Value" "TYPE-C-31-M-12"
 			(at 30.6578 126.3396 0)
 			(effects
@@
 			)
 		)
-		(property "LCSC" "C72043"
+		(property "LCSC" "C19171301"
 			(at 142.24 163.83 0)
 			(effects
@@
 			)
 		)
-		(property "LCSC" "C72041"
+		(property "LCSC" "C2288"
 			(at 156.21 163.83 0)
 			(effects
@@
 			(at 184.15 81.28 0)
 			(effects
+				(font
+					(size 1.27 1.27)
+				)
+				(hide yes)
+			)
+		)
+		(property "LCSC" "C2915304"
+			(at 184.15 81.28 0)
+			(effects

Commit message: Ready for order
Parts:
- JP3, JP4: value ~ -> SolderJumper_2_Open
- U2: value STM32F401RCTx -> STM32F402RCTx
