File: mcustm32f402/mcustm32f402.kicad_pcb (KiCad board)
At the start: 2 copper layers, 76.2 x 50.8 mm, 37 parts, among them J2 STM32WORLD_CONNECTOR_1, J3 STM32WORLD_CONNECTOR_2, J4 STM32WORLD_BOARD, SW1 TS-1088R-02526, SW2 TS-1088R-02526, U1 AMS1117-3.3, U2 STM32F401RCTx, Y1 X_16MHZ

Commit message: Hmmm
Connections:
- U2 pad 13: unconnected-(U2-VREF+-Pad13) -> VA
Routing:
- net VA: track 2.05 -> 7.93 mm
- net BO0: vias 3 -> 4
Changed lines of the file:
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@@
 	(net 83 "HNRST")
 	(net 84 "HBO0")
-	(net 85 "unconnected-(U2-VREF+-Pad13)")
-	(net 86 "unconnected-(J2-PB11-Pad23)")
+	(net 85 "unconnected-(J2-PB11-Pad23)")
 	(footprint "Diode_SMD:D_SOD-123"
 		(layer "F.Cu")
@@
 			(layers "*.Cu" "*.Mask")
 			(remove_unused_layers no)
-			(net 86 "unconnected-(J2-PB11-Pad23)")
+			(net 85 "unconnected-(J2-PB11-Pad23)")
 			(pinfunction "PB11")
 			(pintype "passive+no_connect")
@@
 			(layers "F.Cu" "F.Mask" "F.Paste")
 			(roundrect_rratio 0.25)
-			(net 85 "unconnected-(U2-VREF+-Pad13)")
+			(net 78 "VA")
 			(pinfunction "VREF+")
 			(pintype "input")
@@
 	(segment
 		(start 133.35 83.82)
-		(end 133.35 92.725)
+		(end 133.35 92.71)
 		(width 0.2286)
 		(layer "F.Cu")
@@
 	)
 	(segment
-		(start 142.832311 96.562689)
-		(end 145.619622 99.35)
+		(start 133.35 92.71)
+		(end 133.35 92.725)
 		(width 0.2286)
 		(layer "F.Cu")
@@
 	)
 	(segment
-		(start 141.59 92.725)
-		(end 141.605 92.71)
+		(start 142.832311 96.562689)
+		(end 145.619622 99.35)
 		(width 0.2286)
 		(layer "F.Cu")
@@
 	)
 	(via
+		(at 133.35 92.71)
+		(size 0.7)
+		(drill 0.35)
+		(layers "F.Cu" "B.Cu")
+		(locked yes)
+		(net 55)
+	)
+	(via
 		(at 141.605 92.71)
 		(size 0.7)
@@
 	)
 	(segment
+		(start 146.725 103.85)
+		(end 144.48267 103.85)
+		(width 0.2286)
+		(layer "F.Cu")
+		(net 78)
+	)
+	(segment
+		(start 144.48267 103.85)
+		(end 142.28767 106.045)
+		(width 0.2286)
+		(layer "F.Cu")
+		(net 78)
+	)
+	(segment
 		(start 141.745 105.905)
 		(end 141.745 107.95)
 		(width 0.2286)
 		(layer "F.Cu")
+		(net 78)
+	)
+	(segment
+		(start 142.28767 106.045)
+		(end 141.745 106.045)
+		(width 0.2286)
+		(layer "F.Cu")

Commit message: Hmmm
Changed lines of the file:
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@@
 			)
 		)
-		(property "LCSC" "C72043"
+		(property "LCSC" "C19171301"
 			(at 0 0 0)
 			(layer "F.Fab")
@@
 			)
 		)
-		(property "LCSC" "C72041"
+		(property "LCSC" "C2288"
 			(at 0 0 0)
 			(layer "F.Fab")
@@
 			)
 		)
+		(property "LCSC" "C2915304"
+			(at 0 0 0)
+			(unlocked yes)
+			(layer "F.Fab")
+			(hide yes)
+			(effects
+				(font
+					(size 1 1)
+					(thickness 0.15)
+				)
+			)
+		)
 		(property ki_fp_filters "LQFP*10x10mm*P0.5mm*")
 		(sheetname "/")
@@
 	)
 	(segment
-		(start 158.075 97.85)
-		(end 156.15 97.85)
-		(width 0.2286)
-		(layer "F.Cu")
-		(net 1)
-	)
-	(segment
 		(start 149.365 108.725)
 		(end 149.365 109.855)
@@
 	)
 	(segment
+		(start 156.15 97.85)
+		(end 153.035 100.965)
+		(width 0.3048)
+		(layer "F.Cu")
+		(net 1)
+	)
+	(segment
 		(start 149.65 108.44)
 		(end 149.365 108.725)
@@
 	)
 	(segment
-		(start 156.15 97.85)
-		(end 153.035 100.965)
+		(start 115.91 110.49)
+		(end 115.91 113.03)
 		(width 0.2286)
 		(layer "F.Cu")
@@
 	)
 	(segment
-		(start 115.91 110.49)
-		(end 115.91 113.03)
-		(width 0.2286)
+		(start 158.075 97.85)
+		(end 156.15 97.85)
+		(width 0.3048)
 		(layer "F.Cu")
 		(net 1)
@@
 		(drill 0.35)
 		(layers "F.Cu" "B.Cu")
+		(locked yes)
 		(net 1)
 	)
@@
 		(drill 0.35)
 		(layers "F.Cu" "B.Cu")
+		(locked yes)
 		(net 1)
 	)
@@
 		(drill 0.35)
 		(layers "F.Cu" "B.Cu")
+		(locked yes)
 		(net 1)
 	)
@@
 		(drill 0.35)
 		(layers "F.Cu" "B.Cu")
+		(locked yes)
 		(net 1)
 	)
@@
 		(drill 0.35)
 		(layers "F.Cu" "B.Cu")
+		(locked yes)
 		(net 2)
 	)
@@
 		(drill 0.35)
 		(layers "F.Cu" "B.Cu")
+		(locked yes)
 		(net 2)
 	)
@@
 		(drill 0.35)
 		(layers "F.Cu" "B.Cu")
+		(locked yes)
 		(net 2)
 	)
@@
 		(drill 0.35)
 		(layers "F.Cu" "B.Cu")
+		(locked yes)
 		(net 2)
 	)

Commit message: Ready for order
Parts:
- D2: value ~ -> B5819W
- J1: value ~ -> TYPE-C-31-M-12
- JP3, JP4: value ~ -> JUMP2
- U2: value STM32F401RCTx -> STM32F402RCTx
Other:
- board text added: "16 MHz Xtal"
- board text added: "STM32F402"

Commit message: Started working on stmw2
Routing:
- net PC13: track 51.5 -> 44.9 mm, vias 0 -> 2
- net GND: vias 36 -> 37
Changed lines of the file:
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@@
 	(property "AUTHOR_EMAIL" "lth@stm32world.com")
 	(property "COMPANY" "STM32World")
-	(property "REVISION" "a")
+	(property "REVISION" "b")
 	(property "TITLE" "MCUSTM32F402")
 	(property "URL" "https://stm32world.com/wiki/MCUSTM32F402")
@@
 	)
 	(via
+		(at 141.605 87.63)
+		(size 0.7)
+		(drill 0.35)
+		(layers "F.Cu" "B.Cu")
+		(free yes)
+		(net 2)
+	)
+	(via
 		(at 145.415 92.075)
 		(size 0.7)
@@
 	)
 	(segment
-		(start 143.593313 96.157529)
-		(end 143.593313 91.082093)
+		(start 146.725 98.35)
+		(end 145.785784 98.35)
 		(width 0.2286)
 		(layer "F.Cu")
@@
 	)
 	(segment
-		(start 122.555 89.725)
-		(end 120.84 91.44)
+		(start 128.905 88.9)
+		(end 126.365 91.44)
 		(width 0.2286)
 		(layer "F.Cu")
@@
 	)
 	(segment
-		(start 146.725 98.35)
-		(end 145.785784 98.35)
+		(start 139.389332 86.36)
+		(end 136.849333 83.82)
+		(width 0.2286)
+		(layer "F.Cu")
+		(net 50)
+	)
+	(segment
+		(start 142.875 86.995)
+		(end 142.24 86.36)
 		(width 0.2286)
 		(layer "F.Cu")
@@
 	)
 	(segment
-		(start 122.555 81.28)
-		(end 122.555 89.725)
+		(start 142.24 86.36)
+		(end 139.389332 86.36)
 		(width 0.2286)
 		(layer "F.Cu")
@@
 	)
 	(segment
-		(start 143.593313 91.082093)
-		(end 136.33122 83.82)
+		(start 143.593313 89.618313)
+		(end 142.875 88.9)
 		(width 0.2286)
 		(layer "F.Cu")
@@
 	)
 	(segment
-		(start 135.89 83.82)
-		(end 137.0067 82.7033)
+		(start 129.54 88.9)
+		(end 128.905 88.9)
 		(width 0.2286)
 		(layer "F.Cu")
@@
 	)
 	(segment
-		(start 137.0067 82.7033)
-		(end 137.0067 79.2217)
+		(start 143.593313 96.157529)
+		(end 143.593313 89.618313)
+		(width 0.2286)
+		(layer "F.Cu")
+		(net 50)
+	)
+	(segment
+		(start 126.365 91.44)
+		(end 120.84 91.44)
 		(width 0.2286)
 		(layer "F.Cu")
@@
 	)
 	(segment
-		(start 137.0067 79.2217)
-		(end 135.89 78.105)
+		(start 136.849333 83.82)
+		(end 135.89 83.82)
 		(width 0.2286)
 		(layer "F.Cu")
@@
 	)
 	(segment
-		(start 125.73 78.105)
-		(end 122.555 81.28)
+		(start 142.875 88.9)
+		(end 142.875 86.995)
 		(width 0.2286)
 		(layer "F.Cu")
 		(net 50)
 	)
+	(via
+		(at 129.54 88.9)
+		(size 0.7)
+		(drill 0.35)
+		(layers "F.Cu" "B.Cu")
+		(net 50)
+	)
+	(via
+		(at 142.875 88.9)
+		(size 0.7)
+		(drill 0.35)
+		(layers "F.Cu" "B.Cu")
+		(net 50)
+	)
 	(segment
-		(start 135.89 78.105)
-		(end 125.73 78.105)
+		(start 142.875 88.9)
+		(end 129.54 88.9)
 		(width 0.2286)
-		(layer "F.Cu")
+		(layer "B.Cu")
 		(net 50)
 	)
