File: stmw-bp-6/bp.kicad_pcb (KiCad board)
At the start: 2 copper layers, 100 x 67 mm, 8 parts, among them J1 Conn_02x25_Odd_Even, J2 Conn_02x25_Odd_Even, U1 X1611WVS-98-9TV01, U2 X1611WVS-98-9TV01, U3 X1611WVS-98-9TV01, U4 X1611WVS-98-9TV01, U5 X1611WVS-98-9TV01, U6 X1611WVS-98-9TV01

Commit message: Tweaking backplane
Parts:
- moved J2 1.54 mm to (182.0, 43.0)
- moved J1 1.00 mm to (96.0, 43.0)
Routing:
- net GND: track 15.0 -> 75.0 mm
Other:
- outline, holes or cut-outs redrawn

Commit message: Hmmmm
Parts:
- J1: footprint Connector_PinHeader_2.54mm:PinHeader_2x25_P2.54mm_Vertical -> Connector_IDC:IDC-Header_2x25_P2.54mm_Vertical
- moved J1 61.2 mm to (98.4, 104.1), turned to 180 degrees
- moved J2 61.2 mm to (184.2, 104.1), turned to 180 degrees
Connections:
- J1 pad 1: unconnected-(J1-Pin_1-Pad1) -> A1
- J1 pad 10: unconnected-(J1-Pin_10-Pad10) -> A10
- J1 pad 11: unconnected-(J1-Pin_11-Pad11) -> A11
- J1 pad 12: unconnected-(J1-Pin_12-Pad12) -> A12
- J1 pad 13: unconnected-(J1-Pin_13-Pad13) -> A13
- J1 pad 14: unconnected-(J1-Pin_14-Pad14) -> A14
- J1 pad 15: unconnected-(J1-Pin_15-Pad15) -> A15
- J1 pad 16: unconnected-(J1-Pin_16-Pad16) -> A16
- J1 pad 17: unconnected-(J1-Pin_17-Pad17) -> A17
- J1 pad 18: unconnected-(J1-Pin_18-Pad18) -> A18
- J1 pad 19: unconnected-(J1-Pin_19-Pad19) -> A19
- J1 pad 2: unconnected-(J1-Pin_2-Pad2) -> A2
- J1 pad 20: unconnected-(J1-Pin_20-Pad20) -> A20
- J1 pad 21: unconnected-(J1-Pin_21-Pad21) -> A21
- J1 pad 22: unconnected-(J1-Pin_22-Pad22) -> A22
- J1 pad 23: unconnected-(J1-Pin_23-Pad23) -> A23
- J1 pad 24: unconnected-(J1-Pin_24-Pad24) -> A24
- J1 pad 25: unconnected-(J1-Pin_25-Pad25) -> A25
- J1 pad 26: unconnected-(J1-Pin_26-Pad26) -> A26
- J1 pad 27: unconnected-(J1-Pin_27-Pad27) -> A27
- J1 pad 28: unconnected-(J1-Pin_28-Pad28) -> A28
- J1 pad 29: unconnected-(J1-Pin_29-Pad29) -> A29
- J1 pad 3: unconnected-(J1-Pin_3-Pad3) -> A3
- J1 pad 30: unconnected-(J1-Pin_30-Pad30) -> A30
- J1 pad 31: unconnected-(J1-Pin_31-Pad31) -> A31
- J1 pad 32: unconnected-(J1-Pin_32-Pad32) -> A32
- J1 pad 33: unconnected-(J1-Pin_33-Pad33) -> A33
- J1 pad 34: unconnected-(J1-Pin_34-Pad34) -> A34
- J1 pad 35: unconnected-(J1-Pin_35-Pad35) -> A35
- J1 pad 36: unconnected-(J1-Pin_36-Pad36) -> A36
- J1 pad 37: unconnected-(J1-Pin_37-Pad37) -> A37
- J1 pad 38: unconnected-(J1-Pin_38-Pad38) -> A38
- J1 pad 39: unconnected-(J1-Pin_39-Pad39) -> A39
- J1 pad 4: unconnected-(J1-Pin_4-Pad4) -> A4
- J1 pad 40: unconnected-(J1-Pin_40-Pad40) -> A40
- J1 pad 41: unconnected-(J1-Pin_41-Pad41) -> A41
- J1 pad 42: unconnected-(J1-Pin_42-Pad42) -> A42
- J1 pad 43: unconnected-(J1-Pin_43-Pad43) -> A43
- J1 pad 44: unconnected-(J1-Pin_44-Pad44) -> A44
- J1 pad 45: unconnected-(J1-Pin_45-Pad45) -> A45
- J1 pad 46: unconnected-(J1-Pin_46-Pad46) -> A46
- J1 pad 47: unconnected-(J1-Pin_47-Pad47) -> A47
- J1 pad 48: unconnected-(J1-Pin_48-Pad48) -> A48
- J1 pad 49: unconnected-(J1-Pin_49-Pad49) -> A49
- J1 pad 5: unconnected-(J1-Pin_5-Pad5) -> A5
- J1 pad 50: unconnected-(J1-Pin_50-Pad50) -> GND
- J1 pad 6: unconnected-(J1-Pin_6-Pad6) -> A6
- J1 pad 7: unconnected-(J1-Pin_7-Pad7) -> A7
- J1 pad 8: unconnected-(J1-Pin_8-Pad8) -> A8
- J1 pad 9: unconnected-(J1-Pin_9-Pad9) -> A9
- J2 pad 1: unconnected-(J2-Pin_1-Pad1) -> B2
- J2 pad 10: unconnected-(J2-Pin_10-Pad10) -> B9
- J2 pad 11: unconnected-(J2-Pin_11-Pad11) -> B12
- J2 pad 12: unconnected-(J2-Pin_12-Pad12) -> B11
- J2 pad 13: unconnected-(J2-Pin_13-Pad13) -> B14
- J2 pad 14: unconnected-(J2-Pin_14-Pad14) -> B13
- J2 pad 15: unconnected-(J2-Pin_15-Pad15) -> B16
- J2 pad 16: unconnected-(J2-Pin_16-Pad16) -> B15
- J2 pad 17: unconnected-(J2-Pin_17-Pad17) -> B18
- J2 pad 18: unconnected-(J2-Pin_18-Pad18) -> B17
- J2 pad 19: unconnected-(J2-Pin_19-Pad19) -> B20
- J2 pad 2: unconnected-(J2-Pin_2-Pad2) -> B1
- J2 pad 20: unconnected-(J2-Pin_20-Pad20) -> B19
- J2 pad 21: unconnected-(J2-Pin_21-Pad21) -> B22
- J2 pad 22: unconnected-(J2-Pin_22-Pad22) -> B21
- J2 pad 23: unconnected-(J2-Pin_23-Pad23) -> B24
- J2 pad 24: unconnected-(J2-Pin_24-Pad24) -> B23
- J2 pad 25: unconnected-(J2-Pin_25-Pad25) -> B26
- J2 pad 26: unconnected-(J2-Pin_26-Pad26) -> B25
- J2 pad 27: unconnected-(J2-Pin_27-Pad27) -> B28
- J2 pad 28: unconnected-(J2-Pin_28-Pad28) -> B27
- J2 pad 29: unconnected-(J2-Pin_29-Pad29) -> B30
- J2 pad 3: unconnected-(J2-Pin_3-Pad3) -> B4
- J2 pad 30: unconnected-(J2-Pin_30-Pad30) -> B29
- J2 pad 31: unconnected-(J2-Pin_31-Pad31) -> B32
- J2 pad 32: unconnected-(J2-Pin_32-Pad32) -> B31
- J2 pad 33: unconnected-(J2-Pin_33-Pad33) -> B34
- J2 pad 34: unconnected-(J2-Pin_34-Pad34) -> B33
- J2 pad 35: unconnected-(J2-Pin_35-Pad35) -> B36
- J2 pad 36: unconnected-(J2-Pin_36-Pad36) -> B35
- J2 pad 37: unconnected-(J2-Pin_37-Pad37) -> B38
- J2 pad 38: unconnected-(J2-Pin_38-Pad38) -> B37
- J2 pad 39: unconnected-(J2-Pin_39-Pad39) -> B40
- J2 pad 4: unconnected-(J2-Pin_4-Pad4) -> B3
- J2 pad 40: unconnected-(J2-Pin_40-Pad40) -> B39
- J2 pad 41: unconnected-(J2-Pin_41-Pad41) -> B42
- J2 pad 42: unconnected-(J2-Pin_42-Pad42) -> B41
- J2 pad 43: unconnected-(J2-Pin_43-Pad43) -> B44
- J2 pad 44: unconnected-(J2-Pin_44-Pad44) -> B43
- J2 pad 45: unconnected-(J2-Pin_45-Pad45) -> B46
- J2 pad 46: unconnected-(J2-Pin_46-Pad46) -> B45
- J2 pad 47: unconnected-(J2-Pin_47-Pad47) -> B48
- J2 pad 48: unconnected-(J2-Pin_48-Pad48) -> B47
- J2 pad 49: unconnected-(J2-Pin_49-Pad49) -> GND
- J2 pad 5: unconnected-(J2-Pin_5-Pad5) -> B6
- J2 pad 50: unconnected-(J2-Pin_50-Pad50) -> B49
- J2 pad 6: unconnected-(J2-Pin_6-Pad6) -> B5
- J2 pad 7: unconnected-(J2-Pin_7-Pad7) -> B8
- J2 pad 8: unconnected-(J2-Pin_8-Pad8) -> B7
- J2 pad 9: unconnected-(J2-Pin_9-Pad9) -> B10
Routing:
- net B2: track 77.8 -> 94.2 mm
- net B4: track 77.8 -> 94.0 mm
- net B48: track 78.0 -> 94.1 mm
- net B12: track 77.8 -> 94.0 mm
- net B6: track 77.9 -> 93.9 mm
- net B46: track 77.9 -> 93.8 mm
- net B14: track 78.1 -> 93.9 mm
- net B8: track 77.9 -> 93.6 mm
- net B44: track 77.9 -> 93.5 mm
- net B16: track 77.8 -> 93.5 mm
- net B10: track 78.1 -> 93.7 mm
- net B42: track 77.8 -> 93.3 mm
- net B18: track 77.8 -> 93.3 mm
- net B40: track 77.9 -> 93.2 mm
- net B20: track 77.8 -> 93.1 mm
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
Commit message: Changes
Parts:
- removed U6: X1611WVS-98-9TV01, stm32world:CONN-SMD_98P-P1.00-V_3133
- added H1: MountingHole, MountingHole:MountingHole_2.2mm_M2_DIN965, F.Cu at (92.0, 124.0)
- added H2: MountingHole, MountingHole:MountingHole_2.2mm_M2_DIN965, F.Cu at (188.0, 124.0)
- added H3: MountingHole, MountingHole:MountingHole_2.2mm_M2_DIN965, F.Cu at (188.0, 42.0)
- added H4: MountingHole, MountingHole:MountingHole_2.2mm_M2_DIN965, F.Cu at (92.0, 42.0)
- J2: footprint Connector_PinHeader_2.54mm:PinHeader_2x25_P2.54mm_Vertical -> Connector_IDC:IDC-Header_2x25_P2.54mm_Vertical
- moved J2 52.9 mm to (179.0, 51.5), turned to 0 degrees
- moved J1 8.73 mm to (101.0, 112.5)
- moved U1 6.89 mm to (116.0, 75.8)
- moved U2 6.89 mm to (128.0, 75.8)
- moved U3 6.89 mm to (140.0, 75.8)
- moved U4 6.89 mm to (152.0, 75.8)
- moved U5 6.89 mm to (164.0, 75.8)
Connections:
- J2 pad 1: B2 -> GND
- J2 pad 10: B9 -> B41
- J2 pad 11: B12 -> B40
- J2 pad 12: B11 -> B39
- J2 pad 13: B14 -> B38
- J2 pad 14: B13 -> B37
- J2 pad 15: B16 -> B36
- J2 pad 16: B15 -> B35
- J2 pad 17: B18 -> B34
- J2 pad 18: B17 -> B33
- J2 pad 19: B20 -> B32
- J2 pad 2: B1 -> B49
- J2 pad 20: B19 -> B31
- J2 pad 21: B22 -> B30
- J2 pad 22: B21 -> B29
- J2 pad 23: B24 -> B28
- J2 pad 24: B23 -> B27
- J2 pad 27: B28 -> B24
- J2 pad 28: B27 -> B23
- J2 pad 29: B30 -> B22
- J2 pad 3: B4 -> B48
- J2 pad 30: B29 -> B21
- J2 pad 31: B32 -> B20
- J2 pad 32: B31 -> B19
- J2 pad 33: B34 -> B18
- J2 pad 34: B33 -> B17
- J2 pad 35: B36 -> B16
- J2 pad 36: B35 -> B15
- J2 pad 37: B38 -> B14
- J2 pad 38: B37 -> B13
- J2 pad 39: B40 -> B12
- J2 pad 4: B3 -> B47
- J2 pad 40: B39 -> B11
- J2 pad 41: B42 -> B10
- J2 pad 42: B41 -> B9
- J2 pad 43: B44 -> B8
- J2 pad 44: B43 -> B7
- J2 pad 45: B46 -> B6
- J2 pad 46: B45 -> B5
- J2 pad 47: B48 -> B4
- J2 pad 48: B47 -> B3
- J2 pad 49: GND -> B2
- J2 pad 5: B6 -> B46
- J2 pad 50: B49 -> B1
- J2 pad 6: B5 -> B45
- J2 pad 7: B8 -> B44
- J2 pad 8: B7 -> B43
- J2 pad 9: B10 -> B42
Routing:
- net A48: track 85.8 -> 45.3 mm, vias 6 -> 5
- net B1: track 84.6 -> 45.3 mm, vias 6 -> 5
- net B2: track 94.2 -> 62.7 mm, vias 6 -> 5
- net B4: track 94.0 -> 62.8 mm, vias 6 -> 5
- net B48: track 94.1 -> 62.9 mm, vias 6 -> 5
- net B12: track 94.0 -> 62.8 mm, vias 6 -> 5
- net B6: track 93.9 -> 62.9 mm, vias 6 -> 5
- net B14: track 93.9 -> 63.0 mm, vias 6 -> 5
- net B46: track 93.8 -> 62.8 mm, vias 6 -> 5
- net B8: track 93.6 -> 62.8 mm, vias 6 -> 5
- net B44: track 93.5 -> 62.8 mm, vias 6 -> 5
- net B16: track 93.5 -> 62.8 mm, vias 6 -> 5
- net B10: track 93.7 -> 63.1 mm, vias 6 -> 5
- net B42: track 93.3 -> 62.8 mm, vias 6 -> 5
- net B18: track 93.3 -> 62.8 mm, vias 6 -> 5
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Other:
- board size 100 x 67 mm -> 100 x 86 mm
- board text added: "A1"
- board text added: "A3"
