File: stmw-bp-6/bp.kicad_sch (KiCad schematic)
At the start: 8 parts, among them J1 Conn_02x25_Odd_Even, J2 Conn_02x25_Odd_Even, U1 X1611WVS-98-9TV01, U2 X1611WVS-98-9TV01, U3 X1611WVS-98-9TV01, U4 X1611WVS-98-9TV01, U5 X1611WVS-98-9TV01, U6 X1611WVS-98-9TV01

Commit message: Tweaking backplane
Changed lines of the file:
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@@
 		(on_board yes)
 		(dnp no)
-		(fields_autoplaced yes)
 		(property "Reference" "J1"
-			(at 261.62 20.32 0)
+			(at 259.842 24.384 0)
 			(effects
 				(font
@@
 					(size 1.27 1.27)
 				)
+				(hide yes)
 			)
 		)
@@
 		(on_board yes)
 		(dnp no)
-		(fields_autoplaced yes)
 		(property "Reference" "J2"
-			(at 261.62 90.17 0)
+			(at 259.842 94.234 0)
 			(effects
 				(font
@@
 					(size 1.27 1.27)
 				)
-			)
-		)
+				(hide yes)
+			)
+		)

Commit message: Hmmmm
Parts:
- J1: footprint Connector_PinHeader_2.54mm:PinHeader_2x25_P2.54mm_Vertical -> Connector_IDC:IDC-Header_2x25_P2.54mm_Vertical
Connections:
- net A1: now also J1.1 (Pin_1)
- net A10: now also J1.10 (Pin_10)
- net A11: now also J1.11 (Pin_11)
- net A12: now also J1.12 (Pin_12)
- net A13: now also J1.13 (Pin_13)
- net A14: now also J1.14 (Pin_14)
- net A15: now also J1.15 (Pin_15)
- net A16: now also J1.16 (Pin_16)
- net A17: now also J1.17 (Pin_17)
- net A18: now also J1.18 (Pin_18)
- net A19: now also J1.19 (Pin_19)
- net A2: now also J1.2 (Pin_2)
- net A20: now also J1.20 (Pin_20)
- net A21: now also J1.21 (Pin_21)
- net A22: now also J1.22 (Pin_22)
- net A23: now also J1.23 (Pin_23)
- net A24: now also J1.24 (Pin_24)
- net A25: now also J1.25 (Pin_25)
- net A26: now also J1.26 (Pin_26)
- net A27: now also J1.27 (Pin_27)
- net A28: now also J1.28 (Pin_28)
- net A29: now also J1.29 (Pin_29)
- net A3: now also J1.3 (Pin_3)
- net A30: now also J1.30 (Pin_30)
- net A31: now also J1.31 (Pin_31)
- net A32: now also J1.32 (Pin_32)
- net A33: now also J1.33 (Pin_33)
- net A34: now also J1.34 (Pin_34)
- net A35: now also J1.35 (Pin_35)
- net A36: now also J1.36 (Pin_36)
- net A37: now also J1.37 (Pin_37)
- net A38: now also J1.38 (Pin_38)
- net A39: now also J1.39 (Pin_39)
- net A4: now also J1.4 (Pin_4)
- net A40: now also J1.40 (Pin_40)
- net A41: now also J1.41 (Pin_41)
- net A42: now also J1.42 (Pin_42)
- net A43: now also J1.43 (Pin_43)
- net A44: now also J1.44 (Pin_44)
- net A45: now also J1.45 (Pin_45)
- net A46: now also J1.46 (Pin_46)
- net A47: now also J1.47 (Pin_47)
- net A48: now also J1.48 (Pin_48)
- net A49: now also J1.49 (Pin_49)
- net A5: now also J1.5 (Pin_5)
- net A6: now also J1.6 (Pin_6)
- net A7: now also J1.7 (Pin_7)
- net A8: now also J1.8 (Pin_8)
- net A9: now also J1.9 (Pin_9)
- net B1: now also J2.2 (Pin_2)
- net B10: now also J2.9 (Pin_9)
- net B11: now also J2.12 (Pin_12)
- net B12: now also J2.11 (Pin_11)
- net B13: now also J2.14 (Pin_14)
- net B14: now also J2.13 (Pin_13)
- net B15: now also J2.16 (Pin_16)
- net B16: now also J2.15 (Pin_15)
- net B17: now also J2.18 (Pin_18)
- net B18: now also J2.17 (Pin_17)
- net B19: now also J2.20 (Pin_20)
- net B2: now also J2.1 (Pin_1)
- net B20: now also J2.19 (Pin_19)
- net B21: now also J2.22 (Pin_22)
- net B22: now also J2.21 (Pin_21)
- net B23: now also J2.24 (Pin_24)
- net B24: now also J2.23 (Pin_23)
- net B25: now also J2.26 (Pin_26)
- net B26: now also J2.25 (Pin_25)
- net B27: now also J2.28 (Pin_28)
- net B28: now also J2.27 (Pin_27)
- net B29: now also J2.30 (Pin_30)
- net B3: now also J2.4 (Pin_4)
- net B30: now also J2.29 (Pin_29)
- net B31: now also J2.32 (Pin_32)
- net B32: now also J2.31 (Pin_31)
- net B33: now also J2.34 (Pin_34)
- net B34: now also J2.33 (Pin_33)
- net B35: now also J2.36 (Pin_36)
- net B36: now also J2.35 (Pin_35)
- net B37: now also J2.38 (Pin_38)
- net B38: now also J2.37 (Pin_37)
- net B39: now also J2.40 (Pin_40)
- net B4: now also J2.3 (Pin_3)
- net B40: now also J2.39 (Pin_39)
- net B41: now also J2.42 (Pin_42)
- net B42: now also J2.41 (Pin_41)
- net B43: now also J2.44 (Pin_44)
- net B44: now also J2.43 (Pin_43)
- net B45: now also J2.46 (Pin_46)
- net B46: now also J2.45 (Pin_45)
- net B47: now also J2.48 (Pin_48)
- net B48: now also J2.47 (Pin_47)
- net B49: now also J2.50 (Pin_50)
- net B5: now also J2.6 (Pin_6)
- net B6: now also J2.5 (Pin_5)
- net B7: now also J2.8 (Pin_8)
- net B8: now also J2.7 (Pin_7)
- net B9: now also J2.10 (Pin_10)
- net GND: now also J1.50 (Pin_50), J2.49 (Pin_49)

Commit message: Changes
Parts:
- removed U6: X1611WVS-98-9TV01, stm32world:CONN-SMD_98P-P1.00-V_3133, symbol stm32world:X1611WVS-98-9TV01
- added H1, H2, H3, H4: MountingHole, MountingHole:MountingHole_2.2mm_M2_DIN965, symbol Mechanical:MountingHole
- J2: footprint Connector_PinHeader_2.54mm:PinHeader_2x25_P2.54mm_Vertical -> Connector_IDC:IDC-Header_2x25_P2.54mm_Vertical
Connections:
- net B1: now also J2.50 (Pin_50); no longer J2.2 (Pin_2)
- net B10: now also J2.41 (Pin_41); no longer J2.9 (Pin_9)
- net B11: now also J2.40 (Pin_40); no longer J2.12 (Pin_12)
- net B12: now also J2.39 (Pin_39); no longer J2.11 (Pin_11)
- net B13: now also J2.38 (Pin_38); no longer J2.14 (Pin_14)
- net B14: now also J2.37 (Pin_37); no longer J2.13 (Pin_13)
- net B15: now also J2.36 (Pin_36); no longer J2.16 (Pin_16)
- net B16: now also J2.35 (Pin_35); no longer J2.15 (Pin_15)
- net B17: now also J2.34 (Pin_34); no longer J2.18 (Pin_18)
- net B18: now also J2.33 (Pin_33); no longer J2.17 (Pin_17)
- net B19: now also J2.32 (Pin_32); no longer J2.20 (Pin_20)
- net B2: now also J2.49 (Pin_49); no longer J2.1 (Pin_1)
- net B20: now also J2.31 (Pin_31); no longer J2.19 (Pin_19)
- net B21: now also J2.30 (Pin_30); no longer J2.22 (Pin_22)
- net B22: now also J2.29 (Pin_29); no longer J2.21 (Pin_21)
- net B23: now also J2.28 (Pin_28); no longer J2.24 (Pin_24)
- net B24: now also J2.27 (Pin_27); no longer J2.23 (Pin_23)
- net B27: now also J2.24 (Pin_24); no longer J2.28 (Pin_28)
- net B28: now also J2.23 (Pin_23); no longer J2.27 (Pin_27)
- net B29: now also J2.22 (Pin_22); no longer J2.30 (Pin_30)
- net B3: now also J2.48 (Pin_48); no longer J2.4 (Pin_4)
- net B30: now also J2.21 (Pin_21); no longer J2.29 (Pin_29)
- net B31: now also J2.20 (Pin_20); no longer J2.32 (Pin_32)
- net B32: now also J2.19 (Pin_19); no longer J2.31 (Pin_31)
- net B33: now also J2.18 (Pin_18); no longer J2.34 (Pin_34)
- net B34: now also J2.17 (Pin_17); no longer J2.33 (Pin_33)
- net B35: now also J2.16 (Pin_16); no longer J2.36 (Pin_36)
- net B36: now also J2.15 (Pin_15); no longer J2.35 (Pin_35)
- net B37: now also J2.14 (Pin_14); no longer J2.38 (Pin_38)
- net B38: now also J2.13 (Pin_13); no longer J2.37 (Pin_37)
- net B39: now also J2.12 (Pin_12); no longer J2.40 (Pin_40)
- net B4: now also J2.47 (Pin_47); no longer J2.3 (Pin_3)
- net B40: now also J2.11 (Pin_11); no longer J2.39 (Pin_39)
- net B41: now also J2.10 (Pin_10); no longer J2.42 (Pin_42)
- net B42: now also J2.9 (Pin_9); no longer J2.41 (Pin_41)
- net B43: now also J2.8 (Pin_8); no longer J2.44 (Pin_44)
- net B44: now also J2.7 (Pin_7); no longer J2.43 (Pin_43)
- net B45: now also J2.6 (Pin_6); no longer J2.46 (Pin_46)
- net B46: now also J2.5 (Pin_5); no longer J2.45 (Pin_45)
- net B47: now also J2.4 (Pin_4); no longer J2.48 (Pin_48)
- net B48: now also J2.3 (Pin_3); no longer J2.47 (Pin_47)
- net B49: now also J2.2 (Pin_2); no longer J2.50 (Pin_50)
- net B5: now also J2.46 (Pin_46); no longer J2.6 (Pin_6)
- net B6: now also J2.45 (Pin_45); no longer J2.5 (Pin_5)
- net B7: now also J2.44 (Pin_44); no longer J2.8 (Pin_8)
- net B8: now also J2.43 (Pin_43); no longer J2.7 (Pin_7)
- net B9: now also J2.42 (Pin_42); no longer J2.10 (Pin_10)
- net GND: now also J2.1 (Pin_1); no longer J2.49 (Pin_49)
