File: stmw-mcu-stm32f405/stmw-mcu-stm32f405.kicad_sch (KiCad schematic)
At the start: 38 parts, among them J2 TYPE-C-31-M-12, SW1 TS-1088R-02526, SW2 TS-1088R-02526, U1 AMS1117-3.3, U3 STM32F407VETx, Y1 X_16MHZ

Commit message: Hmmmm
Parts:
- added H1, H2: MountingHole, MountingHole:MountingHole_2.2mm_M2, symbol Mechanical:MountingHole
- C12, C14: value C_2.2UF_0603 -> 2.2uF; Display 2.2uF -> (none)
Connections:
- net BO0: now also U3.9 (PC15)
- net GND: now also J1.B49
- net PA11: now also J1.B46
- net PA12: now also J1.B47
- net PC0: now also J1.A14
- net PC13: now also J1.A16, U3.7 (PC13)
- net PA0: now reaches J1.A10
- net PA0: now also U3.23 (PA0)
- net PC3: now reaches J1.A11
- net PC3: now also U3.18 (PC3)
- net PC2: now reaches J1.A12
- net PC2: now also U3.17 (PC2)
- net PC1: now reaches J1.A13
- net PC1: now also U3.16 (PC1)
- net PC14: now reaches J1.A15
- net PC14: now also U3.8 (PC14)
- net PE6: now reaches J1.A17
- net PE6: now also U3.5 (PE6)
- net PE5: now reaches J1.A18
- net PE5: now also U3.4 (PE5)
- net PE4: now reaches J1.A19
- net PE4: now also U3.3 (PE4)
- net PE3: now reaches J1.A20
- net PE3: now also U3.2 (PE3)
- net PE2: now reaches J1.A21
- net PE2: now also U3.1 (PE2)
- net PE1: now reaches J1.A22
- net PE1: now also U3.98 (PE1)
- net PE0: now reaches J1.A23
- net PE0: now also U3.97 (PE0)
- net PB9: now reaches J1.A24
- net PB9: now also U3.96 (PB9)
- net PB8: now reaches J1.A25
- net PB8: now also U3.95 (PB8)
- net PB7: now reaches J1.A26
- net PB7: now also U3.93 (PB7)
- net PB6: now reaches J1.A27
- net PB6: now also U3.92 (PB6)
- net PB5: now reaches J1.A28
- net PB5: now also U3.91 (PB5)
- net PB4: now reaches J1.A29
- net PB4: now also U3.90 (PB4)
- net PB3: now reaches J1.A30
- net PB3: now also U3.89 (PB3)
- net PD7: now reaches J1.A31
- net PD7: now also U3.88 (PD7)
- net PD6: now reaches J1.A32
- net PD6: now also U3.87 (PD6)
- net PD5: now reaches J1.A33
- net PD5: now also U3.86 (PD5)
- net PD4: now reaches J1.A34
- net PD4: now also U3.85 (PD4)
- net PD3: now reaches J1.A35
- net PD3: now also U3.84 (PD3)
- net PD2: now reaches J1.A36
- net PD2: now also U3.83 (PD2)
- net PD1: now reaches J1.A37
- net PD1: now also U3.82 (PD1)
- net PD0: now reaches J1.A38
- net PD0: now also U3.81 (PD0)
- net PC12: now reaches J1.A39
- net PC12: now also U3.80 (PC12)
- net PC11: now reaches J1.A40
- net PC11: now also U3.79 (PC11)
- net PC10: now reaches J1.A41
- net PC10: now also U3.78 (PC10)
- net PA15: now reaches J1.A42
- net PA15: now also U3.77 (PA15)
- net PA14: now reaches J1.A43
- net PA14: now also U3.76 (PA14)
- net PA2: now reaches J1.A8
- net PA2: now also U3.25 (PA2)
- net PA1: now reaches J1.A9
- net PA1: now also U3.24 (PA1)
- net PA3: now reaches U3.26 (PA3)
- net PA3: now also J1.B8
- net PA4: now reaches U3.29 (PA4)
- net PA4: now also J1.B9
- net PA5: now reaches U3.30 (PA5)
- net PA5: now also J1.B10
- net PA6: now reaches U3.31 (PA6)
- net PA6: now also J1.B11
- net PA7: now reaches U3.32 (PA7)
- net PA7: now also J1.B12
- net PC4: now reaches U3.33 (PC4)
- net PC4: now also J1.B13
- net PC5: now reaches U3.34 (PC5)
- net PC5: now also J1.B14
- net PB0: now reaches U3.35 (PB0)
- net PB0: now also J1.B15
- net PB1: now reaches U3.36 (PB1)
- net PB1: now also J1.B16
- net PB2: now reaches U3.37 (PB2)
- net PB2: now also J1.B17
- net PE7: now reaches U3.38 (PE7)
- net PE7: now also J1.B18
- net PE8: now reaches U3.39 (PE8)
- net PE8: now also J1.B19
- net PE9: now reaches U3.40 (PE9)
- net PE9: now also J1.B20
- net PE10: now reaches U3.41 (PE10)
- net PE10: now also J1.B21
- net PE11: now reaches U3.42 (PE11)
- net PE11: now also J1.B22
- net PE12: now reaches U3.43 (PE12)
- net PE12: now also J1.B23
- net PE13: now reaches U3.44 (PE13)
- net PE13: now also J1.B24
- net PE14: now reaches U3.45 (PE14)
- net PE14: now also J1.B25
- net PE15: now reaches U3.46 (PE15)
- net PE15: now also J1.B26
- net PB10: now reaches U3.47 (PB10)
- net PB11: now reaches U3.48 (PB11)
- net PB12: now reaches U3.51 (PB12)
- net PB12: now also J1.B27
- net PB13: now reaches U3.52 (PB13)
- net PB13: now also J1.B28
- net PB14: now reaches U3.53 (PB14)
- net PB14: now also J1.B29
- net PB15: now reaches U3.54 (PB15)
- net PB15: now also J1.B30
- net PD8: now reaches U3.55 (PD8)
- net PD8: now also J1.B31
- net PD9: now reaches U3.56 (PD9)
- net PD9: now also J1.B32
- net PD10: now reaches U3.57 (PD10)
- net PD10: now also J1.B33
- net PD11: now reaches U3.58 (PD11)
- net PD11: now also J1.B34
- net PD12: now reaches U3.59 (PD12)
- net PD12: now also J1.B35
- net PD13: now reaches U3.60 (PD13)
- net PD13: now also J1.B36
- net PD14: now reaches U3.61 (PD14)
- net PD14: now also J1.B37
- net PD15: now reaches U3.62 (PD15)
- net PD15: now also J1.B38
- net PC6: now reaches U3.63 (PC6)
- net PC6: now also J1.B39
- net PC7: now reaches U3.64 (PC7)
- net PC7: now also J1.B40
- net PC8: now reaches U3.65 (PC8)
- net PC8: now also J1.B41
- net PC9: now reaches U3.66 (PC9)
- net PC9: now also J1.B42
- net PA8: now reaches U3.67 (PA8)
- net PA8: now also J1.B43
- net PA9: now reaches U3.68 (PA9)
- net PA9: now also J1.B44
- net PA10: now reaches U3.69 (PA10)
- net PA10: now also J1.B45
- net PA13: now reaches U3.72 (PA13)
- net PA13: now also J1.B48
Other:
- moved on the sheet: C11, C13, Y1
