File: stmw-mcu-stm32f407/stmw-mcu-stm32f407.kicad_pcb (KiCad board)
At the start: 4 copper layers, 69 x 43.5 mm, 40 parts, among them J2 TYPE-C-31-M-12, SW1 TS-1088R-02526, SW2 TS-1088R-02526, U1 AMS1117-3.3, U3 STM32F407VETx, Y1 X_16MHZ

Commit message: Hmmmm
Parts:
- added NT1: NetTie_2, NetTie:NetTie-2_SMD_Pad0.5mm, F.Cu at (124.0, 103.5)
- JP3, JP4: moved to B.Cu
- moved C10 21.5 mm to (130.2, 94.0)
- moved C12 17.8 mm to (130.2, 98.4)
- moved C7 15.5 mm to (127.0, 89.4)
- moved C9 15.5 mm to (125.1, 89.4)
- moved FB1 15.5 mm to (123.2, 89.4)
- moved JP2 15.5 mm to (123.8, 89.4)
- moved JP3 9.02 mm to (121.3, 100.0), turned to 180 degrees
- moved JP4 9.02 mm to (121.3, 103.5), turned to 180 degrees
- moved JP1 5.12 mm to (143.5, 79.4)
- moved C16 3.70 mm to (152.4, 78.7), turned to 180 degrees
- moved C15 2.01 mm to (163.8, 91.4)
- moved C14 0.90 mm to (163.8, 94.6)
Connections:
- J1 pad A1: unconnected-(J1-PadA1) -> GND
- J1 pad A10: PA0 -> PC0
- J1 pad A11: PC3 -> PC14
- J1 pad A12: PC2 -> U3
- J1 pad A13: PC1 -> PC13
- J1 pad A14: PC0 -> PE6
- J1 pad A15: PC14 -> PE5
- J1 pad A16: PC13 -> PE4
- J1 pad A17: PE6 -> PE3
- J1 pad A18: PE5 -> PE2
- J1 pad A19: PE4 -> U4
- J1 pad A2: unconnected-(J1-PadA2) -> HNRST
- J1 pad A20: PE3 -> PE1
- J1 pad A21: PE2 -> PE0
- J1 pad A22: PE1 -> PB9
- J1 pad A23: PE0 -> PB8
- J1 pad A24: PB9 -> PB7
- J1 pad A25: PB8 -> PB6
- J1 pad A26: PB7 -> PB5
- J1 pad A27: PB6 -> U6
- J1 pad A28: PB5 -> PB4
- J1 pad A29: PB4 -> PB3
- J1 pad A3: unconnected-(J1-PadA3) -> U1
- J1 pad A30: PB3 -> PD7
- J1 pad A31: PD7 -> PD6
- J1 pad A32: PD6 -> PD5
- J1 pad A33: PD5 -> PD4
- J1 pad A34: PD4 -> PD3
- J1 pad A35: PD3 -> PD2
- J1 pad A36: PD2 -> PD1
- J1 pad A37: PD1 -> PD0
- J1 pad A38: PD0 -> U8
- J1 pad A4: unconnected-(J1-PadA4) -> PA2
- J1 pad A44: unconnected-(J1-PadA44) -> PA11
- J1 pad A45: unconnected-(J1-PadA45) -> PA12
- J1 pad A46: unconnected-(J1-PadA46) -> PA13
- J1 pad A47: unconnected-(J1-PadA47) -> +3V3
- J1 pad A48: unconnected-(J1-PadA48) -> +5V
- J1 pad A49: unconnected-(J1-PadA49) -> GND
- J1 pad A5: unconnected-(J1-PadA5) -> PA1
- J1 pad A6: unconnected-(J1-PadA6) -> PA0
- J1 pad A7: unconnected-(J1-PadA7) -> PC3
- J1 pad A8: PA2 -> PC2
- J1 pad A9: PA1 -> PC1
- J1 pad B1: unconnected-(J1-PadB1) -> GND
- J1 pad B10: PA5 -> PC5
- J1 pad B11: PA6 -> PB0
- J1 pad B12: PA7 -> PB1
- J1 pad B13: PC4 -> PB2
- J1 pad B14: PC5 -> PE7
- J1 pad B15: PB0 -> PE8
- J1 pad B16: PB1 -> PE9
- J1 pad B17: PB2 -> PE10
- J1 pad B18: PE7 -> PE11
- J1 pad B19: PE8 -> U5
- J1 pad B2: unconnected-(J1-PadB2) -> HBO0
- J1 pad B20: PE9 -> PE12
- J1 pad B21: PE10 -> PE13
- J1 pad B22: PE11 -> PE14
- J1 pad B23: PE12 -> PE15
- J1 pad B24: PE13 -> PB10
- J1 pad B25: PE14 -> PB11
- J1 pad B26: PE15 -> PB12
- J1 pad B27: PB12 -> U7
- J1 pad B3: unconnected-(J1-PadB3) -> U2
- J1 pad B38: PD15 -> U9
- J1 pad B39: PC6 -> PD15
- J1 pad B4: unconnected-(J1-PadB4) -> PA3
- J1 pad B40: PC7 -> PC6
- J1 pad B41: PC8 -> PC7
- J1 pad B42: PC9 -> PC8
- J1 pad B43: PA8 -> PC9
- J1 pad B44: PA9 -> PA8
- J1 pad B45: PA10 -> PA9
- J1 pad B46: PA11 -> PA10
- J1 pad B47: PA12 -> +3V3
- J1 pad B48: PA13 -> +5V
- J1 pad B5: unconnected-(J1-PadB5) -> PA4
- J1 pad B6: unconnected-(J1-PadB6) -> PA5
- J1 pad B7: unconnected-(J1-PadB7) -> PA6
- J1 pad B8: PA3 -> PA7
- J1 pad B9: PA4 -> PC4
- U3 pad 9: BO0 -> PC15
Routing:
- net PA3: track 0.00 -> 30.8 mm
- net PA4: track 0.00 -> 30.1 mm
- net PA5: track 0.00 -> 28.3 mm
- net PA6: track 0.00 -> 27.7 mm
- net PA7: track 0.00 -> 27.1 mm
- net PA10: track 0.00 -> 26.6 mm
- net PC4: track 0.00 -> 26.4 mm
- net PA9: track 0.00 -> 26.0 mm
- net PC5: track 0.00 -> 25.8 mm
- net PA8: track 0.00 -> 25.4 mm
- net PB0: track 0.00 -> 25.2 mm
- net PC9: track 0.00 -> 24.8 mm
- net PC8: track 0.00 -> 24.2 mm
- net PB1: track 0.00 -> 23.8 mm
- net PC7: track 0.00 -> 23.5 mm
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
Commit message: Hmmm
Parts:
- C1, C3: value C_10UF_0805 -> 10uF
- C10, C15, C16, C2, C5, C6, C7, C8, C9: value C_100NF_0603 -> 100nF
- C11, C13: value C_20PF_0603 -> 20pF
- C4: value C_1UF_0603 -> 1uF
- moved C1 18.6 mm to (183.5, 85.0), turned to 90 degrees
- moved C4 15.2 mm to (176.0, 85.0)
- moved C3 15.1 mm to (178.0, 85.0)
- moved U1 15.0 mm to (177.5, 90.5)
- moved C8 11.6 mm to (127.5, 97.5)
- moved J2 11.5 mm to (181.0, 103.5)
- moved D1 11.5 mm to (171.4, 103.5)
- moved R1 11.5 mm to (174.5, 105.4)
- moved R2 11.5 mm to (174.5, 101.0)
- moved C15 9.07 mm to (163.5, 100.5)
- moved C14 7.39 mm to (163.5, 102.0)
- moved U3 7.16 mm to (150.0, 99.0)
- moved D3 6.53 mm to (170.0, 79.3)
- moved D4 6.53 mm to (166.8, 79.3)
- moved R5 6.53 mm to (170.0, 82.5)
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Connections:
- J1 pad A20: PE1 -> (no net)
- J1 pad A26: PB5 -> (no net)
- J1 pad A28: PB4 -> (no net)
- U3 pad 21: unconnected-(U3-VREF+-Pad21) -> +3V3
Routing:
- net +3V3: track 0.00 -> 112.0 mm, vias 0 -> 6
- net +5V: track 0.00 -> 53.1 mm, vias 0 -> 1
- net PA3: track 30.8 -> 0.00 mm
- net PA4: track 30.1 -> 0.00 mm
- net PC11: track 5.63 -> 35.0 mm
- net PA5: track 28.3 -> 0.00 mm
- net PC10: track 5.38 -> 33.2 mm
- net PA14: track 1.92 -> 29.6 mm
- net PA6: track 27.7 -> 0.00 mm
- net PA7: track 27.1 -> 0.00 mm
- net PA10: track 26.6 -> 0.00 mm
- net PC4: track 26.4 -> 0.00 mm
- net PA9: track 26.0 -> 0.00 mm
- net PC5: track 25.8 -> 0.00 mm
- net PA15: track 5.72 -> 31.4 mm
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- added copper zone on B.Cu, net +3V3
- added copper zone on F.Cu, net +3V3
- removed copper zone on In1.Cu, net +3V3
- removed copper zone on In2.Cu, net GND
Other:
- board size 69 x 43.5 mm -> 70 x 43.5 mm
- copper layers 4 -> 2

Commit message: Hmmmm
Parts:
- moved NT1 22.7 mm to (141.5, 88.0), turned to -90 degrees
- moved C12 20.3 mm to (148.0, 111.0), turned to 0 degrees
- moved FB1 13.6 mm to (136.0, 97.5), turned to 0 degrees
- moved C13 11.6 mm to (139.0, 92.0), turned to 180 degrees
- moved C9 11.2 mm to (136.0, 96.0), turned to 180 degrees
- moved C10 10.2 mm to (136.5, 103.5), turned to 180 degrees
- moved C8 9.19 mm to (136.0, 94.0)
- moved JP3 8.63 mm to (124.0, 109.0), turned to -90 degrees
- moved Y1 8.63 mm to (139.0, 89.0), turned to -90 degrees
- moved C5 8.41 mm to (153.5, 83.5)
- moved JP2 8.30 mm to (128.7, 97.5), turned to 0 degrees
- moved C6 7.82 mm to (122.0, 86.5)
- moved R4 7.50 mm to (130.0, 82.0), turned to 90 degrees
- moved C11 7.11 mm to (139.0, 86.0), turned to 0 degrees
- moved C2 6.71 mm to (144.5, 86.5)
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Connections:
- J1 pad A11: PC14 -> PC15
- J1 pad A12: U3 -> PC14
- J1 pad A20: (no net) -> PE1
- J1 pad A26: (no net) -> PB5
- J1 pad A28: (no net) -> PB4
- J1 pad A3: U1 -> VBAT
- J1 pad B3: U2 -> VA
Routing:
- net +3V3: track 112.0 -> 212.4 mm, vias 6 -> 8
- net BO0: track 0.00 -> 76.7 mm, vias 0 -> 3
- net PC13: track 0.00 -> 74.1 mm, vias 0 -> 1
- net VBAT: track 0.00 -> 59.2 mm, vias 0 -> 1
- net NRST: track 0.00 -> 55.0 mm
- net PE5: track 0.00 -> 43.4 mm
- net PC15: track 0.00 -> 37.8 mm, vias 0 -> 1
- net PE1: track 0.00 -> 37.5 mm
- net PE0: track 0.00 -> 36.8 mm
- net PC14: track 0.00 -> 36.4 mm
- net PB9: track 0.00 -> 36.3 mm
- net PE3: track 0.00 -> 36.3 mm
- net PE4: track 0.00 -> 36.0 mm
- net PE2: track 0.00 -> 35.2 mm
- net PE6: track 0.00 -> 34.9 mm
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