File: stmw-mcu-stm32f407/stmw-mcu-stm32f407.kicad_sch (KiCad schematic)
At the start: 40 parts, among them J2 TYPE-C-31-M-12, SW1 TS-1088R-02526, SW2 TS-1088R-02526, U1 AMS1117-3.3, U3 STM32F407VETx, Y1 X_16MHZ

Commit message: Hmmmm
Connections:
- net GND: now also J1.A1 (GND), J1.A49 (GND), J1.B1 (GND)
Other:
- moved on the sheet: C11, C12, C13, C14, U3, Y1

Commit message: Hmmmm
Parts:
- added NT1: NetTie_2, NetTie:NetTie-2_SMD_Pad0.5mm, symbol Device:NetTie_2
Connections:
- net +3V3: now also J1.A47, J1.B47
- net +5V: now also J1.A48, J1.B48
- net BO0: now also NT1.1; no longer U3.9 (PC15)
- net HBO0: now also J1.B2 (3.3V)
- net HNRST: now also J1.A2 (3.3V)
- net PA0: now also J1.A6; no longer J1.A10
- net PA1: now also J1.A5; no longer J1.A9
- net PA10: now also J1.B46; no longer J1.B45
- net PA11: now also J1.A44; no longer J1.B46
- net PA12: now also J1.A45; no longer J1.B47
- net PA13: now also J1.A46; no longer J1.B48
- net PA2: now also J1.A4; no longer J1.A8
- net PA3: now also J1.B4; no longer J1.B8
- net PA4: now also J1.B5; no longer J1.B9
- net PA5: now also J1.B6; no longer J1.B10
- net PA6: now also J1.B7; no longer J1.B11
- net PA7: now also J1.B8; no longer J1.B12
- net PA8: now also J1.B44; no longer J1.B43
- net PA9: now also J1.B45; no longer J1.B44
- net PB0: now also J1.B11; no longer J1.B15
- net PB1: now also J1.B12; no longer J1.B16
- net PB10: now also J1.B24
- net PB11: now also J1.B25
- net PB12: now also J1.B26; no longer J1.B27
- net PB2: now also J1.B13; no longer J1.B17
- net PB3: now also J1.A29; no longer J1.A30
- net PB4: now also J1.A28; no longer J1.A29
- net PB5: now also J1.A26; no longer J1.A28
- net PB6: now also J1.A25; no longer J1.A27
- net PB7: now also J1.A24; no longer J1.A26
- net PB8: now also J1.A23; no longer J1.A25
- net PB9: now also J1.A22; no longer J1.A24
- net PC0: now also J1.A10; no longer J1.A14
- net PC1: now also J1.A9; no longer J1.A13
- net PC13: now also J1.A13; no longer J1.A16
- net PC14: now also J1.A11; no longer J1.A15
- net PC2: now also J1.A8; no longer J1.A12
- net PC3: now also J1.A7; no longer J1.A11
- net PC4: now also J1.B9; no longer J1.B13
- net PC5: now also J1.B10; no longer J1.B14
- net PC6: now also J1.B40; no longer J1.B39
- net PC7: now also J1.B41; no longer J1.B40
- net PC8: now also J1.B42; no longer J1.B41
- net PC9: now also J1.B43; no longer J1.B42
- net PD0: now also J1.A37; no longer J1.A38
- net PD1: now also J1.A36; no longer J1.A37
- net PD15: now also J1.B39; no longer J1.B38
- net PD2: now also J1.A35; no longer J1.A36
- net PD3: now also J1.A34; no longer J1.A35
- net PD4: now also J1.A33; no longer J1.A34
- net PD5: now also J1.A32; no longer J1.A33
- net PD6: now also J1.A31; no longer J1.A32
- net PD7: now also J1.A30; no longer J1.A31
- net PE0: now also J1.A21; no longer J1.A23
- net PE1: now also J1.A20; no longer J1.A22
- net PE10: now also J1.B17; no longer J1.B21
- net PE11: now also J1.B18; no longer J1.B22
- net PE12: now also J1.B20; no longer J1.B23
- net PE13: now also J1.B21; no longer J1.B24
- net PE14: now also J1.B22; no longer J1.B25
- net PE15: now also J1.B23; no longer J1.B26
- net PE2: now also J1.A18; no longer J1.A21
- net PE3: now also J1.A17; no longer J1.A20
- net PE4: now also J1.A16; no longer J1.A19
- net PE5: now also J1.A15; no longer J1.A18
- net PE6: now also J1.A14; no longer J1.A17
- net PE7: now also J1.B14; no longer J1.B18
- net PE8: now also J1.B15; no longer J1.B19
- net PE9: now also J1.B16; no longer J1.B20
- net U1: now reaches J1.A3 (5V)
- net U2: now reaches J1.B3 (5V)
- new net PC15: NT1.2, U3.9 (PC15)
- new net U3: J1.A12
- new net U4: J1.A19
- new net U5: J1.B19
- new net U6: J1.A27
- new net U7: J1.B27
- new net U8: J1.A38
- new net U9: J1.B38
Other:
- moved on the sheet: J1

Commit message: Hmmm
Parts:
- C1, C3: value C_10UF_0805 -> 10uF
- C10, C15, C16, C2, C5, C6, C7, C8, C9: value C_100NF_0603 -> 100nF
- C11, C13: value C_20PF_0603 -> 20pF
- C4: value C_1UF_0603 -> 1uF
Connections:
- net +3V3: now also U3.21 (VREF+)
- net PB4: now also J1.PB4 (A28); no longer J1.A28
- net PB5: now also J1.PB5; no longer J1.A26
- net PE1: now also J1.PE1 (A20); no longer J1.A20
Other:
- moved on the sheet: C11, C12, C13, C14, J1, U3, Y1

Commit message: Hmmmm
Connections:
- net U1 is gone; now on net VBAT: J1.A3 (VBAT)
- net U2 is gone; now on net VA: J1.B3 (VA)
- net U3 is gone; now on net PC14: J1.A12 (PC14)
- net PB4: now also J1.A28 (PB4); no longer J1.PB4 (A28)
- net PB5: now also J1.A26 (PB5); no longer J1.PB5
- net PC14: no longer J1.A11 (PC14)
- net PC15: now also J1.A11 (PC15)
- net PE1: now also J1.A20 (PE1); no longer J1.PE1 (A20)
Other:
- company: (none) -> ${COMPANY}
- title: (none) -> ${TITLE}
Changed lines of the file:
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@@
 	(generator_version "9.0")
 	(paper "A3")
+	(title_block
+		(title "${TITLE}")
+		(rev "${REVISION}")
+		(company "${COMPANY}")
+		(comment 1 "${URL}")
+		(comment 2 "${AUTHOR}")
+		(comment 3 "${AUTHOR_EMAIL}")
+	)
 	(text "Analog power filtering"
 		(exclude_from_sim no)
@@
 		)
 	)
-	(global_label "PE5"
+	(global_label "PC15"
 		(shape passive)
-		(at 344.17 73.66 180)
+		(at 344.17 63.5 180)
 		(fields_autoplaced yes)
 		(effects
@@
 		)
 		(property "Intersheetrefs" "${INTERSHEET_REFS}"
-			(at 338.6676 73.66 0)
+			(at 337.3371 63.5 0)
 			(effects
 				(font
@@
 		)
 	)
-	(global_label "PE11"
+	(global_label "PE5"
 		(shape passive)
-		(at 231.14 88.9 180)
+		(at 344.17 73.66 180)
 		(fields_autoplaced yes)
 		(effects
@@
 		)
 		(property "Intersheetrefs" "${INTERSHEET_REFS}"
-			(at 224.4281 88.9 0)
+			(at 338.6676 73.66 0)
 			(effects
 				(font
@@
 		)
 	)
-	(global_label "PD11"
+	(global_label "PE11"
 		(shape passive)
-		(at 388.62 121.92 0)
+		(at 231.14 88.9 180)
 		(fields_autoplaced yes)
 		(effects
@@
 				(size 1.27 1.27)
 			)
-			(justify left)
+			(justify right)
 		)
 		(property "Intersheetrefs" "${INTERSHEET_REFS}"
-			(at 395.4529 121.92 0)
+			(at 224.4281 88.9 0)
 			(effects
 				(font
 					(size 1.27 1.27)
 				)
-				(justify left)
+				(justify right)
 				(hide yes)
 			)
 		)
 	)
-	(global_label "U1"
+	(global_label "PD11"
 		(shape passive)
-		(at 344.17 43.18 180)
+		(at 388.62 121.92 0)
 		(fields_autoplaced yes)
 		(effects
@@
 				(size 1.27 1.27)
 			)
-			(justify right)
+			(justify left)
 		)
 		(property "Intersheetrefs" "${INTERSHEET_REFS}"
-			(at 339.7561 43.18 0)
+			(at 395.4529 121.92 0)
 			(effects
 				(font
 					(size 1.27 1.27)
 				)
-				(justify right)
+				(justify left)
 				(hide yes)
 			)
@@
 	(global_label "PC14"
 		(shape passive)
-		(at 344.17 63.5 180)
+		(at 344.17 66.04 180)
 		(fields_autoplaced yes)
 		(effects
@@
 		)
 		(property "Intersheetrefs" "${INTERSHEET_REFS}"
-			(at 337.3371 63.5 0)
+			(at 337.3371 66.04 0)
 			(effects
 				(font
@@
 		)
 	)
-	(global_label "U3"
-		(shape passive)
-		(at 344.17 66.04 180)
-		(fields_autoplaced yes)
-		(effects
-			(font
-				(size 1.27 1.27)
-			)
-			(justify right)
-		)
-		(property "Intersheetrefs" "${INTERSHEET_REFS}"
-			(at 339.7561 66.04 0)
-			(effects
-				(font
-					(size 1.27 1.27)
-				)
-				(justify right)
-				(hide yes)
-			)
-		)
-	)
 	(global_label "PD11"
 		(shape passive)
@@
 		)
 	)
+	(global_label "VA"
+		(shape input)
+		(at 388.62 43.18 0)
+		(fields_autoplaced yes)
+		(effects
+			(font
+				(size 1.27 1.27)
+			)
+			(justify left)
+		)
+		(property "Intersheetrefs" "${INTERSHEET_REFS}"
+			(at 393.7824 43.18 0)
+			(effects
+				(font
+					(size 1.27 1.27)
+				)
+				(justify left)
+				(hide yes)
+			)
+		)
+	)
 	(global_label "HNRST"
 		(shape input)
@@
 		)
 	)
-	(global_label "U2"
-		(shape passive)
-		(at 388.62 43.18 0)
-		(fields_autoplaced yes)
-		(effects
-			(font
-				(size 1.27 1.27)
-			)
-			(justify left)
-		)
-		(property "Intersheetrefs" "${INTERSHEET_REFS}"
-			(at 393.0339 43.18 0)
-			(effects
-				(font
-					(size 1.27 1.27)
-				)
-				(justify left)
-				(hide yes)
-			)
-		)
-	)
 	(global_label "PB10"
 		(shape passive)
@@
 		)
 	)
+	(global_label "VBAT"
+		(shape input)
+		(at 344.17 43.18 180)
+		(fields_autoplaced yes)
+		(effects
+			(font
+				(size 1.27 1.27)
+			)
+			(justify right)
+		)
+		(property "Intersheetrefs" "${INTERSHEET_REFS}"
+			(at 336.77 43.18 0)
+			(effects
+				(font
+					(size 1.27 1.27)
+				)
+				(justify right)
+				(hide yes)
+			)
+		)
+	)
 	(global_label "PD13"
 		(shape passive)
@@
 		(pin "A19"
 		)
-		(pin "PE1"
+		(pin "A20"
 		)
 		(pin "A44"
@@
 		(pin "A41"
 		)
-		(pin "PB5"
+		(pin "A28"
 		)
 		(pin "A30"
@@
 		(pin "A43"
 		)
-		(pin "PB4"
+		(pin "A26"
 		)
 		(pin "B24"
