File: stmw-mcu-stm32f407/stmw-mcu-stm32f407.kicad_sch (KiCad schematic)
At the start: 41 parts, among them J2 TYPE-C-31-M-12, SW1 TS-1088R-02526, SW2 TS-1088R-02526, U1 AMS1117-3.3, U3 STM32F407VETx, Y1 X_16MHZ

Commit message: Hmmm
Parts:
- removed H1, H2: MountingHole, MountingHole:MountingHole_2.2mm_M2, symbol Mechanical:MountingHole
- D3: value LED_GREEN_0603 -> GR; LCSC C19171301 -> C118334
- D4: value LED_BLUE_0603 -> BL; LCSC C2288 -> C84266
- JP1, JP2: now not fitted; now left out of the parts list
- JP3, JP4: now left out of the parts list
Connections:
- net U7 is gone; now on net U4: J1.B27 (U4)
- net U8 is gone; now on net U5: J1.A38 (U5)
- net U9 is gone; now on net U6: J1.B38 (U6)
- net U4: no longer J1.A19 (U4)
- net U5: no longer J1.B19 (U5)
- net U6: no longer J1.A27 (U6)
- new net U1: J1.A19 (U1)
- new net U2: J1.B19 (U2)
- new net U3: J1.A27 (U3)
Changed lines of the file:
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@@
 		)
 	)
-	(global_label "U9"
+	(global_label "U6"
 		(shape passive)
 		(at 388.62 132.08 0)
@@
 		)
 	)
-	(global_label "U8"
+	(global_label "U5"
 		(shape passive)
 		(at 344.17 132.08 180)
@@
 		)
 	)
-	(global_label "U4"
+	(global_label "U1"
 		(shape passive)
 		(at 344.17 83.82 180)
@@
 		)
 	)
-	(global_label "U6"
+	(global_label "U3"
 		(shape passive)
 		(at 344.17 104.14 180)
@@
 		)
 	)
-	(global_label "U7"
+	(global_label "U4"
 		(shape passive)
 		(at 388.62 104.14 0)
@@
 		)
 	)
-	(global_label "U5"
+	(global_label "U2"
 		(shape passive)
 		(at 388.62 83.82 0)
@@
 			)
 		)
-		(property "Value" "LED_GREEN_0603"
-			(at 147.32 248.92 0)
+		(property "Value" "GR"
+			(at 152.654 257.81 90)
 			(effects
 				(font
 					(size 1.27 1.27)
 				)
-				(hide yes)
 			)
 		)
@@
 					(size 1.27 1.27)
 				)
+				(hide yes)
 			)
 		)
@@
 				)
 				(justify left)
+				(hide yes)
 			)
 		)
-		(property "LCSC" "C19171301"
+		(property "LCSC" "C118334"
 			(at 142.24 254 0)
 			(effects
@@
 			)
 		)
-		(property "Value" "LED_BLUE_0603"
-			(at 161.29 248.92 0)
+		(property "Value" "BL"
+			(at 166.624 257.81 90)
 			(effects
 				(font
 					(size 1.27 1.27)
 				)
-				(hide yes)
 			)
 		)
@@
 					(size 1.27 1.27)
 				)
+				(hide yes)
 			)
 		)
@@
 				)
 				(justify left)
+				(hide yes)
 			)
 		)
-		(property "LCSC" "C2288"
+		(property "LCSC" "C84266"
 			(at 156.21 254 0)
 			(effects
@@
 		(unit 1)
 		(exclude_from_sim no)
-		(in_bom yes)
+		(in_bom no)
 		(on_board yes)
 		(dnp no)
@@
 		(unit 1)
 		(exclude_from_sim no)
-		(in_bom yes)
+		(in_bom no)
 		(on_board yes)
 		(dnp no)
@@
 	)
 	(symbol
-		(lib_id "Mechanical:MountingHole")
-		(at 292.1 273.05 0)
-		(unit 1)
-		(exclude_from_sim no)
-		(in_bom no)
-		(on_board yes)
-		(dnp no)
-		(property "Reference" "H1"
-			(at 294.64 273.05 0)
-			(effects
-				(font
-					(size 1.27 1.27)
-				)
-				(justify left)
-			)
-		)
-		(property "Value" "MountingHole"
-			(at 294.64 274.3199 0)
-			(effects
-				(font
-					(size 1.27 1.27)
-				)
-				(justify left)
-				(hide yes)
-			)
-		)
-		(property "Footprint" "MountingHole:MountingHole_2.2mm_M2"
-			(at 292.1 273.05 0)
-			(effects
-				(font
-					(size 1.27 1.27)
-				)
-				(hide yes)
-			)
-		)
-		(property "Datasheet" "~"
-			(at 292.1 273.05 0)
-			(effects
-				(font
-					(size 1.27 1.27)
-				)
-				(hide yes)
-			)
-		)
-		(property "Description" "Mounting Hole without connection"
-			(at 292.1 273.05 0)
-			(effects
-				(font
-					(size 1.27 1.27)
-				)
-				(hide yes)
-			)
-		)
-		(instances
-			(project ""
-				(path "/a2bbec60-ecf6-4da0-b0d6-da34253985fb"
-					(reference "H1")
-					(unit 1)
-				)
-			)
-		)
-	)
-	(symbol
 		(lib_id "power:+3V3")
 		(at 76.2 24.13 0)
@@
 	)
 	(symbol
-		(lib_id "Mechanical:MountingHole")
-		(at 292.1 278.13 0)
-		(unit 1)
-		(exclude_from_sim no)
-		(in_bom no)
-		(on_board yes)
-		(dnp no)
-		(property "Reference" "H2"
-			(at 294.64 278.13 0)
-			(effects
-				(font
-					(size 1.27 1.27)
-				)
-				(justify left)
-			)
-		)
-		(property "Value" "MountingHole"
-			(at 294.64 279.3999 0)
-			(effects
-				(font
-					(size 1.27 1.27)
-				)
-				(justify left)
-				(hide yes)
-			)
-		)
-		(property "Footprint" "MountingHole:MountingHole_2.2mm_M2"
-			(at 292.1 278.13 0)
-			(effects
-				(font
-					(size 1.27 1.27)
-				)
-				(hide yes)
-			)
-		)
-		(property "Datasheet" "~"
-			(at 292.1 278.13 0)
-			(effects
-				(font
-					(size 1.27 1.27)
-				)
-				(hide yes)
-			)
-		)
-		(property "Description" "Mounting Hole without connection"
-			(at 292.1 278.13 0)
-			(effects
-				(font
-					(size 1.27 1.27)
-				)
-				(hide yes)
-			)
-		)
-		(instances
-			(project "stmw-mcu-stm32f405"
-				(path "/a2bbec60-ecf6-4da0-b0d6-da34253985fb"
-					(reference "H2")
-					(unit 1)
-				)
-			)
-		)
-	)
-	(symbol
 		(lib_id "power:PWR_FLAG")
 		(at 83.82 68.58 180)
@@
 		(unit 1)
 		(exclude_from_sim no)
-		(in_bom yes)
+		(in_bom no)
 		(on_board yes)
-		(dnp no)
+		(dnp yes)
 		(property "Reference" "JP1"
 			(at 29.21 66.04 0)
@@
 		(unit 1)
 		(exclude_from_sim no)
-		(in_bom yes)
+		(in_bom no)
 		(on_board yes)
-		(dnp no)
+		(dnp yes)
 		(property "Reference" "JP2"
 			(at 77.47 66.04 0)
