File: stmw-bp-5/stmw-bp-5.kicad_sch (KiCad schematic)
At the start: 11 parts, among them J1 Conn_02x25_Odd_Even, J2 Conn_02x25_Odd_Even, U1 X1611WVS-98-9TV01, U2 X1611WVS-98-9TV01, U3 X1611WVS-98-9TV01, U4 X1611WVS-98-9TV01, U5 X1611WVS-98-9TV01

Commit message: Hmmm
Parts:
- U1, U2, U3, U4, U5: symbol stm32world:X1611WVS-98-9TV01 -> stm32world:STMW_CONNECTOR
